Commit message: Se agrega fichero con la inercia mejorada

File: iri_wam_description/urdf/wam_sim_with_inertial.urdf (robot description, URDF)
Before this commit: robot iri_wam, 8 links, 7 joints
Links:
- link wam_fk/wam1: mass 0.1 -> 8.3936
- link wam_fk/wam2: mass 0.1 -> 4.8487
- link wam_fk/wam3: mass 0.1 -> 1.7251
- link wam_fk/wam4: mass 0.1 -> 2.0824
- link wam_fk/wam5: mass 0.1 -> 0.3067
- link wam_fk/wam6: mass 0.1 -> 0.4278
- link wam_fk/wam7: mass 0.1 -> 0.0557
- link wambase: mass 1 -> 1000
Joints:
- joint j2: axis 0 0 1  -> 0 1 0
