Commit message: new testing wam.urdfs -> to be removed in the future. This is done in order to try to use the same urdf files for rviz and gazebo

File: iri_wam_description/urdf/wam_sim.urdf (robot description, URDF)
Before this commit: robot iri_wam, 9 links, 8 joints
Links:
- removed link wam_fk/wam0
- link wam_fk/wam1: mass 1 -> 0.1
- link wam_fk/wam2: mass 1 -> 0.1
- link wam_fk/wam3: mass 1 -> 0.1
- link wam_fk/wam4: mass 1 -> 0.1
- link wam_fk/wam5: mass 1 -> 0.1
- link wam_fk/wam6: mass 1 -> 0.1
- link wam_fk/wam7: mass 1 -> 0.1
Joints:
- removed joint j0
- joint j1: axis 1 0 0 -> 0 0 1; origin xyz=0 0 0 rpy=-1.57 0 0 -> xyz=0.22 0.14 0.346 rpy=0 0 0; parent wam_fk/wam0 -> wambase
- joint j2: axis 1 0 0 -> 0 0 1; origin xyz=0 0 0 rpy=1.57 0 0 -> xyz=0 0 0 rpy=-1.5708 0 0
- joint j3: axis 1 0 0 -> 0 0 1; origin xyz=0.045 0 0.55 rpy=-1.57 0 0 -> xyz=0.0 0.0 0.0 rpy=1.5708 0 0
- joint j4: axis 1 0 0 -> 0 0 1; origin xyz=-0.045 0 0 rpy=1.57 0 0 -> xyz=0.045 0 0.55 rpy=-1.5708 0 0
- joint j5: axis 1 0 0 -> 0 0 1; origin xyz=0 0 0.3 rpy=-1.57 0 0 -> xyz=-0.045 -0.3 0 rpy=1.5708 0 0
- joint j6: axis 1 0 0 -> 0 0 1; origin xyz=0 0 0 rpy=1.57 0 0 -> xyz=0 0 0 rpy=-1.5708 0 0
- joint j7: axis 1 0 0 -> 0 0 1; origin xyz=0 0 0.06 rpy=0 0 0 -> xyz=0 0 0 rpy=1.5708 0 0

File: iri_wam_description/xacro/wam_sim.urdf.xacro (robot description, xacro)
@@ -84,4 +84,6 @@
   <xacro:Transmission name="link6_link7" jointName="j7" reduction="1" torque="1"/>
   <!-- PLUGINS -->
+<!--
   <include filename="$(find iri_wam_gazebo)/urdf/iri_wam.gazebo.xacro" />
+-->
 </robot>

Commit message: stl and urdf files updated

File: iri_wam_description/urdf/wam_sim.urdf (robot description, URDF)
Before this commit: robot iri_wam, 8 links, 7 joints
Joints:
- joint j4: limit lower=-2.8 upper=2.8 effort=30 velocity=2 -> lower=-0.9 upper=3.1 effort=30 velocity=2
- joint j5: limit lower=-2.8 upper=2.8 effort=30 velocity=2 -> lower=-4.8 upper=1.3 effort=30 velocity=2
- joint j6: limit lower=-2.8 upper=2.8 effort=30 velocity=2 -> lower=-1.6 upper=1.6 effort=30 velocity=2
- joint j7: limit lower=-2.8 upper=2.8 effort=30 velocity=2 -> lower=-2.2 upper=2.2 effort=30 velocity=2

Commit message: last good xacro and urdf files for simulated wam

File: iri_wam_description/urdf/wam_sim.urdf (robot description, URDF)
Before this commit: robot iri_wam, 8 links, 7 joints
Joints:
- joint j2: axis 0 1 0 -> 0 0 1

File: iri_wam_description/xacro/wam_sim.urdf.xacro (robot description, xacro)
@@ -86,4 +86,5 @@
   <xacro:Transmission name="link6_link7" jointName="j7" reduction="1" torque="1"/>
   <!-- PLUGINS -->
-  <include filename="$(find iri_wam_gazebo)/urdf/iri_wam.gazebo.xacro" />
+<!--  <include filename="$(find iri_wam_gazebo)/urdf/iri_wam.gazebo.xacro" />
+-->
 </robot>

Commit message: Add mass

File: iri_wam_description/urdf/wam_sim.urdf (robot description, URDF)
Before this commit: robot iri_wam, 8 links, 7 joints
Links:
- link wam_fk/wam1: mass 0.1 -> 8.3936
- link wam_fk/wam2: mass 0.1 -> 4.8487
- link wam_fk/wam3: mass 0.1 -> 1.7251
- link wam_fk/wam4: mass 0.1 -> 2.0824
- link wam_fk/wam5: mass 0.1 -> 0.3067
- link wam_fk/wam6: mass 0.1 -> 0.4278
- link wam_fk/wam7: mass 0.1 -> 0.0557
- link wambase: mass 1 -> 20
Joints:
- joint j2: axis 0 0 1  -> 0 1 0 

File: iri_wam_description/xacro/wam_sim.urdf.xacro (robot description, xacro)
@@ -58,17 +58,17 @@
 </xacro:macro>
   <!-- LINKS   -->
-  <xacro:Link name="wambase" xyz="0 0 0" rpy="0 0 0" mass="1" prefix=""/>
+  <xacro:Link name="wambase" xyz="0 0 0" rpy="0 0 0" mass="20" prefix=""/>
 <!-- TODO: Try to add wam0 virtual Link and its corresponding joint since it is how it is defined on the real kinematics
            Not sure if this is possible -->
-  <xacro:Link name="wam1" xyz="0 0 0" rpy="0 0 0" mass="0.1" prefix="wam_fk/"/>
-  <xacro:Link name="wam2" xyz="0 0 0" rpy="0 0 0" mass="0.1" prefix="wam_fk/"/>
-  <xacro:Link name="wam3" xyz="0 0 0" rpy="0 0 0" mass="0.1" prefix="wam_fk/"/>
-  <xacro:Link name="wam4" xyz="0 0 0" rpy="0 0 0" mass="0.1" prefix="wam_fk/"/>
-  <xacro:Link name="wam5" xyz="0 0 0" rpy="0 0 0" mass="0.1" prefix="wam_fk/"/>
-  <xacro:Link name="wam6" xyz="0 0 0" rpy="0 0 0" mass="0.1" prefix="wam_fk/"/>
-  <xacro:Link name="wam7" xyz="0 0 0" rpy="0 0 0" mass="0.1" prefix="wam_fk/"/>
+  <xacro:Link name="wam1" xyz="0 0 0" rpy="0 0 0" mass="8.3936" prefix="wam_fk/"/>
+  <xacro:Link name="wam2" xyz="0 0 0" rpy="0 0 0" mass="4.8487" prefix="wam_fk/"/>
+  <xacro:Link name="wam3" xyz="0 0 0" rpy="0 0 0" mass="1.7251" prefix="wam_fk/"/>
+  <xacro:Link name="wam4" xyz="0 0 0" rpy="0 0 0" mass="2.0824" prefix="wam_fk/"/>
+  <xacro:Link name="wam5" xyz="0 0 0" rpy="0 0 0" mass="0.3067" prefix="wam_fk/"/>
+  <xacro:Link name="wam6" xyz="0 0 0" rpy="0 0 0" mass="0.4278" prefix="wam_fk/"/>
+  <xacro:Link name="wam7" xyz="0 0 0" rpy="0 0 0" mass="0.0557" prefix="wam_fk/"/>
   <!-- JOINTS  -->
   <xacro:Joint name="j1" type="revolute" xyz="0.22 0.14 0.346" rpy="0 0 0" upperLim="2.6" lowerLim="-2.6" effort="30" velocity="2" axis="0 0 1" parent="wambase" child="wam_fk/wam1" />
-  <xacro:Joint name="j2" type="revolute" xyz="0 0 0" rpy="0 0 0" upperLim="2.0" lowerLim="-2.0" effort="30" velocity="2" axis="0 0 1 " parent="wam_fk/wam1" child="wam_fk/wam2" />
+  <xacro:Joint name="j2" type="revolute" xyz="0 0 0" rpy="0 0 0" upperLim="2.0" lowerLim="-2.0" effort="30" velocity="2" axis="0 1 0 " parent="wam_fk/wam1" child="wam_fk/wam2" />
   <xacro:Joint name="j3" type="revolute" xyz="0.0 0.0 0.0" rpy="0 0 0" upperLim="2.8" lowerLim="-2.8" effort="30" velocity="2" axis="0 0 1" parent="wam_fk/wam2" child="wam_fk/wam3" />
   <xacro:Joint name="j4" type="revolute" xyz="0.045 0 0.55" rpy="-${pi/2} 0 0" upperLim="3.1" lowerLim="-0.9" effort="30" velocity="2" axis="0 0 1" parent="wam_fk/wam3" child="wam_fk/wam4" />

Commit message: trying to make urdf definitions better

File: iri_wam_description/urdf/wam_sim.urdf (robot description, URDF)
Before this commit: robot iri_wam, 8 links, 7 joints
Links:
- added link world
- link wambase: mass 20 -> 1
Joints:
- added joint base_fix: type fixed, parent world, child wambase, origin xyz=0 0 0 rpy=0 0 0

File: iri_wam_description/xacro/wam_sim.urdf.xacro (robot description, xacro)
@@ -58,5 +58,6 @@
 </xacro:macro>
   <!-- LINKS   -->
-  <xacro:Link name="wambase" xyz="0 0 0" rpy="0 0 0" mass="20" prefix=""/>
+  <link name="world" />
+  <xacro:Link name="wambase" xyz="0 0 0" rpy="0 0 0" mass="1" prefix=""/>
 <!-- TODO: Try to add wam0 virtual Link and its corresponding joint since it is how it is defined on the real kinematics
            Not sure if this is possible -->
@@ -69,4 +70,9 @@
   <xacro:Link name="wam7" xyz="0 0 0" rpy="0 0 0" mass="0.0557" prefix="wam_fk/"/>
   <!-- JOINTS  -->
+  <joint name="base_fix" type="fixed">
+    <parent link="world"/>
+    <child link="wambase"/>
+    <origin rpy="0 0 0" xyz="0 0 0"/>
+  </joint>
   <xacro:Joint name="j1" type="revolute" xyz="0.22 0.14 0.346" rpy="0 0 0" upperLim="2.6" lowerLim="-2.6" effort="30" velocity="2" axis="0 0 1" parent="wambase" child="wam_fk/wam1" />
   <xacro:Joint name="j2" type="revolute" xyz="0 0 0" rpy="0 0 0" upperLim="2.0" lowerLim="-2.0" effort="30" velocity="2" axis="0 1 0 " parent="wam_fk/wam1" child="wam_fk/wam2" />

Commit message: Cambios en Joint's , Funcionando Perfectamente

File: iri_wam_description/urdf/wam_sim.urdf (robot description, URDF)
Before this commit: robot iri_wam, 9 links, 8 joints
Links:
- link wam_fk/wam1: geometry collision mesh filename=package://iri_wam_description/mesh/wam1.stl scale=1.0 1.0 1.0; visual mesh filename=package://iri_wam_description/mesh/wam1.stl scale=1.0 1.0 1.0
- link wam_fk/wam2: geometry collision mesh filename=package://iri_wam_description/mesh/wam2.stl scale=1.0 1.0 1.0; visual mesh filename=package://iri_wam_description/mesh/wam2.stl scale=1.0 1.0 1.0
- link wam_fk/wam3: geometry collision mesh filename=package://iri_wam_description/mesh/wam3.stl scale=1.0 1.0 1.0; visual mesh filename=package://iri_wam_description/mesh/wam3.stl scale=1.0 1.0 1.0
- link wam_fk/wam4: geometry collision mesh filename=package://iri_wam_description/mesh/wam4.stl scale=1.0 1.0 1.0; visual mesh filename=package://iri_wam_description/mesh/wam4.stl scale=1.0 1.0 1.0
- link wam_fk/wam5: geometry collision mesh filename=package://iri_wam_description/mesh/wam5.stl scale=1.0 1.0 1.0; visual mesh filename=package://iri_wam_description/mesh/wam5.stl scale=1.0 1.0 1.0
- link wam_fk/wam6: geometry collision mesh filename=package://iri_wam_description/mesh/wam6.stl scale=1.0 1.0 1.0; visual mesh filename=package://iri_wam_description/mesh/wam6.stl scale=1.0 1.0 1.0
- link wam_fk/wam7: geometry collision mesh filename=package://iri_wam_description/mesh/wam7.stl scale=1.0 1.0 1.0; visual mesh filename=package://iri_wam_description/mesh/wam7.stl scale=1.0 1.0 1.0
- link wambase: mass 1 -> 20; geometry collision mesh filename=package://iri_wam_description/mesh/wambase.stl scale=1.0 1.0 1.0; visual mesh filename=package://iri_wam_description/mesh/wambase.stl scale=1.0 1.0 1.0
Joints:
- joint base_fix: origin xyz=0 0 0 rpy=0 0 0 -> (none)
- joint j1: limit lower=-2.6 upper=2.6 effort=30 velocity=2 -> lower=-2.6 upper=2.6 effort=30 velocity=2.0
- joint j2: axis 0 1 0  -> 0 1 0; limit lower=-2.0 upper=2.0 effort=30 velocity=2 -> lower=-2.0 upper=2.0 effort=30 velocity=2.0; origin xyz=0 0 0 rpy=0 0 0 -> xyz=0.0 0.0 0.0 rpy=0 0 0
- joint j3: limit lower=-2.8 upper=2.8 effort=30 velocity=2 -> lower=-2.8 upper=2.8 effort=30 velocity=2.0
- joint j4: limit lower=-0.9 upper=3.1 effort=30 velocity=2 -> lower=-0.9 upper=2.8 effort=35 velocity=2.0; origin xyz=0.045 0 0.55 rpy=-1.5708 0 0 -> xyz=0.045 0.0 0.55 rpy=-1.57079632679 0 0
- joint j5: limit lower=-4.8 upper=1.3 effort=30 velocity=2 -> lower=-4.8 upper=1.3 effort=30 velocity=2.0; origin xyz=-0.045 -0.3 0 rpy=1.5708 0 0 -> xyz=-0.045 -0.3 0.0 rpy=1.57079632679 0 0
- joint j6: limit lower=-1.6 upper=1.6 effort=30 velocity=2 -> lower=-1.6 upper=1.6 effort=30 velocity=2.0; origin xyz=0 0 0 rpy=-1.5708 0 0 -> xyz=0.0 0.0 0.0 rpy=-1.57079632679 0 0
- joint j7: limit lower=-2.2 upper=2.2 effort=30 velocity=2 -> lower=-2.2 upper=2.2 effort=30 velocity=2.0; origin xyz=0 0 0 rpy=1.5708 0 0 -> xyz=0.0 0.0 0.0 rpy=1.57079632679 0 0

File: iri_wam_description/xacro/transmission.urdf.xacro (robot description, xacro)
@@ -6,6 +6,6 @@
        name="iri_wam">
 <xacro:macro name="Transmission" params="name jointName reduction torque">
-       <transmission type="pr2_mechanism_model/SimpleTransmission" name="${name}_trans">
-           <actuator name="${name}_motor" />
+       <transmission type="pr2_mechanism_model/SimpleTransmission" name="${name}_transmision">
+           <actuator name="${name}_controller" />
             <joint name="${jointName}" />
             <mechanicalReduction>${reduction}</mechanicalReduction>

File: iri_wam_description/xacro/wam1.urdf.xacro (robot description, xacro)
@@ -24,4 +24,5 @@
 -->
             </geometry>
+            <contact_coefficients kd="1.0" kp="1000.0" mu="0"/>
         </collision>
     </link>
@@ -35,7 +36,8 @@
         <origin xyz="0.22 0.14 0.346" rpy="0 0 0" />
         <axis xyz="0 0 1" />
-        <limit lower="-2.6" upper="2.6" effort="10" velocity="1.0"/>
-        <dynamics damping="200.5"/>
-    </joint>
+        <limit lower="-2.6" upper="2.6" effort="30" velocity="2.0"/>
+   <!--  <safety_controller k_velocity="0.5"/>-->
+        <dynamics damping="100"/>
+     </joint>
     <transmission type="pr2_mechanism_model/SimpleTransmission" name="wam_fk/wam1_transmission">
       <actuator name="wam_fk/wam1_rotation" />
@@ -43,5 +45,4 @@
       <mechanicalReduction>1</mechanicalReduction>
       <motorTorqueConstant>1</motorTorqueConstant>
-      <pulsesPerRevolution>90000</pulsesPerRevolution>
     </transmission>
   </xacro:macro>

File: iri_wam_description/xacro/wam2.urdf.xacro (robot description, xacro)
@@ -23,4 +23,5 @@
 <!--                <box size="0.10 0.10 0.10"/> -->
             </geometry>
+            <contact_coefficients kd="1.0" kp="1000.0" mu="0"/>
         </collision>
     </link>
@@ -34,6 +35,7 @@
         <origin xyz="0.0 0.0 0.0" rpy="0 0 0" />
         <axis xyz="0 1 0" />
-        <limit lower="-2.0" upper="2.0" effort="10" velocity="1.0"/>
-        <dynamics damping="200.5"/>
+        <limit lower="-2.0" upper="2.0" effort="30" velocity="2.0"/>
+        <!--<safety_controller k_velocity="0.5"/>-->
+        <dynamics damping="100"/>
     </joint>
     <transmission type="pr2_mechanism_model/SimpleTransmission" name="wam_fk/wam2_transmission">
@@ -42,5 +44,5 @@
       <mechanicalReduction>1</mechanicalReduction>
       <motorTorqueConstant>1</motorTorqueConstant>
-      <pulsesPerRevolution>90000</pulsesPerRevolution>
+      <!--<pulsesPerRevolution>90000</pulsesPerRevolution>-->
     </transmission>
   </xacro:macro>

File: iri_wam_description/xacro/wam3.urdf.xacro (robot description, xacro)
@@ -23,4 +23,5 @@
 <!--                <box size="0.10 0.10 0.10"/> -->
             </geometry>
+            <contact_coefficients kd="1.0" kp="1000.0" mu="0"/>
         </collision>
     </link>
@@ -34,6 +35,7 @@
         <origin xyz="0.0 0.0 0.0" rpy="0 0 0" />
         <axis xyz="0 0 1" />
-        <limit lower="-2.8" upper="2.8" effort="10" velocity="1.0"/>
-        <dynamics damping="200.5"/>
+        <limit lower="-2.8" upper="2.8" effort="30" velocity="2.0"/>
+        <!--  <safety_controller k_velocity="0.5"/>-->
+        <dynamics damping="100"/>
     </joint>
     <transmission type="pr2_mechanism_model/SimpleTransmission" name="wam_fk/wam3_transmission">
@@ -42,5 +44,5 @@
       <mechanicalReduction>1</mechanicalReduction>
       <motorTorqueConstant>1</motorTorqueConstant>
-      <pulsesPerRevolution>90000</pulsesPerRevolution>
+     <!-- <pulsesPerRevolution>90000</pulsesPerRevolution>-->
     </transmission>
   </xacro:macro>

File: iri_wam_description/xacro/wam4.urdf.xacro (robot description, xacro)
@@ -24,4 +24,5 @@
 <!--                <box size="0.10 0.10 0.10"/> -->
             </geometry>
+            <contact_coefficients kd="1.0" kp="1000.0" mu="0"/>
         </collision>
     </link>
@@ -35,6 +36,7 @@
         <origin xyz="0.045 0.0 0.55" rpy="-${M_PI/2} 0 0" />
         <axis xyz="0 0 1" />
-        <limit lower="-0.9" upper="2.8" effort="10" velocity="1.0"/>
-        <dynamics damping="200.5"/>
+        <limit lower="-0.9" upper="2.8" effort="35" velocity="2.0"/>
+  <!--  <safety_controller k_velocity="0.5"/>-->
+  <dynamics damping="100"/>
     </joint>
     <transmission type="pr2_mechanism_model/SimpleTransmission" name="wam_fk/wam4_transmission">
@@ -43,5 +45,5 @@
       <mechanicalReduction>1</mechanicalReduction>
       <motorTorqueConstant>1</motorTorqueConstant>
-      <pulsesPerRevolution>90000</pulsesPerRevolution>
+      <!--<pulsesPerRevolution>90000</pulsesPerRevolution>-->
     </transmission>
   </xacro:macro>

File: iri_wam_description/xacro/wam5.urdf.xacro (robot description, xacro)
@@ -24,4 +24,5 @@
 <!--                <box size="0.10 0.10 0.10"/> -->
             </geometry>
+            <contact_coefficients kd="1.0" kp="1000.0" mu="0"/>
         </collision>
     </link>
@@ -35,6 +36,7 @@
         <origin xyz="-0.045 -0.3 0.0" rpy="${M_PI/2} 0 0" />
         <axis xyz="0 0 1" />
-        <limit lower="-4.8" upper="1.3" effort="10" velocity="1.0"/>
-        <dynamics damping="200.5"/>
+        <limit lower="-4.8" upper="1.3" effort="30" velocity="2.0"/>
+   <!--  <safety_controller k_velocity="0.5"/>-->
+   <dynamics damping="100"/>
     </joint>
     <transmission type="pr2_mechanism_model/SimpleTransmission" name="wam_fk/wam5_transmission">
@@ -43,5 +45,5 @@
       <mechanicalReduction>1</mechanicalReduction>
       <motorTorqueConstant>1</motorTorqueConstant>
-      <pulsesPerRevolution>90000</pulsesPerRevolution>
+    <!--  <pulsesPerRevolution>90000</pulsesPerRevolution>-->
     </transmission>
   </xacro:macro>

File: iri_wam_description/xacro/wam6.urdf.xacro (robot description, xacro)
@@ -24,4 +24,5 @@
 <!--                <box size="0.10 0.10 0.10"/> -->
             </geometry>
+            <contact_coefficients kd="1.0" kp="1000.0" mu="0"/>
         </collision>
     </link>
@@ -35,6 +36,7 @@
         <origin xyz="0.0 0.0 0.0" rpy="-${M_PI/2} 0 0" />
         <axis xyz="0 0 1" />
-        <limit lower="-1.6" upper="1.6" effort="10" velocity="1.0"/>
-        <dynamics damping="200.5"/>
+        <limit lower="-1.6" upper="1.6" effort="30" velocity="2.0"/>
+        <!--  <safety_controller k_velocity="0.5"/>-->
+        <dynamics damping="100"/>
     </joint>
     <transmission type="pr2_mechanism_model/SimpleTransmission" name="wam_fk/wam6_transmission">
@@ -43,5 +45,5 @@
       <mechanicalReduction>1</mechanicalReduction>
       <motorTorqueConstant>1</motorTorqueConstant>
-      <pulsesPerRevolution>90000</pulsesPerRevolution>
+    <!--  <pulsesPerRevolution>90000</pulsesPerRevolution>-->
     </transmission>
   </xacro:macro>

File: iri_wam_description/xacro/wam7.urdf.xacro (robot description, xacro)
@@ -24,4 +24,5 @@
 <!--                <box size="0.10 0.10 0.10"/> -->
             </geometry>
+            <contact_coefficients kd="1.0" kp="1000.0" mu="0"/>
         </collision>
     </link>
@@ -35,6 +36,7 @@
         <origin xyz="0.0 0.0 0.0" rpy="${M_PI/2} 0 0" />
         <axis xyz="0 0 1" />
-        <limit lower="-2.2" upper="2.2" effort="10" velocity="1.0"/>
-        <dynamics damping="200.5"/>
+        <limit lower="-2.2" upper="2.2" effort="30" velocity="2.0"/>
+      <!--  <safety_controller k_velocity="0.5"/>-->
+      <dynamics damping="100"/>
     </joint>
     <transmission type="pr2_mechanism_model/SimpleTransmission" name="wam_fk/wam7_transmission">
@@ -43,5 +45,5 @@
       <mechanicalReduction>1</mechanicalReduction>
       <motorTorqueConstant>1</motorTorqueConstant>
-      <pulsesPerRevolution>90000</pulsesPerRevolution>
+      <!--<pulsesPerRevolution>90000</pulsesPerRevolution>-->
     </transmission>
   </xacro:macro>

File: iri_wam_description/xacro/wam_sim.urdf.xacro (robot description, xacro)
@@ -31,4 +31,4 @@
   </xacro:wam7>
   <!-- PLUGINS -->
-  <!--  <include filename="$(find iri_wam_gazebo)/urdf/iri_wam.gazebo.xacro" /> -->
+  <include filename="$(find iri_wam_gazebo)/urdf/iri_wam.gazebo.xacro" />
 </robot>

File: iri_wam_description/xacro/wambase.urdf.xacro (robot description, xacro)
@@ -23,7 +23,7 @@
       <geometry name="wambase_collision">
         <mesh filename="package://iri_wam_description/mesh/wambase.stl" scale="1.0 1.0 1.0" />
-<!--        <box size="0.35 0.28 0.16"/>
--->
+<!--        <box size="0.35 0.28 0.16"/>-->
       </geometry>
+      <contact_coefficients kd="1.0" kp="1000.0" mu="0"/>
     </collision>
   </link>
@@ -35,5 +35,4 @@
     <parent link="world"/>
     <child link="wambase"/>
-    <origin rpy="0 0 0" xyz="0 0 0"/>
   </joint>
 </xacro:macro>
