Commit message: getting better with gazebo and rviz correspondence although not good enough yet

File: iri_wam_description/urdf/wam.urdf (robot description, URDF)
Before this commit: robot iri_wam, 9 links, 8 joints
Links:
- link wam_fk/wam0: mass 1 -> 0.1; geometry collision mesh filename=package://iri_wam_description/mesh/wam0.stl
- link wam_fk/wam1: mass 1 -> 0.1
- link wam_fk/wam2: mass 1 -> 0.1
- link wam_fk/wam3: mass 1 -> 0.1
- link wam_fk/wam4: mass 1 -> 0.1
- link wam_fk/wam5: mass 1 -> 0.1
- link wam_fk/wam6: mass 1 -> 0.1
- link wam_fk/wam7: mass 1 -> 0.1
Joints:
- joint j0: axis 1 0 0 -> 0 0 1; type fixed -> revolute
- joint j1: axis 1 0 0 -> 0 1 0; origin xyz=0 0 0 rpy=-1.57 0 0 -> xyz=0 0 0 rpy=-1.5708 0 0
- joint j2: axis 1 0 0 -> 0 1 0; origin xyz=0 0 0 rpy=1.57 0 0 -> xyz=0 0 0 rpy=1.5708 0 0
- joint j3: axis 1 0 0 -> 0 0 1; origin xyz=0.045 0 0.55 rpy=-1.57 0 0 -> xyz=0.045 0 0.55 rpy=-1.5708 0 0
- joint j4: axis 1 0 0 -> 0 0 1; origin xyz=-0.045 0 0 rpy=1.57 0 0 -> xyz=-0.045 0 0 rpy=1.5708 0 0
- joint j5: axis 1 0 0 -> 0 0 1; origin xyz=0 0 0.3 rpy=-1.57 0 0 -> xyz=0 0 0.3 rpy=-1.5708 0 0
- joint j6: axis 1 0 0 -> 0 0 1; origin xyz=0 0 0 rpy=1.57 0 0 -> xyz=0 0 0 rpy=1.5708 0 0
- joint j7: axis 1 0 0 -> 0 0 1

File: iri_wam_description/xacro/wam.urdf.xacro (robot description, xacro)
@@ -6,11 +6,11 @@
        name="iri_wam">
       <!-- Constants -->
- <xacro:property name="pi" value="1.57" />
+ <xacro:property name="pi" value="3.1416" />
    <!-- Includes -->
 <include filename="$(find iri_wam_description)/xacro/transmission.urdf.xacro" />
 <!-- MACROS -->
-<xacro:macro name="intertial_default" params="mass">
+<xacro:macro name="intertial_default" params="mass xyz rpy">
 	<inertial>
-	   <origin xyz="0 0 0" rpy="0 0 0" />
+	   <origin xyz="${xyz}" rpy="${rpy}" />
        <mass value="${mass}"/>
        <inertia ixx="100"  ixy="0"  ixz="0" iyy="100" iyz="0" izz="100" />
@@ -43,5 +43,5 @@
 <xacro:macro name="Link"  params="name xyz rpy mass prefix">
   <link name="${prefix}${name}">
-	<xacro:intertial_default mass="${mass}"/>
+	<xacro:intertial_default mass="${mass}" xyz="${xyz}" rpy="${rpy}" />
 	<xacro:Visual name="${name}" xyz="${xyz}" rpy="${rpy}" />
 	<xacro:Collision name="${name}" xyz="${xyz}" rpy="${rpy}"/>
@@ -60,26 +60,44 @@
   <xacro:Link name="wambase" xyz="0 0 0" rpy="0 0 0" mass="1" prefix=""/>
   <link name="wam_fk/wam0">
-  	<inertial>
-	   <origin xyz="0 0 0" rpy="0 0 0" />
-       <mass value="1"/>
-       <inertia ixx="100"  ixy="0"  ixz="0" iyy="100" iyz="0" izz="100" />
-	</inertial>
+    <inertial>
+      <origin rpy="0 0 0" xyz="0 0 0"/>
+      <mass value="0.1"/>
+      <inertia ixx="100" ixy="0" ixz="0" iyy="100" iyz="0" izz="100"/>
+    </inertial>
+<!--
+    <visual>
+      <origin rpy="0 0 0" xyz="0 0 0"/>
+      <geometry name="wam0-geom">
+        <mesh filename="package://iri_wam_description/mesh/wam0.stl"/>
+      </geometry>
+      <material name="wam0-mat">
+        <color rgba="0.75 0.75 0.75 1.0"/>
+      </material>
+    </visual>
+-->
+    <collision>
+      <origin rpy="0 0 0" xyz="0 0 0"/>
+      <geometry name="wam0-geom">
+        <mesh filename="package://iri_wam_description/mesh/wam0.stl"/>
+      </geometry>
+      <contact_coefficients kd="1.0" kp="1000.0" mu="0"/>
+    </collision>
   </link>
-  <xacro:Link name="wam1" xyz="0 0 0" rpy="${pi} 0 0" mass="1" prefix="wam_fk/"/>
-  <xacro:Link name="wam2" xyz="0 0 0" rpy="-${pi} 0 0" mass="1" prefix="wam_fk/"/>
-  <xacro:Link name="wam3" xyz="-0.045 0.55 0" rpy="${pi} 0 0" mass="1" prefix="wam_fk/"/>
-  <xacro:Link name="wam4" xyz="0.045 0 0" rpy="-${pi} 0 0" mass="1" prefix="wam_fk/"/>
-  <xacro:Link name="wam5" xyz="0 0 0" rpy="${pi} 0 0" mass="1" prefix="wam_fk/"/>
-  <xacro:Link name="wam6" xyz="0 0 0" rpy="-${pi} 0 0" mass="1" prefix="wam_fk/"/>
-  <xacro:Link name="wam7" xyz="0 0 -0.06" rpy="0 0 0" mass="1" prefix="wam_fk/"/>
+  <xacro:Link name="wam1" xyz="0 0 0" rpy="${pi/2} 0 0" mass="0.1" prefix="wam_fk/"/>
+  <xacro:Link name="wam2" xyz="0 0 0" rpy="-${pi/2} 0 0" mass="0.1" prefix="wam_fk/"/>
+  <xacro:Link name="wam3" xyz="-0.045 0.55 0" rpy="${pi/2} 0 0" mass="0.1" prefix="wam_fk/"/>
+  <xacro:Link name="wam4" xyz="0.045 0 0" rpy="-${pi/2} 0 0" mass="0.1" prefix="wam_fk/"/>
+  <xacro:Link name="wam5" xyz="0 0 0" rpy="${pi/2} 0 0" mass="0.1" prefix="wam_fk/"/>
+  <xacro:Link name="wam6" xyz="0 0 0" rpy="-${pi/2} 0 0" mass="0.1" prefix="wam_fk/"/>
+  <xacro:Link name="wam7" xyz="0 0 -0.06" rpy="0 0 0" mass="0.1" prefix="wam_fk/"/>
 <!-- JOINTS  -->
-  <xacro:Joint name="j0" type="fixed"    xyz="0.22 0.14 0.346" rpy="0 0 0" upperLim="2.6" lowerLim="-2.6" effort="30" velocity="2" axis="1 0 0" parent="wambase" child="wam_fk/wam0" />
-  <xacro:Joint name="j1" type="revolute" xyz="0 0 0" rpy="-${pi} 0 0" upperLim="2.6" lowerLim="-2.6" effort="30" velocity="2" axis="1 0 0" parent="wam_fk/wam0" child="wam_fk/wam1" />
-  <xacro:Joint name="j2" type="revolute" xyz="0 0 0" rpy="${pi} 0 0" upperLim="2.0" lowerLim="-2.0" effort="30" velocity="2" axis="1 0 0" parent="wam_fk/wam1" child="wam_fk/wam2" />
-  <xacro:Joint name="j3" type="revolute" xyz="0.045 0 0.55" rpy="-${pi} 0 0" upperLim="2.8" lowerLim="-2.8" effort="30" velocity="2" axis="1 0 0" parent="wam_fk/wam2" child="wam_fk/wam3" />
-  <xacro:Joint name="j4" type="revolute" xyz="-0.045 0 0" rpy="${pi} 0 0" upperLim="2.8" lowerLim="-2.8" effort="30" velocity="2" axis="1 0 0" parent="wam_fk/wam3" child="wam_fk/wam4" />
-  <xacro:Joint name="j5" type="revolute" xyz="0 0 0.3" rpy="-${pi} 0 0" upperLim="2.8" lowerLim="-2.8" effort="30" velocity="2" axis="1 0 0" parent="wam_fk/wam4" child="wam_fk/wam5" />
-  <xacro:Joint name="j6" type="revolute" xyz="0 0 0" rpy="${pi} 0 0" upperLim="2.8" lowerLim="-2.8" effort="30" velocity="2" axis="1 0 0" parent="wam_fk/wam5" child="wam_fk/wam6" />
-  <xacro:Joint name="j7" type="revolute" xyz="0 0 0.06" rpy="0 0 0" upperLim="2.8" lowerLim="-2.8" effort="30" velocity="2" axis="1 0 0" parent="wam_fk/wam6" child="wam_fk/wam7" />
+  <xacro:Joint name="j0" type="revolute" xyz="0.22 0.14 0.346" rpy="0 0 0" upperLim="2.6" lowerLim="-2.6" effort="30" velocity="2" axis="0 0 1" parent="wambase" child="wam_fk/wam0" />
+  <xacro:Joint name="j1" type="revolute" xyz="0 0 0" rpy="-${pi/2} 0 0" upperLim="2.6" lowerLim="-2.6" effort="30" velocity="2" axis="0 1 0" parent="wam_fk/wam0" child="wam_fk/wam1" />
+  <xacro:Joint name="j2" type="revolute" xyz="0 0 0" rpy="${pi/2} 0 0" upperLim="2.0" lowerLim="-2.0" effort="30" velocity="2" axis="0 1 0" parent="wam_fk/wam1" child="wam_fk/wam2" />
+  <xacro:Joint name="j3" type="revolute" xyz="0.045 0 0.55" rpy="-${pi/2} 0 0" upperLim="2.8" lowerLim="-2.8" effort="30" velocity="2" axis="0 0 1" parent="wam_fk/wam2" child="wam_fk/wam3" />
+  <xacro:Joint name="j4" type="revolute" xyz="-0.045 0 0" rpy="${pi/2} 0 0" upperLim="2.8" lowerLim="-2.8" effort="30" velocity="2" axis="0 0 1" parent="wam_fk/wam3" child="wam_fk/wam4" />
+  <xacro:Joint name="j5" type="revolute" xyz="0 0 0.3" rpy="-${pi/2} 0 0" upperLim="2.8" lowerLim="-2.8" effort="30" velocity="2" axis="0 0 1" parent="wam_fk/wam4" child="wam_fk/wam5" />
+  <xacro:Joint name="j6" type="revolute" xyz="0 0 0" rpy="${pi/2} 0 0" upperLim="2.8" lowerLim="-2.8" effort="30" velocity="2" axis="0 0 1" parent="wam_fk/wam5" child="wam_fk/wam6" />
+  <xacro:Joint name="j7" type="revolute" xyz="0 0 0.06" rpy="0 0 0" upperLim="2.8" lowerLim="-2.8" effort="30" velocity="2" axis="0 0 1" parent="wam_fk/wam6" child="wam_fk/wam7" />
   <!-- Transmission -->
   <xacro:Transmission name="linkb_link0" jointName="j0" reduction="1" torque="1"/>

Commit message: tests for checking wam description on gazebo and rviz

File: iri_wam_description/urdf/wam.urdf (robot description, URDF)
Before this commit: robot iri_wam, 9 links, 8 joints
Links:
- removed link wam_fk/wam3
- removed link wam_fk/wam4
- removed link wam_fk/wam5
- removed link wam_fk/wam6
- removed link wam_fk/wam7
- link wam_fk/wam0: geometry 
Joints:
- removed joint j3
- removed joint j4
- removed joint j5
- removed joint j6
- removed joint j7
- joint j0: axis 0 0 1 -> 0 0 0; limit lower=-2.6 upper=2.6 effort=30 velocity=2 -> lower=0.0 upper=0.0 effort=0.0 velocity=0.0; origin xyz=0.22 0.14 0.346 rpy=0 0 0 -> xyz=0 0 0 rpy=0 0 0; type revolute -> fixed
- joint j1: axis 0 1 0 -> 0 -1 0; origin xyz=0 0 0 rpy=-1.5708 0 0 -> xyz=0 0 0 rpy=-1.57080 0 0
- joint j2: origin xyz=0 0 0 rpy=1.5708 0 0 -> xyz=0 0 0 rpy=1.57080 0 0

Commit message: urdf files updated

File: iri_wam_description/urdf/wam.urdf (robot description, URDF)
Before this commit: robot iri_wam, 4 links, 3 joints
Links:
- added link wam_fk/wam3, mass 0.1; collision mesh filename=package://iri_wam_description/mesh/wam3.stl; visual mesh filename=package://iri_wam_description/mesh/wam3.stl
- added link wam_fk/wam4, mass 0.1; collision mesh filename=package://iri_wam_description/mesh/wam4.stl; visual mesh filename=package://iri_wam_description/mesh/wam4.stl
- added link wam_fk/wam5, mass 0.1; collision mesh filename=package://iri_wam_description/mesh/wam5.stl; visual mesh filename=package://iri_wam_description/mesh/wam5.stl
- added link wam_fk/wam6, mass 0.1; collision mesh filename=package://iri_wam_description/mesh/wam6.stl; visual mesh filename=package://iri_wam_description/mesh/wam6.stl
- added link wam_fk/wam7, mass 0.1; collision mesh filename=package://iri_wam_description/mesh/wam7.stl; visual mesh filename=package://iri_wam_description/mesh/wam7.stl
Joints:
- added joint j3: type revolute, parent wam_fk/wam2, child wam_fk/wam3, origin xyz=0.045 0 0.55 rpy=-1.5708 0 0, axis 0 -1 0, limit lower=-2.8 upper=2.8 effort=30 velocity=2
- added joint j4: type revolute, parent wam_fk/wam3, child wam_fk/wam4, origin xyz=-0.045 0 0 rpy=1.5708 0 0, axis 0 1 0, limit lower=-0.9 upper=3.1 effort=30 velocity=2
- added joint j5: type revolute, parent wam_fk/wam4, child wam_fk/wam5, origin xyz=0 0 0.3 rpy=-1.5708 0 0, axis 0 -1 0, limit lower=-4.8 upper=1.3 effort=30 velocity=2
- added joint j6: type revolute, parent wam_fk/wam5, child wam_fk/wam6, origin xyz=0 0 0 rpy=1.5708 0 0, axis 0 1 0, limit lower=-1.6 upper=1.6 effort=30 velocity=2
- added joint j7: type revolute, parent wam_fk/wam6, child wam_fk/wam7, origin xyz=0 0 0.06 rpy=0 0 0, axis 0 0 1, limit lower=-2.2 upper=2.2 effort=30 velocity=2
- joint j0: origin xyz=0 0 0 rpy=0 0 0 -> xyz=0.22 0.14 0.346 rpy=0 0 0
- joint j1: origin xyz=0 0 0 rpy=-1.57080 0 0 -> xyz=0.22 0.14 0.346 rpy=-1.5708 0 0; parent wam_fk/wam0 -> wambase
- joint j2: origin xyz=0 0 0 rpy=1.57080 0 0 -> xyz=0 0 0 rpy=1.5708 0 0

File: iri_wam_description/urdf/wam_sim.urdf (robot description, URDF)
Before this commit: robot iri_wam, 8 links, 7 joints
Joints:
- joint j2: axis 0 0 1 -> 0 1 0; origin xyz=0 0 0 rpy=-1.5708 0 0 -> xyz=0 0 0 rpy=0 0 0
- joint j3: origin xyz=0.0 0.0 0.0 rpy=1.5708 0 0 -> xyz=0.0 0.0 0.0 rpy=0 0 0

Commit message: pfc ivan,Falta probarlo

File: iri_wam_description/urdf/wam.urdf (robot description, URDF)
Before this commit: robot iri_wam, 9 links, 8 joints
Links:
- link wam_fk/wam0: mass 0.1 -> 1; geometry collision cylinder length=0.015 radius=0.015; visual cylinder length=0.015 radius=0.015
Joints:
- joint j1: origin xyz=0.22 0.14 0.346 rpy=-1.5708 0 0 -> xyz=0 0 0 rpy=-1.57  0 0
- joint j2: origin xyz=0 0 0 rpy=1.5708 0 0 -> xyz=0 0 0 rpy=1.57 0 0
- joint j3: origin xyz=0.045 0 0.55 rpy=-1.5708 0 0 -> xyz=0.045 0 0.55 rpy=-1.57 0 0
- joint j4: origin xyz=-0.045 0 0 rpy=1.5708 0 0 -> xyz=-0.045 0 0 rpy=1.57 0 0
- joint j5: origin xyz=0 0 0.3 rpy=-1.5708 0 0 -> xyz=0 0 0.3 rpy=-1.57 0 0
- joint j6: origin xyz=0 0 0 rpy=1.5708 0 0 -> xyz=0 0 0 rpy=1.57 0 0

File: iri_wam_description/xacro/wam.urdf.xacro (robot description, xacro)
@@ -65,4 +65,20 @@
       <inertia ixx="100" ixy="0" ixz="0" iyy="100" iyz="0" izz="100"/>
     </inertial>
+	<visual>
+	  <origin xyz="0 0 0" rpy="0 0 0" />
+      <geometry name="wam_fk/wam0-geom">
+        <cylinder radius="0.015" length="0.015" />
+      </geometry>
+      <material name="Cyan">
+        <color rgba="1 0 0 1"/>
+      </material>
+	</visual>
+	<collision>
+	  <origin xyz="0 0 0" rpy="0 0 0" />
+      <geometry name="wam_fk/wam0-geom">
+        <cylinder radius="0.015" length="0.015" />
+      </geometry>
+       <contact_coefficients mu="0" kp="1000.0" kd="1.0"/>
+     </collision>
   </link>
   <xacro:Link name="wam1" xyz="0 0 0" rpy="${pi/2} 0 0" mass="0.1" prefix="wam_fk/"/>
@@ -77,10 +93,27 @@
   <xacro:Joint name="j1" type="revolute" xyz="0.22 0.14 0.346" rpy="-${pi/2} 0 0" upperLim="2.6" lowerLim="-2.6" effort="30" velocity="2" axis="0 -1 0" parent="wambase" child="wam_fk/wam1" />
   <xacro:Joint name="j2" type="revolute" xyz="0 0 0" rpy="${pi/2} 0 0" upperLim="2.0" lowerLim="-2.0" effort="30" velocity="2" axis="0 1 0" parent="wam_fk/wam1" child="wam_fk/wam2" />
-  <xacro:Joint name="j3" type="revolute" xyz="0.045 0 0.55" rpy="-${pi/2} 0 0" upperLim="2.8" lowerLim="-2.8" effort="30" velocity="2" axis="0 -1 0" parent="wam_fk/wam2" child="wam_fk/wam3" />
-  <xacro:Joint name="j4" type="revolute" xyz="-0.045 0 0" rpy="${pi/2} 0 0" upperLim="3.1" lowerLim="-0.9" effort="30" velocity="2" axis="0 1 0" parent="wam_fk/wam3" child="wam_fk/wam4" />
-  <xacro:Joint name="j5" type="revolute" xyz="0 0 0.3" rpy="-${pi/2} 0 0" upperLim="1.3" lowerLim="-4.8" effort="30" velocity="2" axis="0 -1 0" parent="wam_fk/wam4" child="wam_fk/wam5" />
-  <xacro:Joint name="j6" type="revolute" xyz="0 0 0" rpy="${pi/2} 0 0" upperLim="1.6" lowerLim="-1.6" effort="30" velocity="2" axis="0 1 0" parent="wam_fk/wam5" child="wam_fk/wam6" />
-  <xacro:Joint name="j7" type="revolute" xyz="0 0 0.06" rpy="0 0 0" upperLim="2.2" lowerLim="-2.2" effort="30" velocity="2" axis="0 0 1" parent="wam_fk/wam6" child="wam_fk/wam7" />
+  <xacro:Joint name="j3" type="revolute" xyz="0.045 0 0.55" rpy="-${pi/2} 0 0" upperLim="2.8" lowerLim="-2.8" effort="30" velocity="2" axis="0 0 1" parent="wam_fk/wam2" child="wam_fk/wam3" />
+  <xacro:Joint name="j4" type="revolute" xyz="-0.045 0 0" rpy="${pi/2} 0 0" upperLim="2.8" lowerLim="-2.8" effort="30" velocity="2" axis="0 0 1" parent="wam_fk/wam3" child="wam_fk/wam4" />
+  <xacro:Joint name="j5" type="revolute" xyz="0 0 0.3" rpy="-${pi/2} 0 0" upperLim="2.8" lowerLim="-2.8" effort="30" velocity="2" axis="0 0 1" parent="wam_fk/wam4" child="wam_fk/wam5" />
+  <xacro:Joint name="j6" type="revolute" xyz="0 0 0" rpy="${pi/2} 0 0" upperLim="2.8" lowerLim="-2.8" effort="30" velocity="2" axis="0 0 1" parent="wam_fk/wam5" child="wam_fk/wam6" />
+  <xacro:Joint name="j7" type="revolute" xyz="0 0 0.06" rpy="0 0 0" upperLim="2.8" lowerLim="-2.8" effort="30" velocity="2" axis="0 0 1" parent="wam_fk/wam6" child="wam_fk/wam7" />
+  <xacro:Joint name="j0" type="fixed"    xyz="0.22 0.14 0.346" rpy="0 0 0" upperLim="2.6" lowerLim="-2.6" effort="30" velocity="2" axis="1 0 0" parent="wambase" child="wam_fk/wam0" />
+  <xacro:Joint name="j1" type="revolute" xyz="0 0 0" rpy="-${pi}  0 0" upperLim="2.6" lowerLim="-2.6" effort="30" velocity="2" axis="1 0 0" parent="wam_fk/wam0" child="wam_fk/wam1" />
+  <xacro:Joint name="j2" type="revolute" xyz="0 0 0" rpy="${pi} 0 0" upperLim="2.0" lowerLim="-2.0" effort="30" velocity="2" axis="1 0 0" parent="wam_fk/wam1" child="wam_fk/wam2" />
+  <xacro:Joint name="j3" type="revolute" xyz="0.045 0 0.55" rpy="-${pi} 0 0" upperLim="2.8" lowerLim="-2.8" effort="30" velocity="2" axis="1 0 0" parent="wam_fk/wam2" child="wam_fk/wam3" />
+  <xacro:Joint name="j4" type="revolute" xyz="-0.045 0 0" rpy="${pi} 0 0" upperLim="2.8" lowerLim="-2.8" effort="30" velocity="2" axis="1 0 0" parent="wam_fk/wam3" child="wam_fk/wam4" />
+  <xacro:Joint name="j5" type="revolute" xyz="0 0 0.3" rpy="-${pi} 0 0" upperLim="2.8" lowerLim="-2.8" effort="30" velocity="2" axis="1 0 0" parent="wam_fk/wam4" child="wam_fk/wam5" />
+  <xacro:Joint name="j6" type="revolute" xyz="0 0 0" rpy="${pi} 0 0" upperLim="2.8" lowerLim="-2.8" effort="30" velocity="2" axis="1 0 0" parent="wam_fk/wam5" child="wam_fk/wam6" />
+  <xacro:Joint name="j7" type="revolute" xyz="0 0 0.06" rpy="0 0 0" upperLim="2.8" lowerLim="-2.8" effort="30" velocity="2" axis="1 0 0" parent="wam_fk/wam6" child="wam_fk/wam7" />
+  <!-- Transmission -->
+  <xacro:Transmission name="linkb_link0" jointName="j0" reduction="1" torque="1"/>
+  <xacro:Transmission name="link0_link1" jointName="j1" reduction="1" torque="1"/>
+  <xacro:Transmission name="link1_link2" jointName="j2" reduction="1" torque="1"/>
+  <xacro:Transmission name="link2_link3" jointName="j3" reduction="1" torque="1"/>
+  <xacro:Transmission name="link3_link4" jointName="j4" reduction="1" torque="1"/>
+  <xacro:Transmission name="link4_link5" jointName="j5" reduction="1" torque="1"/>
+  <xacro:Transmission name="link5_link6" jointName="j6" reduction="1" torque="1"/>
+  <xacro:Transmission name="link6_link7" jointName="j7" reduction="1" torque="1"/>
 <!-- PLUGINS -->
-<!--  <include filename="$(find iri_wam_gazebo)/urdf/iri_wam.gazebo.xacro" /> -->
+<include filename="$(find iri_wam_gazebo)/urdf/iri_wam.gazebo.xacro" />
 </robot>

File: iri_wam_description/xacro/wam_sim.urdf.xacro (robot description, xacro)
@@ -86,6 +86,4 @@
   <xacro:Transmission name="link6_link7" jointName="j7" reduction="1" torque="1"/>
   <!-- PLUGINS -->
-<!--
   <include filename="$(find iri_wam_gazebo)/urdf/iri_wam.gazebo.xacro" />
--->
 </robot>

Commit message: updating to previous working files

File: iri_wam_description/urdf/wam.urdf (robot description, URDF)
Before this commit: robot iri_wam, 9 links, 8 joints
Links:
- link wam_fk/wam0: mass 1 -> 0.1; geometry 
Joints:
- joint j1: origin xyz=0 0 0 rpy=-1.57  0 0 -> xyz=0.22 0.14 0.346 rpy=-1.5708 0 0
- joint j2: origin xyz=0 0 0 rpy=1.57 0 0 -> xyz=0 0 0 rpy=1.5708 0 0
- joint j3: origin xyz=0.045 0 0.55 rpy=-1.57 0 0 -> xyz=0.045 0 0.55 rpy=-1.5708 0 0
- joint j4: origin xyz=-0.045 0 0 rpy=1.57 0 0 -> xyz=-0.045 0 0 rpy=1.5708 0 0
- joint j5: origin xyz=0 0 0.3 rpy=-1.57 0 0 -> xyz=0 0 0.3 rpy=-1.5708 0 0
- joint j6: origin xyz=0 0 0 rpy=1.57 0 0 -> xyz=0 0 0 rpy=1.5708 0 0

Commit message: removing unnecessary files

File: iri_wam_description/urdf/wam.urdf (robot description, URDF)
Before this commit: robot iri_wam, 9 links, 8 joints
Links:
- removed link wam_fk/wam0
- added link world
- link wam_fk/wam1: mass 0.1 -> 8.3936; geometry collision mesh filename=package://iri_wam_description/mesh/wam1.stl scale=1.0 1.0 1.0; visual mesh filename=package://iri_wam_description/mesh/wam1.stl scale=1.0 1.0 1.0
- link wam_fk/wam2: mass 0.1 -> 4.8487; geometry collision mesh filename=package://iri_wam_description/mesh/wam2.stl scale=1.0 1.0 1.0; visual mesh filename=package://iri_wam_description/mesh/wam2.stl scale=1.0 1.0 1.0
- link wam_fk/wam3: mass 0.1 -> 1.7251; geometry collision mesh filename=package://iri_wam_description/mesh/wam3.stl scale=1.0 1.0 1.0; visual mesh filename=package://iri_wam_description/mesh/wam3.stl scale=1.0 1.0 1.0
- link wam_fk/wam4: mass 0.1 -> 2.0824; geometry collision mesh filename=package://iri_wam_description/mesh/wam4.stl scale=1.0 1.0 1.0; visual mesh filename=package://iri_wam_description/mesh/wam4.stl scale=1.0 1.0 1.0
- link wam_fk/wam5: mass 0.1 -> 0.3067; geometry collision mesh filename=package://iri_wam_description/mesh/wam5.stl scale=1.0 1.0 1.0; visual mesh filename=package://iri_wam_description/mesh/wam5.stl scale=1.0 1.0 1.0
- link wam_fk/wam6: mass 0.1 -> 0.4278; geometry collision mesh filename=package://iri_wam_description/mesh/wam6.stl scale=1.0 1.0 1.0; visual mesh filename=package://iri_wam_description/mesh/wam6.stl scale=1.0 1.0 1.0
- link wam_fk/wam7: mass 0.1 -> 0.0557; geometry collision mesh filename=package://iri_wam_description/mesh/wam7.stl scale=1.0 1.0 1.0; visual mesh filename=package://iri_wam_description/mesh/wam7.stl scale=1.0 1.0 1.0
- link wambase: mass 1 -> 20; geometry collision mesh filename=package://iri_wam_description/mesh/wambase.stl scale=1.0 1.0 1.0; visual mesh filename=package://iri_wam_description/mesh/wambase.stl scale=1.0 1.0 1.0
Joints:
- removed joint j0
- removed joint j1
- removed joint j2
- removed joint j3
- removed joint j4
- removed joint j5
- removed joint j6
- removed joint j7
- added joint base_fix: type fixed, parent world, child wambase
- added joint j1_joint: type revolute, parent wambase, child wam_fk/wam1, origin xyz=0.22 0.14 0.346 rpy=0 0 0, axis 0 0 1, limit lower=-2.6 upper=2.6 effort=30 velocity=2.0
- added joint j2_joint: type revolute, parent wam_fk/wam1, child wam_fk/wam2, origin xyz=0.0 0.0 0.0 rpy=0 0 0, axis 0 1 0, limit lower=-2.0 upper=2.0 effort=30 velocity=2.0
- added joint j3_joint: type revolute, parent wam_fk/wam2, child wam_fk/wam3, origin xyz=0.0 0.0 0.0 rpy=0 0 0, axis 0 0 1, limit lower=-2.8 upper=2.8 effort=30 velocity=2.0
- added joint j4_joint: type revolute, parent wam_fk/wam3, child wam_fk/wam4, origin xyz=0.045 0.0 0.55 rpy=-1.57079632679 0 0, axis 0 0 1, limit lower=-0.9 upper=2.8 effort=35 velocity=2.0
- added joint j5_joint: type revolute, parent wam_fk/wam4, child wam_fk/wam5, origin xyz=-0.045 -0.3 0.0 rpy=1.57079632679 0 0, axis 0 0 1, limit lower=-4.8 upper=1.3 effort=30 velocity=2.0
- added joint j6_joint: type revolute, parent wam_fk/wam5, child wam_fk/wam6, origin xyz=0.0 0.0 0.0 rpy=-1.57079632679 0 0, axis 0 0 1, limit lower=-1.6 upper=1.6 effort=30 velocity=2.0
- added joint j7_joint: type revolute, parent wam_fk/wam6, child wam_fk/wam7, origin xyz=0.0 0.0 0.0 rpy=1.57079632679 0 0, axis 0 0 1, limit lower=-2.2 upper=2.2 effort=30 velocity=2.0
