Commit message: cambiando nombres, de wam_fk/wam a lk_wam

File: iri_wam_description/urdf/wam.urdf (robot description, URDF)
Before this commit: robot iri_wam, 9 links, 8 joints
Links:
- removed link wam_fk/wam1
- removed link wam_fk/wam2
- removed link wam_fk/wam3
- removed link wam_fk/wam4
- removed link wam_fk/wam5
- removed link wam_fk/wam6
- removed link wam_fk/wam7
- added link lk_wam1, mass 8.3936; collision mesh filename=package://iri_wam_description/mesh/wam1.stl scale=1.0 1.0 1.0; visual mesh filename=package://iri_wam_description/mesh/wam1.stl scale=1.0 1.0 1.0
- added link lk_wam2, mass 4.8487; collision mesh filename=package://iri_wam_description/mesh/wam2.stl scale=1.0 1.0 1.0; visual mesh filename=package://iri_wam_description/mesh/wam2.stl scale=1.0 1.0 1.0
- added link lk_wam3, mass 1.7251; collision mesh filename=package://iri_wam_description/mesh/wam3.stl scale=1.0 1.0 1.0; visual mesh filename=package://iri_wam_description/mesh/wam3.stl scale=1.0 1.0 1.0
- added link lk_wam4, mass 2.0824; collision mesh filename=package://iri_wam_description/mesh/wam4.stl scale=1.0 1.0 1.0; visual mesh filename=package://iri_wam_description/mesh/wam4.stl scale=1.0 1.0 1.0
- added link lk_wam5, mass 0.3067; collision mesh filename=package://iri_wam_description/mesh/wam5.stl scale=1.0 1.0 1.0; visual mesh filename=package://iri_wam_description/mesh/wam5.stl scale=1.0 1.0 1.0
- added link lk_wam6, mass 0.4278; collision mesh filename=package://iri_wam_description/mesh/wam6.stl scale=1.0 1.0 1.0; visual mesh filename=package://iri_wam_description/mesh/wam6.stl scale=1.0 1.0 1.0
- added link lk_wam7, mass 0.0557; collision mesh filename=package://iri_wam_description/mesh/wam7.stl scale=1.0 1.0 1.0; visual mesh filename=package://iri_wam_description/mesh/wam7.stl scale=1.0 1.0 1.0
Joints:
- joint j1_joint: child wam_fk/wam1 -> lk_wam1
- joint j2_joint: child wam_fk/wam2 -> lk_wam2; parent wam_fk/wam1 -> lk_wam1
- joint j3_joint: child wam_fk/wam3 -> lk_wam3; parent wam_fk/wam2 -> lk_wam2
- joint j4_joint: child wam_fk/wam4 -> lk_wam4; parent wam_fk/wam3 -> lk_wam3
- joint j5_joint: child wam_fk/wam5 -> lk_wam5; parent wam_fk/wam4 -> lk_wam4
- joint j6_joint: child wam_fk/wam6 -> lk_wam6; parent wam_fk/wam5 -> lk_wam5
- joint j7_joint: child wam_fk/wam7 -> lk_wam7; parent wam_fk/wam6 -> lk_wam6

File: iri_wam_description/xacro/wam.urdf.xacro (robot description, xacro)
@@ -23,19 +23,19 @@
   <xacro:wam0>
   </xacro:wam0>
-  <xacro:wam1 parent="wam_fk/wam0">
+  <xacro:wam1 parent="lk_wam0">
   </xacro:wam1>
-  <xacro:wam2 parent="wam_fk/wam1">
+  <xacro:wam2 parent="lk_wam1">
   </xacro:wam2>
-  <xacro:wam3 parent="wam_fk/wam2">
+  <xacro:wam3 parent="lk_wam2">
   </xacro:wam3>
-  <xacro:wam4 parent="wam_fk/wam3">
+  <xacro:wam4 parent="lk_wam3">
   </xacro:wam4>
-  <xacro:wam5 parent="wam_fk/wam4">
+  <xacro:wam5 parent="lk_wam4">
   </xacro:wam5>
-  <xacro:wam6 parent="wam_fk/wam5">
+  <xacro:wam6 parent="lk_wam5">
   </xacro:wam6>
-  <xacro:wam7 parent="wam_fk/wam6">
+  <xacro:wam7 parent="lk_wam6">
   </xacro:wam7>
-  <xacro:wamtcp parent="wam_fk/wam7">
+  <xacro:wamtcp parent="lk_wam7">
   </xacro:wamtcp>
 </robot>

File: iri_wam_description/xacro/wam0.urdf.xacro (robot description, xacro)
@@ -3,5 +3,5 @@
   <xacro:macro name="wam0">
     <link name="world"/>
-    <link name="wam_fk/wam0">
+    <link name="lk_wam0">
         <inertial>
             <mass value="20" />
@@ -11,5 +11,5 @@
         <visual>
             <origin xyz="0.0 0.0 0.0" rpy="0 0 0" />
-            <geometry name="wam_fk/wam0_visual">
+            <geometry name="lk_wam0_visual">
                 <mesh filename="package://iri_wam_description/mesh/wambase.stl" scale="1.0 1.0 1.0" />
             </geometry>
@@ -20,5 +20,5 @@
         <collision>
             <origin xyz="0.0 0.0 0.0" rpy="0 0 0"/>
-            <geometry name="wam_fk/wam0_collision">
+            <geometry name="lk_wam0_collision">
                 <mesh filename="package://iri_wam_description/mesh/wambase.stl" scale="1.0 1.0 1.0" />
 <!--
@@ -29,5 +29,5 @@
         </collision>
     </link>
-    <gazebo reference="wam_fk/wam0">
+    <gazebo reference="lk_wam0">
         <material>Gazebo/Grey</material>
         <selfCollide>true</selfCollide>
@@ -35,5 +35,5 @@
     <joint name="wam0_fix" type="fixed">
         <parent link="world"/>
-        <child link="wam_fk/wam0"/>
+        <child link="lk_wam0"/>
         <origin xyz="0.22 0.14 0.346" rpy="0 0 0" />
      </joint>

File: iri_wam_description/xacro/wam1.urdf.xacro (robot description, xacro)
@@ -2,5 +2,5 @@
 <robot xmlns:xacro="http://www.ros.org/wiki/xacro">
   <xacro:macro name="wam1" params="parent">
-    <link name="wam_fk/wam1">
+    <link name="lk_wam1">
         <inertial>
             <mass value="8.3936" />
@@ -10,5 +10,5 @@
         <visual>
             <origin xyz="0.0 0.0 0.0" rpy="0 0 0" />
-            <geometry name="wam_fk/wam1_visual">
+            <geometry name="lk_wam1_visual">
                 <mesh filename="package://iri_wam_description/mesh/wam1.stl" scale="1.0 1.0 1.0" />
             </geometry>
@@ -19,5 +19,5 @@
         <collision>
             <origin xyz="0.0 0.0 0.0" rpy="0 0 0"/>
-            <geometry name="wam_fk/wam1_collision">
+            <geometry name="lk_wam1_collision">
                 <mesh filename="package://iri_wam_description/mesh/wam1.stl" scale="1.0 1.0 1.0" />
 <!--                <box size="0.20 0.40 0.40"/>
@@ -27,5 +27,5 @@
         </collision>
     </link>
-    <gazebo reference="wam_fk/wam1">
+    <gazebo reference="lk_wam1">
         <material>Gazebo/Grey</material>
         <selfCollide>true</selfCollide>
@@ -33,5 +33,5 @@
     <joint name="j1_joint" type="revolute">
         <parent link="${parent}"/>
-        <child link="wam_fk/wam1"/>
+        <child link="lk_wam1"/>
         <origin xyz="0.0 0.0 0.0" rpy="0 0 0" />
         <axis xyz="0 0 1" />

File: iri_wam_description/xacro/wam2.urdf.xacro (robot description, xacro)
@@ -2,5 +2,5 @@
 <robot xmlns:xacro="http://www.ros.org/wiki/xacro">
   <xacro:macro name="wam2" params="parent">
-    <link name="wam_fk/wam2">
+    <link name="lk_wam2">
         <inertial>
             <origin xyz="0 0 0" rpy="0 0 0" />
@@ -10,5 +10,5 @@
         <visual>
             <origin xyz="0.0 0.0 0.0" rpy="0 0 0" />
-            <geometry name="wam_fk/wam2_visual">
+            <geometry name="lk_wam2_visual">
                 <mesh filename="package://iri_wam_description/mesh/wam2.stl" scale="1.0 1.0 1.0" />
             </geometry>
@@ -19,5 +19,5 @@
         <collision>
             <origin xyz="0.0 0.0 0.0" rpy="0 0 0"/>
-            <geometry name="wam_fk/wam2_collision">
+            <geometry name="lk_wam2_collision">
                 <mesh filename="package://iri_wam_description/mesh/wam2.stl" scale="1.0 1.0 1.0" />
 <!--                <box size="0.10 0.10 0.10"/> -->
@@ -26,5 +26,5 @@
         </collision>
     </link>
-    <gazebo reference="wam_fk/wam2">
+    <gazebo reference="lk_wam2">
         <material>Gazebo/Grey</material>
         <selfCollide>true</selfCollide>
@@ -32,5 +32,5 @@
     <joint name="j2_joint" type="revolute">
         <parent link="${parent}"/>
-        <child link="wam_fk/wam2"/>
+        <child link="lk_wam2"/>
         <origin xyz="0.0 0.0 0.0" rpy="0 0 0" />
         <axis xyz="0 1 0" />

File: iri_wam_description/xacro/wam3.urdf.xacro (robot description, xacro)
@@ -2,5 +2,5 @@
 <robot xmlns:xacro="http://www.ros.org/wiki/xacro">
   <xacro:macro name="wam3" params="parent">
-    <link name="wam_fk/wam3">
+    <link name="lk_wam3">
         <inertial>
             <mass value="1.7251" />
@@ -10,5 +10,5 @@
         <visual>
             <origin xyz="0.0 0.0 0.0" rpy="0 0 0" />
-            <geometry name="wam_fk/wam3_visual">
+            <geometry name="lk_wam3_visual">
                 <mesh filename="package://iri_wam_description/mesh/wam3.stl" scale="1.0 1.0 1.0" />
             </geometry>
@@ -19,5 +19,5 @@
         <collision>
             <origin xyz="0.0 0.0 0.0" rpy="0 0 0"/>
-            <geometry name="wam_fk/wam3_collision">
+            <geometry name="lk_wam3_collision">
                 <mesh filename="package://iri_wam_description/mesh/wam3.stl" scale="1.0 1.0 1.0" />
 <!--                <box size="0.10 0.10 0.10"/> -->
@@ -26,5 +26,5 @@
         </collision>
     </link>
-    <gazebo reference="wam_fk/wam3">
+    <gazebo reference="lk_wam3">
         <material>Gazebo/Grey</material>
         <selfCollide>true</selfCollide>
@@ -32,5 +32,5 @@
     <joint name="j3_joint" type="revolute">
         <parent link="${parent}"/>
-        <child link="wam_fk/wam3"/>
+        <child link="lk_wam3"/>
         <origin xyz="0.0 0.0 0.0" rpy="0 0 0" />
         <axis xyz="0 0 1" />

File: iri_wam_description/xacro/wam4.urdf.xacro (robot description, xacro)
@@ -3,5 +3,5 @@
 <property name="M_PI" value="3.1415926535897931" />
   <xacro:macro name="wam4" params="parent">
-    <link name="wam_fk/wam4">
+    <link name="lk_wam4">
         <inertial>
             <mass value="2.0824" />
@@ -11,5 +11,5 @@
         <visual>
             <origin xyz="0.0 0.0 0.0" rpy="0 0 0" />
-            <geometry name="wam_fk/wam4_visual">
+            <geometry name="lk_wam4_visual">
                 <mesh filename="package://iri_wam_description/mesh/wam4.stl" scale="1.0 1.0 1.0" />
             </geometry>
@@ -20,5 +20,5 @@
         <collision>
             <origin xyz="0.0 0.0 0.0" rpy="0 0 0"/>
-            <geometry name="wam_fk/wam4_collision">
+            <geometry name="lk_wam4_collision">
                 <mesh filename="package://iri_wam_description/mesh/wam4.stl" scale="1.0 1.0 1.0" />
 <!--                <box size="0.10 0.10 0.10"/> -->
@@ -27,5 +27,5 @@
         </collision>
     </link>
-    <gazebo reference="wam_fk/wam4">
+    <gazebo reference="lk_wam4">
         <material>Gazebo/Grey</material>
         <selfCollide>true</selfCollide>
@@ -33,5 +33,5 @@
     <joint name="j4_joint" type="revolute">
         <parent link="${parent}"/>
-        <child link="wam_fk/wam4"/>
+        <child link="lk_wam4"/>
         <origin xyz="0.045 0.0 0.55" rpy="-${M_PI/2} 0 0" />
         <axis xyz="0 0 1" />

File: iri_wam_description/xacro/wam5.urdf.xacro (robot description, xacro)
@@ -3,5 +3,5 @@
 <property name="M_PI" value="3.1415926535897931" />
   <xacro:macro name="wam5" params="parent">
-    <link name="wam_fk/wam5">
+    <link name="lk_wam5">
         <inertial>
             <origin xyz="0 0 0" rpy="0 0 0" />
@@ -11,5 +11,5 @@
         <visual>
             <origin xyz="0.0 0.0 0.0" rpy="0 0 0" />
-            <geometry name="wam_fk/wam5_visual">
+            <geometry name="lk_wam5_visual">
                 <mesh filename="package://iri_wam_description/mesh/wam5.stl" scale="1.0 1.0 1.0" />
             </geometry>
@@ -20,5 +20,5 @@
         <collision>
             <origin xyz="0.0 0.0 0.0" rpy="0 0 0"/>
-            <geometry name="wam_fk/wam5_collision">
+            <geometry name="lk_wam5_collision">
                 <mesh filename="package://iri_wam_description/mesh/wam5.stl" scale="1.0 1.0 1.0" />
 <!--                <box size="0.10 0.10 0.10"/> -->
@@ -27,5 +27,5 @@
         </collision>
     </link>
-    <gazebo reference="wam_fk/wam5">
+    <gazebo reference="lk_wam5">
         <material>Gazebo/Grey</material>
         <selfCollide>true</selfCollide>
@@ -33,5 +33,5 @@
     <joint name="j5_joint" type="revolute">
         <parent link="${parent}"/>
-        <child link="wam_fk/wam5"/>
+        <child link="lk_wam5"/>
         <origin xyz="-0.045 -0.3 0.0" rpy="${M_PI/2} 0 0" />
         <axis xyz="0 0 1" />

File: iri_wam_description/xacro/wam6.urdf.xacro (robot description, xacro)
@@ -3,5 +3,5 @@
 <property name="M_PI" value="3.1415926535897931" />
   <xacro:macro name="wam6" params="parent">
-    <link name="wam_fk/wam6">
+    <link name="lk_wam6">
         <inertial>
             <origin xyz="0 0 0" rpy="0 0 0" />
@@ -11,5 +11,5 @@
         <visual>
             <origin xyz="0.0 0.0 0.0" rpy="0 0 0" />
-            <geometry name="wam_fk/wam6_visual">
+            <geometry name="lk_wam6_visual">
                 <mesh filename="package://iri_wam_description/mesh/wam6.stl" scale="1.0 1.0 1.0" />
             </geometry>
@@ -20,5 +20,5 @@
         <collision>
             <origin xyz="0.0 0.0 0.0" rpy="0 0 0"/>
-            <geometry name="wam_fk/wam6_collision">
+            <geometry name="lk_wam6_collision">
                 <mesh filename="package://iri_wam_description/mesh/wam6.stl" scale="1.0 1.0 1.0" />
 <!--                <box size="0.10 0.10 0.10"/> -->
@@ -27,5 +27,5 @@
         </collision>
     </link>
-    <gazebo reference="wam_fk/wam6">
+    <gazebo reference="lk_wam6">
         <material>Gazebo/Grey</material>
         <selfCollide>true</selfCollide>
@@ -33,5 +33,5 @@
     <joint name="j6_joint" type="revolute">
         <parent link="${parent}"/>
-        <child link="wam_fk/wam6"/>
+        <child link="lk_wam6"/>
         <origin xyz="0.0 0.0 0.0" rpy="-${M_PI/2} 0 0" />
         <axis xyz="0 0 1" />

File: iri_wam_description/xacro/wam7.urdf.xacro (robot description, xacro)
@@ -3,5 +3,5 @@
 <property name="M_PI" value="3.1415926535897931" />
   <xacro:macro name="wam7" params="parent">
-    <link name="wam_fk/wam7">
+    <link name="lk_wam7">
         <inertial>
             <origin xyz="0 0 0" rpy="0 0 0" />
@@ -11,5 +11,5 @@
         <visual>
             <origin xyz="0.0 0.0 0.0" rpy="0 0 0" />
-            <geometry name="wam_fk/wam7_visual">
+            <geometry name="lk_wam7_visual">
                 <mesh filename="package://iri_wam_description/mesh/wam7.stl" scale="1.0 1.0 1.0" />
             </geometry>
@@ -20,5 +20,5 @@
         <collision>
             <origin xyz="0.0 0.0 0.0" rpy="0 0 0"/>
-            <geometry name="wam_fk/wam7_collision">
+            <geometry name="lk_wam7_collision">
                 <mesh filename="package://iri_wam_description/mesh/wam7.stl" scale="1.0 1.0 1.0" />
 <!--                <box size="0.10 0.10 0.10"/> -->
@@ -27,5 +27,5 @@
         </collision>
     </link>
-    <gazebo reference="wam_fk/wam7">
+    <gazebo reference="lk_wam7">
         <material>Gazebo/Grey</material>
         <selfCollide>true</selfCollide>
@@ -33,5 +33,5 @@
     <joint name="j7_joint" type="revolute">
         <parent link="${parent}"/>
-        <child link="wam_fk/wam7"/>
+        <child link="lk_wam7"/>
         <origin xyz="0.0 0.0 0.0" rpy="${M_PI/2} 0 0" />
         <axis xyz="0 0 1" />
