Commit message: cambio de lk_wam a wam_link

File: iri_wam_description/urdf/wam.urdf (robot description, URDF)
Before this commit: robot iri_wam, 9 links, 8 joints
Links:
- removed link lk_wam1
- removed link lk_wam2
- removed link lk_wam3
- removed link lk_wam4
- removed link lk_wam5
- removed link lk_wam6
- removed link lk_wam7
- added link wam_link1, mass 8.3936; collision mesh filename=package://iri_wam_description/mesh/wam1.stl scale=1.0 1.0 1.0; visual mesh filename=package://iri_wam_description/mesh/wam1.stl scale=1.0 1.0 1.0
- added link wam_link2, mass 4.8487; collision mesh filename=package://iri_wam_description/mesh/wam2.stl scale=1.0 1.0 1.0; visual mesh filename=package://iri_wam_description/mesh/wam2.stl scale=1.0 1.0 1.0
- added link wam_link3, mass 1.7251; collision mesh filename=package://iri_wam_description/mesh/wam3.stl scale=1.0 1.0 1.0; visual mesh filename=package://iri_wam_description/mesh/wam3.stl scale=1.0 1.0 1.0
- added link wam_link4, mass 2.0824; collision mesh filename=package://iri_wam_description/mesh/wam4.stl scale=1.0 1.0 1.0; visual mesh filename=package://iri_wam_description/mesh/wam4.stl scale=1.0 1.0 1.0
- added link wam_link5, mass 0.3067; collision mesh filename=package://iri_wam_description/mesh/wam5.stl scale=1.0 1.0 1.0; visual mesh filename=package://iri_wam_description/mesh/wam5.stl scale=1.0 1.0 1.0
- added link wam_link6, mass 0.4278; collision mesh filename=package://iri_wam_description/mesh/wam6.stl scale=1.0 1.0 1.0; visual mesh filename=package://iri_wam_description/mesh/wam6.stl scale=1.0 1.0 1.0
- added link wam_link7, mass 0.0557; collision mesh filename=package://iri_wam_description/mesh/wam7.stl scale=1.0 1.0 1.0; visual mesh filename=package://iri_wam_description/mesh/wam7.stl scale=1.0 1.0 1.0
Joints:
- joint j1_joint: child lk_wam1 -> wam_link1
- joint j2_joint: child lk_wam2 -> wam_link2; parent lk_wam1 -> wam_link1
- joint j3_joint: child lk_wam3 -> wam_link3; parent lk_wam2 -> wam_link2
- joint j4_joint: child lk_wam4 -> wam_link4; parent lk_wam3 -> wam_link3
- joint j5_joint: child lk_wam5 -> wam_link5; parent lk_wam4 -> wam_link4
- joint j6_joint: child lk_wam6 -> wam_link6; parent lk_wam5 -> wam_link5
- joint j7_joint: child lk_wam7 -> wam_link7; parent lk_wam6 -> wam_link6

File: iri_wam_description/xacro/wam.urdf.xacro (robot description, xacro)
@@ -23,19 +23,19 @@
   <xacro:wam0>
   </xacro:wam0>
-  <xacro:wam1 parent="lk_wam0">
+  <xacro:wam1 parent="wam_link0">
   </xacro:wam1>
-  <xacro:wam2 parent="lk_wam1">
+  <xacro:wam2 parent="wam_link1">
   </xacro:wam2>
-  <xacro:wam3 parent="lk_wam2">
+  <xacro:wam3 parent="wam_link2">
   </xacro:wam3>
-  <xacro:wam4 parent="lk_wam3">
+  <xacro:wam4 parent="wam_link3">
   </xacro:wam4>
-  <xacro:wam5 parent="lk_wam4">
+  <xacro:wam5 parent="wam_link4">
   </xacro:wam5>
-  <xacro:wam6 parent="lk_wam5">
+  <xacro:wam6 parent="wam_link5">
   </xacro:wam6>
-  <xacro:wam7 parent="lk_wam6">
+  <xacro:wam7 parent="wam_link6">
   </xacro:wam7>
-  <xacro:wamtcp parent="lk_wam7">
+  <xacro:wamtcp parent="wam_link7">
   </xacro:wamtcp>
 </robot>

File: iri_wam_description/xacro/wam0.urdf.xacro (robot description, xacro)
@@ -3,5 +3,5 @@
   <xacro:macro name="wam0">
     <link name="world"/>
-    <link name="lk_wam0">
+    <link name="wam_link0">
         <inertial>
             <mass value="20" />
@@ -11,5 +11,5 @@
         <visual>
             <origin xyz="0.0 0.0 0.0" rpy="0 0 0" />
-            <geometry name="lk_wam0_visual">
+            <geometry name="wam_link0_visual">
                 <mesh filename="package://iri_wam_description/mesh/wambase.stl" scale="1.0 1.0 1.0" />
             </geometry>
@@ -20,5 +20,5 @@
         <collision>
             <origin xyz="0.0 0.0 0.0" rpy="0 0 0"/>
-            <geometry name="lk_wam0_collision">
+            <geometry name="wam_link0_collision">
                 <mesh filename="package://iri_wam_description/mesh/wambase.stl" scale="1.0 1.0 1.0" />
 <!--
@@ -29,5 +29,5 @@
         </collision>
     </link>
-    <gazebo reference="lk_wam0">
+    <gazebo reference="wam_link0">
         <material>Gazebo/Grey</material>
         <selfCollide>true</selfCollide>
@@ -35,5 +35,5 @@
     <joint name="wam0_fix" type="fixed">
         <parent link="world"/>
-        <child link="lk_wam0"/>
+        <child link="wam_link0"/>
         <origin xyz="0.22 0.14 0.346" rpy="0 0 0" />
      </joint>

File: iri_wam_description/xacro/wam1.urdf.xacro (robot description, xacro)
@@ -2,5 +2,5 @@
 <robot xmlns:xacro="http://www.ros.org/wiki/xacro">
   <xacro:macro name="wam1" params="parent">
-    <link name="lk_wam1">
+    <link name="wam_link1">
         <inertial>
             <mass value="8.3936" />
@@ -10,5 +10,5 @@
         <visual>
             <origin xyz="0.0 0.0 0.0" rpy="0 0 0" />
-            <geometry name="lk_wam1_visual">
+            <geometry name="wam_link1_visual">
                 <mesh filename="package://iri_wam_description/mesh/wam1.stl" scale="1.0 1.0 1.0" />
             </geometry>
@@ -19,5 +19,5 @@
         <collision>
             <origin xyz="0.0 0.0 0.0" rpy="0 0 0"/>
-            <geometry name="lk_wam1_collision">
+            <geometry name="wam_link1_collision">
                 <mesh filename="package://iri_wam_description/mesh/wam1.stl" scale="1.0 1.0 1.0" />
 <!--                <box size="0.20 0.40 0.40"/>
@@ -27,5 +27,5 @@
         </collision>
     </link>
-    <gazebo reference="lk_wam1">
+    <gazebo reference="wam_link1">
         <material>Gazebo/Grey</material>
         <selfCollide>true</selfCollide>
@@ -33,5 +33,5 @@
     <joint name="j1_joint" type="revolute">
         <parent link="${parent}"/>
-        <child link="lk_wam1"/>
+        <child link="wam_link1"/>
         <origin xyz="0.0 0.0 0.0" rpy="0 0 0" />
         <axis xyz="0 0 1" />

File: iri_wam_description/xacro/wam2.urdf.xacro (robot description, xacro)
@@ -2,5 +2,5 @@
 <robot xmlns:xacro="http://www.ros.org/wiki/xacro">
   <xacro:macro name="wam2" params="parent">
-    <link name="lk_wam2">
+    <link name="wam_link2">
         <inertial>
             <origin xyz="0 0 0" rpy="0 0 0" />
@@ -10,5 +10,5 @@
         <visual>
             <origin xyz="0.0 0.0 0.0" rpy="0 0 0" />
-            <geometry name="lk_wam2_visual">
+            <geometry name="wam_link2_visual">
                 <mesh filename="package://iri_wam_description/mesh/wam2.stl" scale="1.0 1.0 1.0" />
             </geometry>
@@ -19,5 +19,5 @@
         <collision>
             <origin xyz="0.0 0.0 0.0" rpy="0 0 0"/>
-            <geometry name="lk_wam2_collision">
+            <geometry name="wam_link2_collision">
                 <mesh filename="package://iri_wam_description/mesh/wam2.stl" scale="1.0 1.0 1.0" />
 <!--                <box size="0.10 0.10 0.10"/> -->
@@ -26,5 +26,5 @@
         </collision>
     </link>
-    <gazebo reference="lk_wam2">
+    <gazebo reference="wam_link2">
         <material>Gazebo/Grey</material>
         <selfCollide>true</selfCollide>
@@ -32,5 +32,5 @@
     <joint name="j2_joint" type="revolute">
         <parent link="${parent}"/>
-        <child link="lk_wam2"/>
+        <child link="wam_link2"/>
         <origin xyz="0.0 0.0 0.0" rpy="0 0 0" />
         <axis xyz="0 1 0" />

File: iri_wam_description/xacro/wam3.urdf.xacro (robot description, xacro)
@@ -2,5 +2,5 @@
 <robot xmlns:xacro="http://www.ros.org/wiki/xacro">
   <xacro:macro name="wam3" params="parent">
-    <link name="lk_wam3">
+    <link name="wam_link3">
         <inertial>
             <mass value="1.7251" />
@@ -10,5 +10,5 @@
         <visual>
             <origin xyz="0.0 0.0 0.0" rpy="0 0 0" />
-            <geometry name="lk_wam3_visual">
+            <geometry name="wam_link3_visual">
                 <mesh filename="package://iri_wam_description/mesh/wam3.stl" scale="1.0 1.0 1.0" />
             </geometry>
@@ -19,5 +19,5 @@
         <collision>
             <origin xyz="0.0 0.0 0.0" rpy="0 0 0"/>
-            <geometry name="lk_wam3_collision">
+            <geometry name="wam_link3_collision">
                 <mesh filename="package://iri_wam_description/mesh/wam3.stl" scale="1.0 1.0 1.0" />
 <!--                <box size="0.10 0.10 0.10"/> -->
@@ -26,5 +26,5 @@
         </collision>
     </link>
-    <gazebo reference="lk_wam3">
+    <gazebo reference="wam_link3">
         <material>Gazebo/Grey</material>
         <selfCollide>true</selfCollide>
@@ -32,5 +32,5 @@
     <joint name="j3_joint" type="revolute">
         <parent link="${parent}"/>
-        <child link="lk_wam3"/>
+        <child link="wam_link3"/>
         <origin xyz="0.0 0.0 0.0" rpy="0 0 0" />
         <axis xyz="0 0 1" />

File: iri_wam_description/xacro/wam4.urdf.xacro (robot description, xacro)
@@ -3,5 +3,5 @@
 <property name="M_PI" value="3.1415926535897931" />
   <xacro:macro name="wam4" params="parent">
-    <link name="lk_wam4">
+    <link name="wam_link4">
         <inertial>
             <mass value="2.0824" />
@@ -11,5 +11,5 @@
         <visual>
             <origin xyz="0.0 0.0 0.0" rpy="0 0 0" />
-            <geometry name="lk_wam4_visual">
+            <geometry name="wam_link4_visual">
                 <mesh filename="package://iri_wam_description/mesh/wam4.stl" scale="1.0 1.0 1.0" />
             </geometry>
@@ -20,5 +20,5 @@
         <collision>
             <origin xyz="0.0 0.0 0.0" rpy="0 0 0"/>
-            <geometry name="lk_wam4_collision">
+            <geometry name="wam_link4_collision">
                 <mesh filename="package://iri_wam_description/mesh/wam4.stl" scale="1.0 1.0 1.0" />
 <!--                <box size="0.10 0.10 0.10"/> -->
@@ -27,5 +27,5 @@
         </collision>
     </link>
-    <gazebo reference="lk_wam4">
+    <gazebo reference="wam_link4">
         <material>Gazebo/Grey</material>
         <selfCollide>true</selfCollide>
@@ -33,5 +33,5 @@
     <joint name="j4_joint" type="revolute">
         <parent link="${parent}"/>
-        <child link="lk_wam4"/>
+        <child link="wam_link4"/>
         <origin xyz="0.045 0.0 0.55" rpy="-${M_PI/2} 0 0" />
         <axis xyz="0 0 1" />

File: iri_wam_description/xacro/wam5.urdf.xacro (robot description, xacro)
@@ -3,5 +3,5 @@
 <property name="M_PI" value="3.1415926535897931" />
   <xacro:macro name="wam5" params="parent">
-    <link name="lk_wam5">
+    <link name="wam_link5">
         <inertial>
             <origin xyz="0 0 0" rpy="0 0 0" />
@@ -11,5 +11,5 @@
         <visual>
             <origin xyz="0.0 0.0 0.0" rpy="0 0 0" />
-            <geometry name="lk_wam5_visual">
+            <geometry name="wam_link5_visual">
                 <mesh filename="package://iri_wam_description/mesh/wam5.stl" scale="1.0 1.0 1.0" />
             </geometry>
@@ -20,5 +20,5 @@
         <collision>
             <origin xyz="0.0 0.0 0.0" rpy="0 0 0"/>
-            <geometry name="lk_wam5_collision">
+            <geometry name="wam_link5_collision">
                 <mesh filename="package://iri_wam_description/mesh/wam5.stl" scale="1.0 1.0 1.0" />
 <!--                <box size="0.10 0.10 0.10"/> -->
@@ -27,5 +27,5 @@
         </collision>
     </link>
-    <gazebo reference="lk_wam5">
+    <gazebo reference="wam_link5">
         <material>Gazebo/Grey</material>
         <selfCollide>true</selfCollide>
@@ -33,5 +33,5 @@
     <joint name="j5_joint" type="revolute">
         <parent link="${parent}"/>
-        <child link="lk_wam5"/>
+        <child link="wam_link5"/>
         <origin xyz="-0.045 -0.3 0.0" rpy="${M_PI/2} 0 0" />
         <axis xyz="0 0 1" />

File: iri_wam_description/xacro/wam6.urdf.xacro (robot description, xacro)
@@ -3,5 +3,5 @@
 <property name="M_PI" value="3.1415926535897931" />
   <xacro:macro name="wam6" params="parent">
-    <link name="lk_wam6">
+    <link name="wam_link6">
         <inertial>
             <origin xyz="0 0 0" rpy="0 0 0" />
@@ -11,5 +11,5 @@
         <visual>
             <origin xyz="0.0 0.0 0.0" rpy="0 0 0" />
-            <geometry name="lk_wam6_visual">
+            <geometry name="wam_link6_visual">
                 <mesh filename="package://iri_wam_description/mesh/wam6.stl" scale="1.0 1.0 1.0" />
             </geometry>
@@ -20,5 +20,5 @@
         <collision>
             <origin xyz="0.0 0.0 0.0" rpy="0 0 0"/>
-            <geometry name="lk_wam6_collision">
+            <geometry name="wam_link6_collision">
                 <mesh filename="package://iri_wam_description/mesh/wam6.stl" scale="1.0 1.0 1.0" />
 <!--                <box size="0.10 0.10 0.10"/> -->
@@ -27,5 +27,5 @@
         </collision>
     </link>
-    <gazebo reference="lk_wam6">
+    <gazebo reference="wam_link6">
         <material>Gazebo/Grey</material>
         <selfCollide>true</selfCollide>
@@ -33,5 +33,5 @@
     <joint name="j6_joint" type="revolute">
         <parent link="${parent}"/>
-        <child link="lk_wam6"/>
+        <child link="wam_link6"/>
         <origin xyz="0.0 0.0 0.0" rpy="-${M_PI/2} 0 0" />
         <axis xyz="0 0 1" />

File: iri_wam_description/xacro/wam7.urdf.xacro (robot description, xacro)
@@ -3,5 +3,5 @@
 <property name="M_PI" value="3.1415926535897931" />
   <xacro:macro name="wam7" params="parent">
-    <link name="lk_wam7">
+    <link name="wam_link7">
         <inertial>
             <origin xyz="0 0 0" rpy="0 0 0" />
@@ -11,5 +11,5 @@
         <visual>
             <origin xyz="0.0 0.0 0.0" rpy="0 0 0" />
-            <geometry name="lk_wam7_visual">
+            <geometry name="wam_link7_visual">
                 <mesh filename="package://iri_wam_description/mesh/wam7.stl" scale="1.0 1.0 1.0" />
             </geometry>
@@ -20,5 +20,5 @@
         <collision>
             <origin xyz="0.0 0.0 0.0" rpy="0 0 0"/>
-            <geometry name="lk_wam7_collision">
+            <geometry name="wam_link7_collision">
                 <mesh filename="package://iri_wam_description/mesh/wam7.stl" scale="1.0 1.0 1.0" />
 <!--                <box size="0.10 0.10 0.10"/> -->
@@ -27,5 +27,5 @@
         </collision>
     </link>
-    <gazebo reference="lk_wam7">
+    <gazebo reference="wam_link7">
         <material>Gazebo/Grey</material>
         <selfCollide>true</selfCollide>
@@ -33,5 +33,5 @@
     <joint name="j7_joint" type="revolute">
         <parent link="${parent}"/>
-        <child link="lk_wam7"/>
+        <child link="wam_link7"/>
         <origin xyz="0.0 0.0 0.0" rpy="${M_PI/2} 0 0" />
         <axis xyz="0 0 1" />
