Commit message: gazebo feature added

File: iri_wam_description/xacro/wam.urdf.xacro (robot description, xacro)
@@ -29,7 +29,7 @@
 <xacro:macro name="Visual" params="name xyz rpy">
     <visual>
-      <origin xyz="${xyz}" rpy="${rpy}" />
-      <xacro:geometry_default name="${name}"/>
-      <xacro:material_default name="${name}"/>
+       <origin xyz="${xyz}" rpy="${rpy}" />
+       <xacro:geometry_default name="${name}"/>
+       <xacro:material_default name="${name}"/>
     </visual>
 </xacro:macro>
@@ -59,22 +59,29 @@
 <!-- LINKS   -->
   <xacro:Link name="wambase" xyz="0 0 0" rpy="0 0 0" mass="1" prefix=""/>
-  <link name="wam_fk/wam0"/>
+  <link name="wam_fk/wam0">
+  	<inertial>
+	   <origin xyz="0 0 0" rpy="0 0 0" />
+       <mass value="1"/>
+       <inertia ixx="100"  ixy="0"  ixz="0" iyy="100" iyz="0" izz="100" />
+	</inertial>
+  </link>
   <xacro:Link name="wam1" xyz="0 0 0" rpy="${pi} 0 0" mass="1" prefix="wam_fk/"/>
   <xacro:Link name="wam2" xyz="0 0 0" rpy="-${pi} 0 0" mass="1" prefix="wam_fk/"/>
-  <xacro:Link name="wam3" xyz="-0.045 0.55 0" rpy="${pi}0 0 0" mass="1" prefix="wam_fk/"/>
-  <xacro:Link name="wam4" xyz="0.045 0 0" rpy="-${pi}0 0 0" mass="1" prefix="wam_fk/"/>
+  <xacro:Link name="wam3" xyz="-0.045 0.55 0" rpy="${pi} 0 0" mass="1" prefix="wam_fk/"/>
+  <xacro:Link name="wam4" xyz="0.045 0 0" rpy="-${pi} 0 0" mass="1" prefix="wam_fk/"/>
   <xacro:Link name="wam5" xyz="0 0.3 0" rpy="${pi} 0 0" mass="1" prefix="wam_fk/"/>
   <xacro:Link name="wam6" xyz="0 0 0" rpy="-${pi} 0 0" mass="1" prefix="wam_fk/"/>
   <xacro:Link name="wam7" xyz="0 0 -0.06" rpy="0 0 0" mass="1" prefix="wam_fk/"/>
 <!-- JOINTS  -->
-  <xacro:Joint name="j0" type="fixed" xyz="0 0 0" rpy="0 0 0" upperLim="2.6" lowerLim="-2.6" effort="30" velocity="2" axis="1 0 0" parent="wambase" child="wam_fk/wam0" />
-  <xacro:Joint name="j1" type="revolute" xyz="0 0 0" rpy="0 0 0" upperLim="2.6" lowerLim="-2.6" effort="30" velocity="2" axis="1 0 0" parent="wam_fk/wam0" child="wam_fk/wam1" />
-  <xacro:Joint name="j2" type="revolute" xyz="0 0 0" rpy="0 0 0" upperLim="2.0" lowerLim="-2.0" effort="30" velocity="2" axis="1 0 0" parent="wam_fk/wam1" child="wam_fk/wam2" />
-  <xacro:Joint name="j3" type="revolute" xyz="0 0 0" rpy="0 0 0" upperLim="2.8" lowerLim="-2.8" effort="30" velocity="2" axis="1 0 0" parent="wam_fk/wam2" child="wam_fk/wam3" />
-  <xacro:Joint name="j4" type="revolute" xyz="0 0 0" rpy="0 0 0" upperLim="2.8" lowerLim="-2.8" effort="30" velocity="2" axis="1 0 0" parent="wam_fk/wam3" child="wam_fk/wam4" />
-  <xacro:Joint name="j5" type="revolute" xyz="0 0 0" rpy="0 0 0" upperLim="2.8" lowerLim="-2.8" effort="30" velocity="2" axis="1 0 0" parent="wam_fk/wam4" child="wam_fk/wam5" />
-  <xacro:Joint name="j6" type="revolute" xyz="0 0 0" rpy="0 0 0" upperLim="2.8" lowerLim="-2.8" effort="30" velocity="2" axis="1 0 0" parent="wam_fk/wam5" child="wam_fk/wam6" />
-  <xacro:Joint name="j7" type="revolute" xyz="0 0 0" rpy="0 0 0" upperLim="2.8" lowerLim="-2.8" effort="30" velocity="2" axis="1 0 0" parent="wam_fk/wam6" child="wam_fk/wam7" />
-<!-- Transmission -->
+  <xacro:Joint name="j0" type="fixed"    xyz="0.22 0.14 0.346" rpy="0 0 0" upperLim="2.6" lowerLim="-2.6" effort="30" velocity="2" axis="1 0 0" parent="wambase" child="wam_fk/wam0" />
+  <xacro:Joint name="j1" type="revolute" xyz="0 0 0" rpy="-${pi} 0 0" upperLim="2.6" lowerLim="-2.6" effort="30" velocity="2" axis="1 0 0" parent="wam_fk/wam0" child="wam_fk/wam1" />
+  <xacro:Joint name="j2" type="revolute" xyz="0 0 0" rpy="${pi} 0 0" upperLim="2.0" lowerLim="-2.0" effort="30" velocity="2" axis="1 0 0" parent="wam_fk/wam1" child="wam_fk/wam2" />
+  <xacro:Joint name="j3" type="revolute" xyz="0.045 0 0.55" rpy="-${pi} 0 0" upperLim="2.8" lowerLim="-2.8" effort="30" velocity="2" axis="1 0 0" parent="wam_fk/wam2" child="wam_fk/wam3" />
+  <xacro:Joint name="j4" type="revolute" xyz="-0.045 0 0" rpy="${pi} 0 0" upperLim="2.8" lowerLim="-2.8" effort="30" velocity="2" axis="1 0 0" parent="wam_fk/wam3" child="wam_fk/wam4" />
+  <xacro:Joint name="j5" type="revolute" xyz="0 0 0.3" rpy="-${pi} 0 0" upperLim="2.8" lowerLim="-2.8" effort="30" velocity="2" axis="1 0 0" parent="wam_fk/wam4" child="wam_fk/wam5" />
+  <xacro:Joint name="j6" type="revolute" xyz="0 0 0" rpy="${pi} 0 0" upperLim="2.8" lowerLim="-2.8" effort="30" velocity="2" axis="1 0 0" parent="wam_fk/wam5" child="wam_fk/wam6" />
+  <xacro:Joint name="j7" type="revolute" xyz="0 0 0.06" rpy="0 0 0" upperLim="2.8" lowerLim="-2.8" effort="30" velocity="2" axis="1 0 0" parent="wam_fk/wam6" child="wam_fk/wam7" />
+  <!-- Transmission -->
+  <xacro:Transmission name="linkb_link0" jointName="j0" reduction="1" torque="1"/>
   <xacro:Transmission name="link0_link1" jointName="j1" reduction="1" torque="1"/>
   <xacro:Transmission name="link1_link2" jointName="j2" reduction="1" torque="1"/>
@@ -85,6 +92,4 @@
   <xacro:Transmission name="link6_link7" jointName="j7" reduction="1" torque="1"/>
 <!-- PLUGINS -->
-<!--
   <include filename="$(find iri_wam_gazebo)/urdf/iri_wam.gazebo.xacro" />
--->
 </robot>

Commit message: tests for checking wam description on gazebo and rviz

File: iri_wam_description/xacro/wam.urdf.xacro (robot description, xacro)
@@ -76,5 +76,5 @@
     </visual>
 -->
-    <collision>
+<!--    <collision>
       <origin rpy="0 0 0" xyz="0 0 0"/>
       <geometry name="wam0-geom">
@@ -83,7 +83,9 @@
       <contact_coefficients kd="1.0" kp="1000.0" mu="0"/>
     </collision>
+-->
   </link>
-  <xacro:Link name="wam1" xyz="0 0 0" rpy="${pi/2} 0 0" mass="0.1" prefix="wam_fk/"/>
-  <xacro:Link name="wam2" xyz="0 0 0" rpy="-${pi/2} 0 0" mass="0.1" prefix="wam_fk/"/>
+  <xacro:Link name="wam1" xyz="0 0 0" rpy="0 0 0" mass="0.1" prefix="wam_fk/"/>
+  <xacro:Link name="wam2" xyz="0 0 0" rpy="0 0 0" mass="0.1" prefix="wam_fk/"/>
+<!--
   <xacro:Link name="wam3" xyz="-0.045 0.55 0" rpy="${pi/2} 0 0" mass="0.1" prefix="wam_fk/"/>
   <xacro:Link name="wam4" xyz="0.045 0 0" rpy="-${pi/2} 0 0" mass="0.1" prefix="wam_fk/"/>
@@ -91,17 +93,21 @@
   <xacro:Link name="wam6" xyz="0 0 0" rpy="-${pi/2} 0 0" mass="0.1" prefix="wam_fk/"/>
   <xacro:Link name="wam7" xyz="0 0 -0.06" rpy="0 0 0" mass="0.1" prefix="wam_fk/"/>
+-->
 <!-- JOINTS  -->
-  <xacro:Joint name="j0" type="revolute" xyz="0.22 0.14 0.346" rpy="0 0 0" upperLim="2.6" lowerLim="-2.6" effort="30" velocity="2" axis="0 0 1" parent="wambase" child="wam_fk/wam0" />
-  <xacro:Joint name="j1" type="revolute" xyz="0 0 0" rpy="-${pi/2} 0 0" upperLim="2.6" lowerLim="-2.6" effort="30" velocity="2" axis="0 1 0" parent="wam_fk/wam0" child="wam_fk/wam1" />
-  <xacro:Joint name="j2" type="revolute" xyz="0 0 0" rpy="${pi/2} 0 0" upperLim="2.0" lowerLim="-2.0" effort="30" velocity="2" axis="0 1 0" parent="wam_fk/wam1" child="wam_fk/wam2" />
-  <xacro:Joint name="j3" type="revolute" xyz="0.045 0 0.55" rpy="-${pi/2} 0 0" upperLim="2.8" lowerLim="-2.8" effort="30" velocity="2" axis="0 0 1" parent="wam_fk/wam2" child="wam_fk/wam3" />
-  <xacro:Joint name="j4" type="revolute" xyz="-0.045 0 0" rpy="${pi/2} 0 0" upperLim="2.8" lowerLim="-2.8" effort="30" velocity="2" axis="0 0 1" parent="wam_fk/wam3" child="wam_fk/wam4" />
-  <xacro:Joint name="j5" type="revolute" xyz="0 0 0.3" rpy="-${pi/2} 0 0" upperLim="2.8" lowerLim="-2.8" effort="30" velocity="2" axis="0 0 1" parent="wam_fk/wam4" child="wam_fk/wam5" />
-  <xacro:Joint name="j6" type="revolute" xyz="0 0 0" rpy="${pi/2} 0 0" upperLim="2.8" lowerLim="-2.8" effort="30" velocity="2" axis="0 0 1" parent="wam_fk/wam5" child="wam_fk/wam6" />
-  <xacro:Joint name="j7" type="revolute" xyz="0 0 0.06" rpy="0 0 0" upperLim="2.8" lowerLim="-2.8" effort="30" velocity="2" axis="0 0 1" parent="wam_fk/wam6" child="wam_fk/wam7" />
+  <xacro:Joint name="j0" type="fixed" xyz="0 0 0" rpy="0 0 0" upperLim="0.0" lowerLim="0.0" effort="0.0" velocity="0.0" axis="0 0 0" parent="wambase" child="wam_fk/wam0" />
+  <xacro:Joint name="j1" type="revolute" xyz="0 0 0" rpy="-${pi/2}0 0 0" upperLim="+2.6" lowerLim="-2.6" effort="30" velocity="2" axis="0 -1 0" parent="wam_fk/wam0" child="wam_fk/wam1" />
+  <xacro:Joint name="j2" type="revolute" xyz="0 0 0" rpy="${pi/2}0 0 0" upperLim="+2.0" lowerLim="-2.0" effort="30" velocity="2" axis="0 1 0" parent="wam_fk/wam1" child="wam_fk/wam2" />
+<!--
+  <xacro:Joint name="j3" type="revolute" xyz="0.045 0 0.55" rpy="-${pi/2} 0 0" upperLim="+2.8" lowerLim="-2.8" effort="30" velocity="2" axis="0 -1 0" parent="wam_fk/wam2" child="wam_fk/wam3" />
+  <xacro:Joint name="j4" type="revolute" xyz="-0.045 0 0" rpy="${pi/2} 0 0" upperLim="+3.1" lowerLim="-0.9" effort="30" velocity="2" axis="0 0 1" parent="wam_fk/wam3" child="wam_fk/wam4" />
+  <xacro:Joint name="j5" type="revolute" xyz="0 0 0.3" rpy="-${pi/2} 0 0" upperLim="+1.3" lowerLim="-4.8" effort="30" velocity="2" axis="0 0 1" parent="wam_fk/wam4" child="wam_fk/wam5" />
+  <xacro:Joint name="j6" type="revolute" xyz="0 0 0" rpy="${pi/2} 0 0" upperLim="+1.6" lowerLim="-1.6" effort="30" velocity="2" axis="0 0 1" parent="wam_fk/wam5" child="wam_fk/wam6" />
+  <xacro:Joint name="j7" type="revolute" xyz="0 0 0.06" rpy="0 0 0" upperLim="+2.2" lowerLim="-2.2" effort="30" velocity="2" axis="0 0 1" parent="wam_fk/wam6" child="wam_fk/wam7" />
+-->
   <!-- Transmission -->
   <xacro:Transmission name="linkb_link0" jointName="j0" reduction="1" torque="1"/>
   <xacro:Transmission name="link0_link1" jointName="j1" reduction="1" torque="1"/>
   <xacro:Transmission name="link1_link2" jointName="j2" reduction="1" torque="1"/>
+<!--
   <xacro:Transmission name="link2_link3" jointName="j3" reduction="1" torque="1"/>
   <xacro:Transmission name="link3_link4" jointName="j4" reduction="1" torque="1"/>
@@ -109,4 +115,5 @@
   <xacro:Transmission name="link5_link6" jointName="j6" reduction="1" torque="1"/>
   <xacro:Transmission name="link6_link7" jointName="j7" reduction="1" torque="1"/>
+-->
 <!-- PLUGINS -->
 <!--  <include filename="$(find iri_wam_gazebo)/urdf/iri_wam.gazebo.xacro" /> -->

Commit message: wam.urdf.xacro is the one for using with the real robot

File: iri_wam_description/xacro/wam.urdf.xacro (robot description, xacro)
@@ -65,27 +65,7 @@
       <inertia ixx="100" ixy="0" ixz="0" iyy="100" iyz="0" izz="100"/>
     </inertial>
-<!--
-    <visual>
-      <origin rpy="0 0 0" xyz="0 0 0"/>
-      <geometry name="wam0-geom">
-        <mesh filename="package://iri_wam_description/mesh/wam0.stl"/>
-      </geometry>
-      <material name="wam0-mat">
-        <color rgba="0.75 0.75 0.75 1.0"/>
-      </material>
-    </visual>
--->
-<!--    <collision>
-      <origin rpy="0 0 0" xyz="0 0 0"/>
-      <geometry name="wam0-geom">
-        <mesh filename="package://iri_wam_description/mesh/wam0.stl"/>
-      </geometry>
-      <contact_coefficients kd="1.0" kp="1000.0" mu="0"/>
-    </collision>
--->
   </link>
-  <xacro:Link name="wam1" xyz="0 0 0" rpy="0 0 0" mass="0.1" prefix="wam_fk/"/>
+  <xacro:Link name="wam1" xyz="0 0 0" rpy="${pi/2} 0 0" mass="0.1" prefix="wam_fk/"/>
   <xacro:Link name="wam2" xyz="0 0 0" rpy="0 0 0" mass="0.1" prefix="wam_fk/"/>
-<!--
   <xacro:Link name="wam3" xyz="-0.045 0.55 0" rpy="${pi/2} 0 0" mass="0.1" prefix="wam_fk/"/>
   <xacro:Link name="wam4" xyz="0.045 0 0" rpy="-${pi/2} 0 0" mass="0.1" prefix="wam_fk/"/>
@@ -93,27 +73,13 @@
   <xacro:Link name="wam6" xyz="0 0 0" rpy="-${pi/2} 0 0" mass="0.1" prefix="wam_fk/"/>
   <xacro:Link name="wam7" xyz="0 0 -0.06" rpy="0 0 0" mass="0.1" prefix="wam_fk/"/>
--->
 <!-- JOINTS  -->
-  <xacro:Joint name="j0" type="fixed" xyz="0 0 0" rpy="0 0 0" upperLim="0.0" lowerLim="0.0" effort="0.0" velocity="0.0" axis="0 0 0" parent="wambase" child="wam_fk/wam0" />
-  <xacro:Joint name="j1" type="revolute" xyz="0 0 0" rpy="-${pi/2}0 0 0" upperLim="+2.6" lowerLim="-2.6" effort="30" velocity="2" axis="0 -1 0" parent="wam_fk/wam0" child="wam_fk/wam1" />
-  <xacro:Joint name="j2" type="revolute" xyz="0 0 0" rpy="${pi/2}0 0 0" upperLim="+2.0" lowerLim="-2.0" effort="30" velocity="2" axis="0 1 0" parent="wam_fk/wam1" child="wam_fk/wam2" />
-<!--
+  <xacro:Joint name="j0" type="fixed" xyz="0.22 0.14 0.346" rpy="0 0 0" upperLim="0.0" lowerLim="0.0" effort="0.0" velocity="0.0" axis="0 0 0" parent="wambase" child="wam_fk/wam0" />
+  <xacro:Joint name="j1" type="revolute" xyz="0.22 0.14 0.346" rpy="-${pi/2} 0 0" upperLim="+2.6" lowerLim="-2.6" effort="30" velocity="2" axis="0 -1 0" parent="wambase" child="wam_fk/wam1" />
+  <xacro:Joint name="j2" type="revolute" xyz="0 0 0" rpy="${pi/2} 0 0" upperLim="+2.0" lowerLim="-2.0" effort="30" velocity="2" axis="0 1 0" parent="wam_fk/wam1" child="wam_fk/wam2" />
   <xacro:Joint name="j3" type="revolute" xyz="0.045 0 0.55" rpy="-${pi/2} 0 0" upperLim="+2.8" lowerLim="-2.8" effort="30" velocity="2" axis="0 -1 0" parent="wam_fk/wam2" child="wam_fk/wam3" />
-  <xacro:Joint name="j4" type="revolute" xyz="-0.045 0 0" rpy="${pi/2} 0 0" upperLim="+3.1" lowerLim="-0.9" effort="30" velocity="2" axis="0 0 1" parent="wam_fk/wam3" child="wam_fk/wam4" />
-  <xacro:Joint name="j5" type="revolute" xyz="0 0 0.3" rpy="-${pi/2} 0 0" upperLim="+1.3" lowerLim="-4.8" effort="30" velocity="2" axis="0 0 1" parent="wam_fk/wam4" child="wam_fk/wam5" />
-  <xacro:Joint name="j6" type="revolute" xyz="0 0 0" rpy="${pi/2} 0 0" upperLim="+1.6" lowerLim="-1.6" effort="30" velocity="2" axis="0 0 1" parent="wam_fk/wam5" child="wam_fk/wam6" />
+  <xacro:Joint name="j4" type="revolute" xyz="-0.045 0 0" rpy="${pi/2} 0 0" upperLim="+3.1" lowerLim="-0.9" effort="30" velocity="2" axis="0 1 0" parent="wam_fk/wam3" child="wam_fk/wam4" />
+  <xacro:Joint name="j5" type="revolute" xyz="0 0 0.3" rpy="-${pi/2} 0 0" upperLim="+1.3" lowerLim="-4.8" effort="30" velocity="2" axis="0 -1 0" parent="wam_fk/wam4" child="wam_fk/wam5" />
+  <xacro:Joint name="j6" type="revolute" xyz="0 0 0" rpy="${pi/2} 0 0" upperLim="+1.6" lowerLim="-1.6" effort="30" velocity="2" axis="0 1 0" parent="wam_fk/wam5" child="wam_fk/wam6" />
   <xacro:Joint name="j7" type="revolute" xyz="0 0 0.06" rpy="0 0 0" upperLim="+2.2" lowerLim="-2.2" effort="30" velocity="2" axis="0 0 1" parent="wam_fk/wam6" child="wam_fk/wam7" />
--->
-  <!-- Transmission -->
-  <xacro:Transmission name="linkb_link0" jointName="j0" reduction="1" torque="1"/>
-  <xacro:Transmission name="link0_link1" jointName="j1" reduction="1" torque="1"/>
-  <xacro:Transmission name="link1_link2" jointName="j2" reduction="1" torque="1"/>
-<!--
-  <xacro:Transmission name="link2_link3" jointName="j3" reduction="1" torque="1"/>
-  <xacro:Transmission name="link3_link4" jointName="j4" reduction="1" torque="1"/>
-  <xacro:Transmission name="link4_link5" jointName="j5" reduction="1" torque="1"/>
-  <xacro:Transmission name="link5_link6" jointName="j6" reduction="1" torque="1"/>
-  <xacro:Transmission name="link6_link7" jointName="j7" reduction="1" torque="1"/>
--->
 <!-- PLUGINS -->
 <!--  <include filename="$(find iri_wam_gazebo)/urdf/iri_wam.gazebo.xacro" /> -->

Commit message: updating to previous working files

File: iri_wam_description/xacro/wam.urdf.xacro (robot description, xacro)
@@ -65,20 +65,4 @@
       <inertia ixx="100" ixy="0" ixz="0" iyy="100" iyz="0" izz="100"/>
     </inertial>
-	<visual>
-	  <origin xyz="0 0 0" rpy="0 0 0" />
-      <geometry name="wam_fk/wam0-geom">
-        <cylinder radius="0.015" length="0.015" />
-      </geometry>
-      <material name="Cyan">
-        <color rgba="1 0 0 1"/>
-      </material>
-	</visual>
-	<collision>
-	  <origin xyz="0 0 0" rpy="0 0 0" />
-      <geometry name="wam_fk/wam0-geom">
-        <cylinder radius="0.015" length="0.015" />
-      </geometry>
-       <contact_coefficients mu="0" kp="1000.0" kd="1.0"/>
-     </collision>
   </link>
   <xacro:Link name="wam1" xyz="0 0 0" rpy="${pi/2} 0 0" mass="0.1" prefix="wam_fk/"/>
@@ -93,27 +77,10 @@
   <xacro:Joint name="j1" type="revolute" xyz="0.22 0.14 0.346" rpy="-${pi/2} 0 0" upperLim="2.6" lowerLim="-2.6" effort="30" velocity="2" axis="0 -1 0" parent="wambase" child="wam_fk/wam1" />
   <xacro:Joint name="j2" type="revolute" xyz="0 0 0" rpy="${pi/2} 0 0" upperLim="2.0" lowerLim="-2.0" effort="30" velocity="2" axis="0 1 0" parent="wam_fk/wam1" child="wam_fk/wam2" />
-  <xacro:Joint name="j3" type="revolute" xyz="0.045 0 0.55" rpy="-${pi/2} 0 0" upperLim="2.8" lowerLim="-2.8" effort="30" velocity="2" axis="0 0 1" parent="wam_fk/wam2" child="wam_fk/wam3" />
-  <xacro:Joint name="j4" type="revolute" xyz="-0.045 0 0" rpy="${pi/2} 0 0" upperLim="2.8" lowerLim="-2.8" effort="30" velocity="2" axis="0 0 1" parent="wam_fk/wam3" child="wam_fk/wam4" />
-  <xacro:Joint name="j5" type="revolute" xyz="0 0 0.3" rpy="-${pi/2} 0 0" upperLim="2.8" lowerLim="-2.8" effort="30" velocity="2" axis="0 0 1" parent="wam_fk/wam4" child="wam_fk/wam5" />
-  <xacro:Joint name="j6" type="revolute" xyz="0 0 0" rpy="${pi/2} 0 0" upperLim="2.8" lowerLim="-2.8" effort="30" velocity="2" axis="0 0 1" parent="wam_fk/wam5" child="wam_fk/wam6" />
-  <xacro:Joint name="j7" type="revolute" xyz="0 0 0.06" rpy="0 0 0" upperLim="2.8" lowerLim="-2.8" effort="30" velocity="2" axis="0 0 1" parent="wam_fk/wam6" child="wam_fk/wam7" />
-  <xacro:Joint name="j0" type="fixed"    xyz="0.22 0.14 0.346" rpy="0 0 0" upperLim="2.6" lowerLim="-2.6" effort="30" velocity="2" axis="1 0 0" parent="wambase" child="wam_fk/wam0" />
-  <xacro:Joint name="j1" type="revolute" xyz="0 0 0" rpy="-${pi}  0 0" upperLim="2.6" lowerLim="-2.6" effort="30" velocity="2" axis="1 0 0" parent="wam_fk/wam0" child="wam_fk/wam1" />
-  <xacro:Joint name="j2" type="revolute" xyz="0 0 0" rpy="${pi} 0 0" upperLim="2.0" lowerLim="-2.0" effort="30" velocity="2" axis="1 0 0" parent="wam_fk/wam1" child="wam_fk/wam2" />
-  <xacro:Joint name="j3" type="revolute" xyz="0.045 0 0.55" rpy="-${pi} 0 0" upperLim="2.8" lowerLim="-2.8" effort="30" velocity="2" axis="1 0 0" parent="wam_fk/wam2" child="wam_fk/wam3" />
-  <xacro:Joint name="j4" type="revolute" xyz="-0.045 0 0" rpy="${pi} 0 0" upperLim="2.8" lowerLim="-2.8" effort="30" velocity="2" axis="1 0 0" parent="wam_fk/wam3" child="wam_fk/wam4" />
-  <xacro:Joint name="j5" type="revolute" xyz="0 0 0.3" rpy="-${pi} 0 0" upperLim="2.8" lowerLim="-2.8" effort="30" velocity="2" axis="1 0 0" parent="wam_fk/wam4" child="wam_fk/wam5" />
-  <xacro:Joint name="j6" type="revolute" xyz="0 0 0" rpy="${pi} 0 0" upperLim="2.8" lowerLim="-2.8" effort="30" velocity="2" axis="1 0 0" parent="wam_fk/wam5" child="wam_fk/wam6" />
-  <xacro:Joint name="j7" type="revolute" xyz="0 0 0.06" rpy="0 0 0" upperLim="2.8" lowerLim="-2.8" effort="30" velocity="2" axis="1 0 0" parent="wam_fk/wam6" child="wam_fk/wam7" />
-  <!-- Transmission -->
-  <xacro:Transmission name="linkb_link0" jointName="j0" reduction="1" torque="1"/>
-  <xacro:Transmission name="link0_link1" jointName="j1" reduction="1" torque="1"/>
-  <xacro:Transmission name="link1_link2" jointName="j2" reduction="1" torque="1"/>
-  <xacro:Transmission name="link2_link3" jointName="j3" reduction="1" torque="1"/>
-  <xacro:Transmission name="link3_link4" jointName="j4" reduction="1" torque="1"/>
-  <xacro:Transmission name="link4_link5" jointName="j5" reduction="1" torque="1"/>
-  <xacro:Transmission name="link5_link6" jointName="j6" reduction="1" torque="1"/>
-  <xacro:Transmission name="link6_link7" jointName="j7" reduction="1" torque="1"/>
+  <xacro:Joint name="j3" type="revolute" xyz="0.045 0 0.55" rpy="-${pi/2} 0 0" upperLim="2.8" lowerLim="-2.8" effort="30" velocity="2" axis="0 -1 0" parent="wam_fk/wam2" child="wam_fk/wam3" />
+  <xacro:Joint name="j4" type="revolute" xyz="-0.045 0 0" rpy="${pi/2} 0 0" upperLim="3.1" lowerLim="-0.9" effort="30" velocity="2" axis="0 1 0" parent="wam_fk/wam3" child="wam_fk/wam4" />
+  <xacro:Joint name="j5" type="revolute" xyz="0 0 0.3" rpy="-${pi/2} 0 0" upperLim="1.3" lowerLim="-4.8" effort="30" velocity="2" axis="0 -1 0" parent="wam_fk/wam4" child="wam_fk/wam5" />
+  <xacro:Joint name="j6" type="revolute" xyz="0 0 0" rpy="${pi/2} 0 0" upperLim="1.6" lowerLim="-1.6" effort="30" velocity="2" axis="0 1 0" parent="wam_fk/wam5" child="wam_fk/wam6" />
+  <xacro:Joint name="j7" type="revolute" xyz="0 0 0.06" rpy="0 0 0" upperLim="2.2" lowerLim="-2.2" effort="30" velocity="2" axis="0 0 1" parent="wam_fk/wam6" child="wam_fk/wam7" />
 <!-- PLUGINS -->
-<include filename="$(find iri_wam_gazebo)/urdf/iri_wam.gazebo.xacro" />
+<!--  <include filename="$(find iri_wam_gazebo)/urdf/iri_wam.gazebo.xacro" /> -->
 </robot>

File: iri_wam_description/xacro/wam_sim.urdf.xacro (robot description, xacro)
@@ -86,4 +86,6 @@
   <xacro:Transmission name="link6_link7" jointName="j7" reduction="1" torque="1"/>
   <!-- PLUGINS -->
+<!--
   <include filename="$(find iri_wam_gazebo)/urdf/iri_wam.gazebo.xacro" />
+-->
 </robot>
