Commit message: new definition of the wam xacro files

File: iri_wam_description/xacro/wam.urdf.xacro (robot description, xacro)
@@ -5,82 +5,28 @@
        xmlns:xacro="http://ros.org/wiki/xacro"
        name="iri_wam">
-      <!-- Constants -->
- <xacro:property name="pi" value="3.1416" />
-   <!-- Includes -->
-<include filename="$(find iri_wam_description)/xacro/transmission.urdf.xacro" />
-<!-- MACROS -->
-<xacro:macro name="intertial_default" params="mass xyz rpy">
-	<inertial>
-	   <origin xyz="${xyz}" rpy="${rpy}" />
-       <mass value="${mass}"/>
-       <inertia ixx="100"  ixy="0"  ixz="0" iyy="100" iyz="0" izz="100" />
-	</inertial>
-</xacro:macro>
-<xacro:macro name= "geometry_default" params="name">
-    <geometry name="${name}-geom">
-       <mesh filename="package://iri_wam_description/mesh/${name}.stl"/>
-    </geometry>
-</xacro:macro>
-<xacro:macro name= "material_default" params="name">
-    <material name="${name}-mat">
-       <color rgba="0.75 0.75 0.75 1.0"/>
-    </material>
-</xacro:macro>
-<xacro:macro name="Visual" params="name xyz rpy">
-    <visual>
-       <origin xyz="${xyz}" rpy="${rpy}" />
-       <xacro:geometry_default name="${name}"/>
-       <xacro:material_default name="${name}"/>
-    </visual>
-</xacro:macro>
-<xacro:macro name="Collision" params="name xyz rpy">
-    <collision>
-       <origin xyz="${xyz}" rpy="${rpy}" />
-       <xacro:geometry_default name="${name}"/>
-       <contact_coefficients mu="0" kp="1000.0" kd="1.0"/>
-    </collision>
-</xacro:macro>
-<xacro:macro name="Link"  params="name xyz rpy mass prefix">
-  <link name="${prefix}${name}">
-	<xacro:intertial_default mass="${mass}" xyz="${xyz}" rpy="${rpy}" />
-	<xacro:Visual name="${name}" xyz="${xyz}" rpy="${rpy}" />
-	<xacro:Collision name="${name}" xyz="${xyz}" rpy="${rpy}"/>
-  </link>
- </xacro:macro>
-<xacro:macro name="Joint" params="name type xyz rpy upperLim lowerLim effort velocity axis parent child">
-  <joint name="${name}" type="${type}">
-      <parent link="${parent}"/>
-      <child link="${child}"/>
-      <origin xyz="${xyz}" rpy="${rpy}"/>
-      <limit upper="${upperLim}" lower="${lowerLim}" effort="${effort}" velocity="${velocity}" />
-      <axis xyz="${axis}"/>
-  </joint>
-</xacro:macro>
-<!-- LINKS   -->
-  <xacro:Link name="wambase" xyz="0 0 0" rpy="0 0 0" mass="1" prefix=""/>
-  <link name="wam_fk/wam0">
-    <inertial>
-      <origin rpy="0 0 0" xyz="0 0 0"/>
-      <mass value="0.1"/>
-      <inertia ixx="100" ixy="0" ixz="0" iyy="100" iyz="0" izz="100"/>
-    </inertial>
-  </link>
-  <xacro:Link name="wam1" xyz="0 0 0" rpy="${pi/2} 0 0" mass="0.1" prefix="wam_fk/"/>
-  <xacro:Link name="wam2" xyz="0 0 0" rpy="0 0 0" mass="0.1" prefix="wam_fk/"/>
-  <xacro:Link name="wam3" xyz="-0.045 0.55 0" rpy="${pi/2} 0 0" mass="0.1" prefix="wam_fk/"/>
-  <xacro:Link name="wam4" xyz="0.045 0 0" rpy="-${pi/2} 0 0" mass="0.1" prefix="wam_fk/"/>
-  <xacro:Link name="wam5" xyz="0 0 0" rpy="${pi/2} 0 0" mass="0.1" prefix="wam_fk/"/>
-  <xacro:Link name="wam6" xyz="0 0 0" rpy="-${pi/2} 0 0" mass="0.1" prefix="wam_fk/"/>
-  <xacro:Link name="wam7" xyz="0 0 -0.06" rpy="0 0 0" mass="0.1" prefix="wam_fk/"/>
-<!-- JOINTS  -->
-  <xacro:Joint name="j0" type="fixed" xyz="0.22 0.14 0.346" rpy="0 0 0" upperLim="0.0" lowerLim="0.0" effort="0.0" velocity="0.0" axis="0 0 0" parent="wambase" child="wam_fk/wam0" />
-  <xacro:Joint name="j1" type="revolute" xyz="0.22 0.14 0.346" rpy="-${pi/2} 0 0" upperLim="2.6" lowerLim="-2.6" effort="30" velocity="2" axis="0 -1 0" parent="wambase" child="wam_fk/wam1" />
-  <xacro:Joint name="j2" type="revolute" xyz="0 0 0" rpy="${pi/2} 0 0" upperLim="2.0" lowerLim="-2.0" effort="30" velocity="2" axis="0 1 0" parent="wam_fk/wam1" child="wam_fk/wam2" />
-  <xacro:Joint name="j3" type="revolute" xyz="0.045 0 0.55" rpy="-${pi/2} 0 0" upperLim="2.8" lowerLim="-2.8" effort="30" velocity="2" axis="0 -1 0" parent="wam_fk/wam2" child="wam_fk/wam3" />
-  <xacro:Joint name="j4" type="revolute" xyz="-0.045 0 0" rpy="${pi/2} 0 0" upperLim="3.1" lowerLim="-0.9" effort="30" velocity="2" axis="0 1 0" parent="wam_fk/wam3" child="wam_fk/wam4" />
-  <xacro:Joint name="j5" type="revolute" xyz="0 0 0.3" rpy="-${pi/2} 0 0" upperLim="1.3" lowerLim="-4.8" effort="30" velocity="2" axis="0 -1 0" parent="wam_fk/wam4" child="wam_fk/wam5" />
-  <xacro:Joint name="j6" type="revolute" xyz="0 0 0" rpy="${pi/2} 0 0" upperLim="1.6" lowerLim="-1.6" effort="30" velocity="2" axis="0 1 0" parent="wam_fk/wam5" child="wam_fk/wam6" />
-  <xacro:Joint name="j7" type="revolute" xyz="0 0 0.06" rpy="0 0 0" upperLim="2.2" lowerLim="-2.2" effort="30" velocity="2" axis="0 0 1" parent="wam_fk/wam6" child="wam_fk/wam7" />
-<!-- PLUGINS -->
-<!--  <include filename="$(find iri_wam_gazebo)/urdf/iri_wam.gazebo.xacro" /> -->
+  <!-- LINKS   -->
+  <include filename="$(find iri_wam_description)/xacro/wambase.urdf.xacro" />
+  <include filename="$(find iri_wam_description)/xacro/wam1.urdf.xacro" />
+  <include filename="$(find iri_wam_description)/xacro/wam2.urdf.xacro" />
+  <include filename="$(find iri_wam_description)/xacro/wam3.urdf.xacro" />
+  <include filename="$(find iri_wam_description)/xacro/wam4.urdf.xacro" />
+  <include filename="$(find iri_wam_description)/xacro/wam5.urdf.xacro" />
+  <include filename="$(find iri_wam_description)/xacro/wam6.urdf.xacro" />
+  <include filename="$(find iri_wam_description)/xacro/wam7.urdf.xacro" />
+  <xacro:wambase>
+  </xacro:wambase>
+  <xacro:wam1 parent="wambase">
+  </xacro:wam1>
+  <xacro:wam2 parent="wam_fk/wam1">
+  </xacro:wam2>
+  <xacro:wam3 parent="wam_fk/wam2">
+  </xacro:wam3>
+  <xacro:wam4 parent="wam_fk/wam3">
+  </xacro:wam4>
+  <xacro:wam5 parent="wam_fk/wam4">
+  </xacro:wam5>
+  <xacro:wam6 parent="wam_fk/wam5">
+  </xacro:wam6>
+  <xacro:wam7 parent="wam_fk/wam6">
+  </xacro:wam7>
 </robot>

File: iri_wam_description/xacro/wam1.urdf.xacro (robot description, xacro)
@@ -31,5 +31,5 @@
         <selfCollide>true</selfCollide>
     </gazebo>
-    <joint name="j1" type="revolute">
+    <joint name="j1_joint" type="revolute">
         <parent link="${parent}"/>
         <child link="wam_fk/wam1"/>
@@ -40,7 +40,7 @@
         <dynamics damping="100"/>
      </joint>
-    <transmission type="pr2_mechanism_model/SimpleTransmission" name="wam_fk/wam1_transmission">
-      <actuator name="wam_fk/wam1_rotation" />
-      <joint name="j1" />
+    <transmission type="pr2_mechanism_model/SimpleTransmission" name="j1_transmission">
+      <actuator name="j1" />
+      <joint name="j1_joint" />
       <mechanicalReduction>1</mechanicalReduction>
       <motorTorqueConstant>1</motorTorqueConstant>

File: iri_wam_description/xacro/wam2.urdf.xacro (robot description, xacro)
@@ -30,5 +30,5 @@
         <selfCollide>true</selfCollide>
     </gazebo>
-    <joint name="j2" type="revolute">
+    <joint name="j2_joint" type="revolute">
         <parent link="${parent}"/>
         <child link="wam_fk/wam2"/>
@@ -39,7 +39,7 @@
         <dynamics damping="100"/>
     </joint>
-    <transmission type="pr2_mechanism_model/SimpleTransmission" name="wam_fk/wam2_transmission">
-      <actuator name="wam_fk/wam2_rotation" />
-      <joint name="j2" />
+    <transmission type="pr2_mechanism_model/SimpleTransmission" name="j2_transmission">
+      <actuator name="j2" />
+      <joint name="j2_joint" />
       <mechanicalReduction>1</mechanicalReduction>
       <motorTorqueConstant>1</motorTorqueConstant>

File: iri_wam_description/xacro/wam3.urdf.xacro (robot description, xacro)
@@ -30,5 +30,5 @@
         <selfCollide>true</selfCollide>
     </gazebo>
-    <joint name="j3" type="revolute">
+    <joint name="j3_joint" type="revolute">
         <parent link="${parent}"/>
         <child link="wam_fk/wam3"/>
@@ -39,7 +39,7 @@
         <dynamics damping="100"/>
     </joint>
-    <transmission type="pr2_mechanism_model/SimpleTransmission" name="wam_fk/wam3_transmission">
-      <actuator name="wam_fk/wam3_rotation" />
-      <joint name="j3" />
+    <transmission type="pr2_mechanism_model/SimpleTransmission" name="j3_transmission">
+      <actuator name="j3" />
+      <joint name="j3_joint" />
       <mechanicalReduction>1</mechanicalReduction>
       <motorTorqueConstant>1</motorTorqueConstant>

File: iri_wam_description/xacro/wam4.urdf.xacro (robot description, xacro)
@@ -31,5 +31,5 @@
         <selfCollide>true</selfCollide>
     </gazebo>
-    <joint name="j4" type="revolute">
+    <joint name="j4_joint" type="revolute">
         <parent link="${parent}"/>
         <child link="wam_fk/wam4"/>
@@ -40,7 +40,7 @@
   <dynamics damping="100"/>
     </joint>
-    <transmission type="pr2_mechanism_model/SimpleTransmission" name="wam_fk/wam4_transmission">
-      <actuator name="wam_fk/wam4_rotation" />
-      <joint name="j4" />
+    <transmission type="pr2_mechanism_model/SimpleTransmission" name="j4_transmission">
+      <actuator name="j4" />
+      <joint name="j4_joint" />
       <mechanicalReduction>1</mechanicalReduction>
       <motorTorqueConstant>1</motorTorqueConstant>

File: iri_wam_description/xacro/wam5.urdf.xacro (robot description, xacro)
@@ -31,5 +31,5 @@
         <selfCollide>true</selfCollide>
     </gazebo>
-    <joint name="j5" type="revolute">
+    <joint name="j5_joint" type="revolute">
         <parent link="${parent}"/>
         <child link="wam_fk/wam5"/>
@@ -40,7 +40,7 @@
    <dynamics damping="100"/>
     </joint>
-    <transmission type="pr2_mechanism_model/SimpleTransmission" name="wam_fk/wam5_transmission">
-      <actuator name="wam_fk/wam5_rotation" />
-      <joint name="j5" />
+    <transmission type="pr2_mechanism_model/SimpleTransmission" name="j5_transmission">
+      <actuator name="j5" />
+      <joint name="j5_joint" />
       <mechanicalReduction>1</mechanicalReduction>
       <motorTorqueConstant>1</motorTorqueConstant>

File: iri_wam_description/xacro/wam6.urdf.xacro (robot description, xacro)
@@ -31,5 +31,5 @@
         <selfCollide>true</selfCollide>
     </gazebo>
-    <joint name="j6" type="revolute">
+    <joint name="j6_joint" type="revolute">
         <parent link="${parent}"/>
         <child link="wam_fk/wam6"/>
@@ -40,7 +40,7 @@
         <dynamics damping="100"/>
     </joint>
-    <transmission type="pr2_mechanism_model/SimpleTransmission" name="wam_fk/wam6_transmission">
-      <actuator name="wam_fk/wam6_rotation" />
-      <joint name="j6" />
+    <transmission type="pr2_mechanism_model/SimpleTransmission" name="j6_transmission">
+      <actuator name="j6" />
+      <joint name="j6_joint" />
       <mechanicalReduction>1</mechanicalReduction>
       <motorTorqueConstant>1</motorTorqueConstant>

File: iri_wam_description/xacro/wam7.urdf.xacro (robot description, xacro)
@@ -31,5 +31,5 @@
         <selfCollide>true</selfCollide>
     </gazebo>
-    <joint name="j7" type="revolute">
+    <joint name="j7_joint" type="revolute">
         <parent link="${parent}"/>
         <child link="wam_fk/wam7"/>
@@ -40,7 +40,7 @@
       <dynamics damping="100"/>
     </joint>
-    <transmission type="pr2_mechanism_model/SimpleTransmission" name="wam_fk/wam7_transmission">
-      <actuator name="wam_fk/wam7_rotation" />
-      <joint name="j7" />
+    <transmission type="pr2_mechanism_model/SimpleTransmission" name="j7_transmission">
+      <actuator name="j7" />
+      <joint name="j7_joint" />
       <mechanicalReduction>1</mechanicalReduction>
       <motorTorqueConstant>1</motorTorqueConstant>

Commit message: wambase link substitution to wam_fk/wam0

File: iri_wam_description/xacro/wam.urdf.xacro (robot description, xacro)
@@ -6,5 +6,7 @@
        name="iri_wam">
   <!-- LINKS   -->
-  <include filename="$(find iri_wam_description)/xacro/wambase.urdf.xacro" />
+<!--  <include filename="$(find iri_wam_description)/xacro/wambase.urdf.xacro" />
+-->
+  <include filename="$(find iri_wam_description)/xacro/wam0.urdf.xacro" />
   <include filename="$(find iri_wam_description)/xacro/wam1.urdf.xacro" />
   <include filename="$(find iri_wam_description)/xacro/wam2.urdf.xacro" />
@@ -14,7 +16,12 @@
   <include filename="$(find iri_wam_description)/xacro/wam6.urdf.xacro" />
   <include filename="$(find iri_wam_description)/xacro/wam7.urdf.xacro" />
+  <include filename="$(find iri_wam_description)/xacro/wamtcp.urdf.xacro" />
+<!--
   <xacro:wambase>
   </xacro:wambase>
-  <xacro:wam1 parent="wambase">
+-->
+  <xacro:wam0>
+  </xacro:wam0>
+  <xacro:wam1 parent="wam_fk/wam0">
   </xacro:wam1>
   <xacro:wam2 parent="wam_fk/wam1">
@@ -30,3 +37,5 @@
   <xacro:wam7 parent="wam_fk/wam6">
   </xacro:wam7>
+  <xacro:wamtcp parent="wam_fk/wam7">
+  </xacro:wamtcp>
 </robot>

File: iri_wam_description/xacro/wam1.urdf.xacro (robot description, xacro)
@@ -34,5 +34,5 @@
         <parent link="${parent}"/>
         <child link="wam_fk/wam1"/>
-        <origin xyz="0.22 0.14 0.346" rpy="0 0 0" />
+        <origin xyz="0.0 0.0 0.0" rpy="0 0 0" />
         <axis xyz="0 0 1" />
         <limit lower="-2.6" upper="2.6" effort="30" velocity="2.0"/>
