Commit message: Added generic_camera.urdf.xacro and wam_with_camera.urdf.xacro

File: iri_wam_description/xacro/wam_with_camera.urdf.xacro (robot description, xacro)
@@ -17,4 +17,6 @@
   <include filename="$(find iri_wam_description)/xacro/wam7.urdf.xacro" />
   <include filename="$(find iri_wam_description)/xacro/wamtcp.urdf.xacro" />
+  <!-- Forward facing camera -->
+  <include filename="$(find iri_wam_description)/xacro/generic_camera.urdf.xacro" />
 <!--
   <xacro:wambase>
@@ -39,3 +41,7 @@
   <xacro:wamtcp parent="wam_link7">
   </xacro:wamtcp>
+<!-- Forward facing camera -->
+  <xacro:generic_camera name="front_cam" parent="wam_link7" ros_topic="camera/image" cam_info_topic="camera/camera_info" update_rate="10" res_x="320" res_y="240" image_format="R8G8B8" hfov="90">
+  <origin xyz="0.05 0.0 -0.06" rpy="0 0 0"/>
+  </xacro:generic_camera>
 </robot>
