Commit message: Added kinton_robot stack

File: iri_wam_description/xacro/generic_camera.urdf.xacro (robot description, xacro)
@@ -8,4 +8,5 @@
     <xacro:macro name="generic_camera" params="name parent *origin ros_topic cam_info_topic update_rate res_x res_y image_format hfov">
       <joint name="${name}_joint" type="fixed">
+        <origin xyz="0 0 0.09" rpy="0.0 ${-M_PI/2} 0.0" />
         <insert_block name="origin" />
         <parent link="${parent}"/>
@@ -28,5 +29,5 @@
         </visual>
         <collision>
-          <origin xyz="0 0 0" rpy="0 0 0" />
+          <origin xyz="0 0 0.09" rpy="0 0 0" />
           <geometry>
             <box size="0.01 0.01 0.01" />
@@ -35,5 +36,5 @@
       </link>
     <joint name="${name}_optical_joint" type="fixed">
-      <origin xyz="0 0 0" rpy="0.0 0.0 ${-M_PI/2}" />
+      <origin xyz="0 0 0" rpy="0.0 ${+M_PI/2} 0.0" />
       <parent link="${name}_link" />
       <child link="${name}_optical_frame"/>
@@ -77,7 +78,13 @@
         </controller:gazebo_ros_camera>
       </sensor:camera>
-      <turnGravityOff>true</turnGravityOff>
+      <turnGravityOff>false</turnGravityOff>
       <material>PR2/Blue</material>
     </gazebo>
+<!--    <joint name="${name}_fix" type="fixed">
+        <origin xyz="0.0 0.0 0.08" rpy="0 0 0" />
+        <parent link="${parent}"/>
+        <child link="${name}_link"/>
+     </joint>
+-->
     </xacro:macro>
   </robot>

File: iri_wam_simulator/gazebo/xacro/iri_wam.gazebo.xacro (robot description, xacro)
@@ -4,5 +4,5 @@
        xmlns:interface="http://playerstage.sourceforge.net/gazebo/xmlschema/#interface"
        name="iri_wam">
-  <include filename="$(find iri_wam_description)/xacro/wam.urdf.xacro" />
+  <include filename="$(find iri_wam_description)/xacro/wam_with_camera.urdf.xacro" />
   <gazebo>
 	<controller:gazebo_ros_controller_manager name="gazebo_ros_controller_manager" plugin="libgazebo_ros_controller_manager.so">
