Commit message: [iri_wam_description]   - New updated urdf file

File: ros/iri-ros-pkg/stacks/iri_wam/trunk/iri_wam_description/urdf/wam.urdf (robot description, URDF)
Before this commit: robot iri_wam, 9 links, 8 joints
Links:
- removed link wambase
- added link wam_link0, mass 20; collision mesh filename=package://iri_wam_description/mesh/wambase.stl scale=1.0 1.0 1.0; visual mesh filename=package://iri_wam_description/mesh/wambase.stl scale=1.0 1.0 1.0
- added link wam_tcp
Joints:
- removed joint base_fix
- added joint wam0_fix: type fixed, parent world, child wam_link0, origin xyz=0.22 0.14 0.346 rpy=0 0 0
- added joint wamtcp_fix: type fixed, parent wam_link7, child wam_tcp, origin xyz=0.0 0.0 0.06 rpy=0 0 0
- joint j1_joint: origin xyz=0.22 0.14 0.346 rpy=0 0 0 -> xyz=0.0 0.0 0.0 rpy=0 0 0; parent wambase -> wam_link0
