Commit message: [iri_wam_description]   - Re-structure of the node   - New link and joint names

File: ros/iri-ros-pkg/stacks/iri_wam/branches/groovy_and_moveit/iri_wam_description/urdf/wam.urdf (robot description, URDF)
Before this commit: robot iri_wam, 10 links, 9 joints
Links:
- removed link wam_link0
- removed link wam_link1
- removed link wam_link2
- removed link wam_link3
- removed link wam_link4
- removed link wam_link5
- removed link wam_link6
- removed link wam_link7
- removed link wam_tcp
- removed link world
- added link wam_link_1, mass 8.3936; collision mesh filename=package://iri_wam_description/mesh/wam1.stl scale=1.0 1.0 1.0; visual mesh filename=package://iri_wam_description/mesh/wam1.stl scale=1.0 1.0 1.0
- added link wam_link_2, mass 4.8487; collision mesh filename=package://iri_wam_description/mesh/wam2.stl scale=1.0 1.0 1.0; visual mesh filename=package://iri_wam_description/mesh/wam2.stl scale=1.0 1.0 1.0
- added link wam_link_3, mass 1.7251; collision mesh filename=package://iri_wam_description/mesh/wam3.stl scale=1.0 1.0 1.0; visual mesh filename=package://iri_wam_description/mesh/wam3.stl scale=1.0 1.0 1.0
- added link wam_link_4, mass 2.0824; collision mesh filename=package://iri_wam_description/mesh/wam4.stl scale=1.0 1.0 1.0; visual mesh filename=package://iri_wam_description/mesh/wam4.stl scale=1.0 1.0 1.0
- added link wam_link_5, mass 0.3067; collision mesh filename=package://iri_wam_description/mesh/wam5.stl scale=1.0 1.0 1.0; visual mesh filename=package://iri_wam_description/mesh/wam5.stl scale=1.0 1.0 1.0
- added link wam_link_6, mass 0.4278; collision mesh filename=package://iri_wam_description/mesh/wam6.stl scale=1.0 1.0 1.0; visual mesh filename=package://iri_wam_description/mesh/wam6.stl scale=1.0 1.0 1.0
- added link wam_link_7, mass 0.0557; collision mesh filename=package://iri_wam_description/mesh/wam7.stl scale=1.0 1.0 1.0; visual mesh filename=package://iri_wam_description/mesh/wam7.stl scale=1.0 1.0 1.0
- added link wam_link_base, mass 20; collision mesh filename=package://iri_wam_description/mesh/wambase.stl scale=1.0 1.0 1.0; visual mesh filename=package://iri_wam_description/mesh/wambase.stl scale=1.0 1.0 1.0
- added link wam_link_footprint
- added link wam_link_tcp
Joints:
- removed joint j1_joint
- removed joint j2_joint
- removed joint j3_joint
- removed joint j4_joint
- removed joint j5_joint
- removed joint j6_joint
- removed joint j7_joint
- removed joint wam0_fix
- removed joint wamtcp_fix
- added joint wam_joint_1: type revolute, parent wam_link_base, child wam_link_1, origin xyz=0.0 0.0 0.0 rpy=0 0 0, axis 0 0 1, limit lower=-2.6 upper=2.6 effort=30 velocity=2.0
- added joint wam_joint_2: type revolute, parent wam_link_1, child wam_link_2, origin xyz=0.0 0.0 0.0 rpy=0 0 0, axis 0 1 0, limit lower=-2.0 upper=2.0 effort=30 velocity=2.0
- added joint wam_joint_3: type revolute, parent wam_link_2, child wam_link_3, origin xyz=0.0 0.0 0.0 rpy=0 0 0, axis 0 0 1, limit lower=-2.8 upper=2.8 effort=30 velocity=2.0
- added joint wam_joint_4: type revolute, parent wam_link_3, child wam_link_4, origin xyz=0.045 0.0 0.55 rpy=-1.57079632679 0 0, axis 0 0 1, limit lower=-0.9 upper=2.8 effort=35 velocity=2.0
- added joint wam_joint_5: type revolute, parent wam_link_4, child wam_link_5, origin xyz=-0.045 -0.3 0.0 rpy=1.57079632679 0 0, axis 0 0 1, limit lower=-4.8 upper=1.3 effort=30 velocity=2.0
- added joint wam_joint_6: type revolute, parent wam_link_5, child wam_link_6, origin xyz=0.0 0.0 0.0 rpy=-1.57079632679 0 0, axis 0 0 1, limit lower=-1.6 upper=1.6 effort=30 velocity=2.0
- added joint wam_joint_7: type revolute, parent wam_link_6, child wam_link_7, origin xyz=0.0 0.0 0.0 rpy=1.57079632679 0 0, axis 0 0 1, limit lower=-2.2 upper=2.2 effort=30 velocity=2.0
- added joint wam_joint_footprint: type fixed, parent wam_link_footprint, child wam_link_base, origin xyz=0.22 0.14 0.346 rpy=0 0 0
- added joint wam_joint_tcp: type fixed, parent wam_link_7, child wam_link_tcp, origin xyz=0.0 0.0 0.06 rpy=0 0 0

File: ros/iri-ros-pkg/stacks/iri_wam/branches/groovy_and_moveit/iri_wam_description/xacro/wam.urdf.xacro (robot description, xacro)
@@ -1,12 +1,6 @@
 <?xml version="1.0"?>
-<robot xmlns:sensor="http://playerstage.sourceforge.net/gazebo/xmlschema/#sensor"
-       xmlns:controller="http://playerstage.sourceforge.net/gazebo/xmlschema/#controller"
-       xmlns:interface="http://playerstage.sourceforge.net/gazebo/xmlschema/#interface"
-       xmlns:xacro="http://ros.org/wiki/xacro"
-       name="iri_wam">
-  <!-- LINKS   -->
-<!--  <include filename="$(find iri_wam_description)/xacro/wambase.urdf.xacro" />
--->
-  <include filename="$(find iri_wam_description)/xacro/wam0.urdf.xacro" />
+<robot name="iri_wam" xmlns:xacro="http://ros.org/wiki/xacro" >
+<!-- Set up definitions of parts of the robot body -->
+  <include filename="$(find iri_wam_description)/xacro/wambase.urdf.xacro" />
   <include filename="$(find iri_wam_description)/xacro/wam1.urdf.xacro" />
   <include filename="$(find iri_wam_description)/xacro/wam2.urdf.xacro" />
@@ -17,25 +11,20 @@
   <include filename="$(find iri_wam_description)/xacro/wam7.urdf.xacro" />
   <include filename="$(find iri_wam_description)/xacro/wamtcp.urdf.xacro" />
-<!--
-  <xacro:wambase>
-  </xacro:wambase>
--->
-  <xacro:wam0>
-  </xacro:wam0>
-  <xacro:wam1 parent="wam_link0">
-  </xacro:wam1>
-  <xacro:wam2 parent="wam_link1">
-  </xacro:wam2>
-  <xacro:wam3 parent="wam_link2">
-  </xacro:wam3>
-  <xacro:wam4 parent="wam_link3">
-  </xacro:wam4>
-  <xacro:wam5 parent="wam_link4">
-  </xacro:wam5>
-  <xacro:wam6 parent="wam_link5">
-  </xacro:wam6>
-  <xacro:wam7 parent="wam_link6">
-  </xacro:wam7>
-  <xacro:wamtcp parent="wam_link7">
-  </xacro:wamtcp>
+  <!-- The first use of a macro.  This one was defined in wambase.urdf.xacro above.
+       A macro like this will expand to a set of link and joint definitions, and to additional
+       Gazebo-related extensions (sensor plugins, etc).  The macro takes an argument, name,
+       that equals "base", and uses it to generate names for its component links and joints
+       (e.g., base_link).  The included origin block is also an argument to the macro.  By convention,
+       the origin block defines where the component is w.r.t its parent (in this case the parent
+       is the world frame). For more, see http://www.ros.org/wiki/xacro -->
+  <property name="robot_name" value="wam"/>
+  <xacro:wambase prefix="${robot_name}"/>
+  <xacro:wam1 prefix="${robot_name}" parent="wam_link_base"/>
+  <xacro:wam2 prefix="${robot_name}" parent="wam_link_1"/>
+  <xacro:wam3 prefix="${robot_name}" parent="wam_link_2"/>
+  <xacro:wam4 prefix="${robot_name}" parent="wam_link_3"/>
+  <xacro:wam5 prefix="${robot_name}" parent="wam_link_4"/>
+  <xacro:wam6 prefix="${robot_name}" parent="wam_link_5"/>
+  <xacro:wam7 prefix="${robot_name}" parent="wam_link_6"/>
+  <xacro:wamtcp prefix="${robot_name}" parent="wam_link_7"/>
 </robot>

File: ros/iri-ros-pkg/stacks/iri_wam/branches/groovy_and_moveit/iri_wam_description/xacro/wam1.urdf.xacro (robot description, xacro)
@@ -1,14 +1,17 @@
 <?xml version="1.0"?>
 <robot xmlns:xacro="http://www.ros.org/wiki/xacro">
-  <xacro:macro name="wam1" params="parent">
-    <link name="wam_link1">
+  <property name="M_PI" value="3.1415926535897931" />
+  <xacro:macro name="wam1" params="prefix parent">
+    <link name="${prefix}_link_1">
         <inertial>
             <mass value="8.3936" />
             <origin xyz="0.0 0.0 0.0" rpy="0 0 0" />
-            <inertia  ixx="1.0" ixy="0.0"  ixz="0.0"  iyy="1.0"  iyz="0.0"  izz="1.0" />
+            <inertia ixx="1.0" ixy="0.0" ixz="0.0"
+                     iyy="1.0" iyz="0.0"
+                     izz="1.0" />
         </inertial>
         <visual>
             <origin xyz="0.0 0.0 0.0" rpy="0 0 0" />
-            <geometry name="wam_link1_visual">
+            <geometry name="${prefix}_link_1_visual">
                 <mesh filename="package://iri_wam_description/mesh/wam1.stl" scale="1.0 1.0 1.0" />
             </geometry>
@@ -19,30 +22,30 @@
         <collision>
             <origin xyz="0.0 0.0 0.0" rpy="0 0 0"/>
-            <geometry name="wam_link1_collision">
+            <geometry name="${prefix}_link_1_collision">
                 <mesh filename="package://iri_wam_description/mesh/wam1.stl" scale="1.0 1.0 1.0" />
-<!--                <box size="0.20 0.40 0.40"/>
--->
+<!--                <box size="0.20 0.40 0.40"/> -->
             </geometry>
             <contact_coefficients kd="1.0" kp="1000.0" mu="0"/>
         </collision>
     </link>
-    <gazebo reference="wam_link1">
+    <gazebo reference="${prefix}_link_1">
         <material>Gazebo/Grey</material>
         <selfCollide>true</selfCollide>
     </gazebo>
-    <joint name="j1_joint" type="revolute">
+    <joint name="${prefix}_joint_1" type="revolute">
         <parent link="${parent}"/>
-        <child link="wam_link1"/>
+        <child link="${prefix}_link_1"/>
         <origin xyz="0.0 0.0 0.0" rpy="0 0 0" />
         <axis xyz="0 0 1" />
         <limit lower="-2.6" upper="2.6" effort="30" velocity="2.0"/>
-   <!--  <safety_controller k_velocity="0.5"/>-->
+        <!-- <safety_controller k_velocity="0.5"/> -->
         <dynamics damping="100"/>
-     </joint>
+    </joint>
     <transmission type="pr2_mechanism_model/SimpleTransmission" name="j1_transmission">
       <actuator name="j1" />
-      <joint name="j1_joint" />
+      <joint name="${prefix}_joint_1" />
       <mechanicalReduction>1</mechanicalReduction>
       <motorTorqueConstant>1</motorTorqueConstant>
+      <!-- <pulsesPerRevolution>90000</pulsesPerRevolution> -->
     </transmission>
   </xacro:macro>

File: ros/iri-ros-pkg/stacks/iri_wam/branches/groovy_and_moveit/iri_wam_description/xacro/wam2.urdf.xacro (robot description, xacro)
@@ -1,14 +1,17 @@
 <?xml version="1.0"?>
 <robot xmlns:xacro="http://www.ros.org/wiki/xacro">
-  <xacro:macro name="wam2" params="parent">
-    <link name="wam_link2">
+  <property name="M_PI" value="3.1415926535897931" />
+  <xacro:macro name="wam2" params="prefix parent">
+    <link name="${prefix}_link_2">
         <inertial>
+            <mass value="4.8487" />
             <origin xyz="0 0 0" rpy="0 0 0" />
-             <mass value="4.8487" />
-            <inertia  ixx="1.0" ixy="0.0"  ixz="0.0"  iyy="0.1"  iyz="0.0"  izz="0.1" />
+            <inertia ixx="1.0" ixy="0.0" ixz="0.0"
+                     iyy="1.0" iyz="0.0"
+                     izz="1.0" />
         </inertial>
         <visual>
             <origin xyz="0.0 0.0 0.0" rpy="0 0 0" />
-            <geometry name="wam_link2_visual">
+            <geometry name="${prefix}_link_2_visual">
                 <mesh filename="package://iri_wam_description/mesh/wam2.stl" scale="1.0 1.0 1.0" />
             </geometry>
@@ -19,5 +22,5 @@
         <collision>
             <origin xyz="0.0 0.0 0.0" rpy="0 0 0"/>
-            <geometry name="wam_link2_collision">
+            <geometry name="${prefix}_link_2_collision">
                 <mesh filename="package://iri_wam_description/mesh/wam2.stl" scale="1.0 1.0 1.0" />
 <!--                <box size="0.10 0.10 0.10"/> -->
@@ -26,23 +29,23 @@
         </collision>
     </link>
-    <gazebo reference="wam_link2">
+    <gazebo reference="${prefix}_link_2">
         <material>Gazebo/Grey</material>
         <selfCollide>true</selfCollide>
     </gazebo>
-    <joint name="j2_joint" type="revolute">
+    <joint name="${prefix}_joint_2" type="revolute">
         <parent link="${parent}"/>
-        <child link="wam_link2"/>
+        <child link="${prefix}_link_2"/>
         <origin xyz="0.0 0.0 0.0" rpy="0 0 0" />
         <axis xyz="0 1 0" />
         <limit lower="-2.0" upper="2.0" effort="30" velocity="2.0"/>
-        <!--<safety_controller k_velocity="0.5"/>-->
+        <!-- <safety_controller k_velocity="0.5"/> -->
         <dynamics damping="100"/>
     </joint>
     <transmission type="pr2_mechanism_model/SimpleTransmission" name="j2_transmission">
       <actuator name="j2" />
-      <joint name="j2_joint" />
+      <joint name="${prefix}_joint_2" />
       <mechanicalReduction>1</mechanicalReduction>
       <motorTorqueConstant>1</motorTorqueConstant>
-      <!--<pulsesPerRevolution>90000</pulsesPerRevolution>-->
+      <!-- <pulsesPerRevolution>90000</pulsesPerRevolution> -->
     </transmission>
   </xacro:macro>

File: ros/iri-ros-pkg/stacks/iri_wam/branches/groovy_and_moveit/iri_wam_description/xacro/wam3.urdf.xacro (robot description, xacro)
@@ -1,14 +1,17 @@
 <?xml version="1.0"?>
 <robot xmlns:xacro="http://www.ros.org/wiki/xacro">
-  <xacro:macro name="wam3" params="parent">
-    <link name="wam_link3">
+  <property name="M_PI" value="3.1415926535897931" />
+  <xacro:macro name="wam3" params="prefix parent">
+    <link name="${prefix}_link_3">
         <inertial>
             <mass value="1.7251" />
             <origin xyz="0 0 0.225" rpy="0 0 0" />
-            <inertia  ixx="1.0" ixy="0.0"  ixz="0.0"  iyy="0.1"  iyz="0.0"  izz="0.1" />
+            <inertia ixx="1.0" ixy="0.0" ixz="0.0"
+                     iyy="1.0" iyz="0.0"
+                     izz="1.0" />
         </inertial>
         <visual>
             <origin xyz="0.0 0.0 0.0" rpy="0 0 0" />
-            <geometry name="wam_link3_visual">
+            <geometry name="${prefix}_link_3_visual">
                 <mesh filename="package://iri_wam_description/mesh/wam3.stl" scale="1.0 1.0 1.0" />
             </geometry>
@@ -19,5 +22,5 @@
         <collision>
             <origin xyz="0.0 0.0 0.0" rpy="0 0 0"/>
-            <geometry name="wam_link3_collision">
+            <geometry name="${prefix}_link_3_collision">
                 <mesh filename="package://iri_wam_description/mesh/wam3.stl" scale="1.0 1.0 1.0" />
 <!--                <box size="0.10 0.10 0.10"/> -->
@@ -26,23 +29,23 @@
         </collision>
     </link>
-    <gazebo reference="wam_link3">
+    <gazebo reference="${prefix}_link_3">
         <material>Gazebo/Grey</material>
         <selfCollide>true</selfCollide>
     </gazebo>
-    <joint name="j3_joint" type="revolute">
+    <joint name="${prefix}_joint_3" type="revolute">
         <parent link="${parent}"/>
-        <child link="wam_link3"/>
+        <child link="${prefix}_link_3"/>
         <origin xyz="0.0 0.0 0.0" rpy="0 0 0" />
         <axis xyz="0 0 1" />
         <limit lower="-2.8" upper="2.8" effort="30" velocity="2.0"/>
-        <!--  <safety_controller k_velocity="0.5"/>-->
+        <!-- <safety_controller k_velocity="0.5"/> -->
         <dynamics damping="100"/>
     </joint>
     <transmission type="pr2_mechanism_model/SimpleTransmission" name="j3_transmission">
       <actuator name="j3" />
-      <joint name="j3_joint" />
+      <joint name="${prefix}_joint_3" />
       <mechanicalReduction>1</mechanicalReduction>
       <motorTorqueConstant>1</motorTorqueConstant>
-     <!-- <pulsesPerRevolution>90000</pulsesPerRevolution>-->
+      <!-- <pulsesPerRevolution>90000</pulsesPerRevolution> -->
     </transmission>
   </xacro:macro>

File: ros/iri-ros-pkg/stacks/iri_wam/branches/groovy_and_moveit/iri_wam_description/xacro/wam4.urdf.xacro (robot description, xacro)
@@ -1,15 +1,17 @@
 <?xml version="1.0"?>
 <robot xmlns:xacro="http://www.ros.org/wiki/xacro">
-<property name="M_PI" value="3.1415926535897931" />
-  <xacro:macro name="wam4" params="parent">
-    <link name="wam_link4">
+  <property name="M_PI" value="3.1415926535897931" />
+  <xacro:macro name="wam4" params="prefix parent">
+    <link name="${prefix}_link_4">
         <inertial>
             <mass value="2.0824" />
             <origin xyz="-0.045 -0.15 0" rpy="0 0 0" />
-            <inertia  ixx="1.0" ixy="0.0"  ixz="0.0"  iyy="0.1"  iyz="0.0"  izz="0.1" />
+            <inertia ixx="1.0" ixy="0.0" ixz="0.0"
+                     iyy="1.0" iyz="0.0"
+                     izz="1.0" />
         </inertial>
         <visual>
             <origin xyz="0.0 0.0 0.0" rpy="0 0 0" />
-            <geometry name="wam_link4_visual">
+            <geometry name="${prefix}_link_4_visual">
                 <mesh filename="package://iri_wam_description/mesh/wam4.stl" scale="1.0 1.0 1.0" />
             </geometry>
@@ -20,5 +22,5 @@
         <collision>
             <origin xyz="0.0 0.0 0.0" rpy="0 0 0"/>
-            <geometry name="wam_link4_collision">
+            <geometry name="${prefix}_link_4_collision">
                 <mesh filename="package://iri_wam_description/mesh/wam4.stl" scale="1.0 1.0 1.0" />
 <!--                <box size="0.10 0.10 0.10"/> -->
@@ -27,23 +29,23 @@
         </collision>
     </link>
-    <gazebo reference="wam_link4">
+    <gazebo reference="${prefix}_link_4">
         <material>Gazebo/Grey</material>
         <selfCollide>true</selfCollide>
     </gazebo>
-    <joint name="j4_joint" type="revolute">
+    <joint name="${prefix}_joint_4" type="revolute">
         <parent link="${parent}"/>
-        <child link="wam_link4"/>
+        <child link="${prefix}_link_4"/>
         <origin xyz="0.045 0.0 0.55" rpy="-${M_PI/2} 0 0" />
         <axis xyz="0 0 1" />
         <limit lower="-0.9" upper="2.8" effort="35" velocity="2.0"/>
-  <!--  <safety_controller k_velocity="0.5"/>-->
-  <dynamics damping="100"/>
+        <!-- <safety_controller k_velocity="0.5"/> -->
+        <dynamics damping="100"/>
     </joint>
     <transmission type="pr2_mechanism_model/SimpleTransmission" name="j4_transmission">
       <actuator name="j4" />
-      <joint name="j4_joint" />
+      <joint name="${prefix}_joint_4" />
       <mechanicalReduction>1</mechanicalReduction>
       <motorTorqueConstant>1</motorTorqueConstant>
-      <!--<pulsesPerRevolution>90000</pulsesPerRevolution>-->
+      <!-- <pulsesPerRevolution>90000</pulsesPerRevolution> -->
     </transmission>
   </xacro:macro>

File: ros/iri-ros-pkg/stacks/iri_wam/branches/groovy_and_moveit/iri_wam_description/xacro/wam5.urdf.xacro (robot description, xacro)
@@ -1,15 +1,17 @@
 <?xml version="1.0"?>
 <robot xmlns:xacro="http://www.ros.org/wiki/xacro">
-<property name="M_PI" value="3.1415926535897931" />
-  <xacro:macro name="wam5" params="parent">
-    <link name="wam_link5">
+  <property name="M_PI" value="3.1415926535897931" />
+  <xacro:macro name="wam5" params="prefix parent">
+    <link name="${prefix}_link_5">
         <inertial>
+            <mass value="0.3067" />
             <origin xyz="0 0 0" rpy="0 0 0" />
-             <mass value="0.3067" />
-            <inertia  ixx="1.0" ixy="0.0"  ixz="0.0"  iyy="0.1"  iyz="0.0"  izz="0.1" />
+            <inertia ixx="1.0" ixy="0.0" ixz="0.0"
+                     iyy="1.0" iyz="0.0"
+                     izz="1.0" />
         </inertial>
         <visual>
             <origin xyz="0.0 0.0 0.0" rpy="0 0 0" />
-            <geometry name="wam_link5_visual">
+            <geometry name="${prefix}_link_5_visual">
                 <mesh filename="package://iri_wam_description/mesh/wam5.stl" scale="1.0 1.0 1.0" />
             </geometry>
@@ -20,5 +22,5 @@
         <collision>
             <origin xyz="0.0 0.0 0.0" rpy="0 0 0"/>
-            <geometry name="wam_link5_collision">
+            <geometry name="${prefix}_link_5_collision">
                 <mesh filename="package://iri_wam_description/mesh/wam5.stl" scale="1.0 1.0 1.0" />
 <!--                <box size="0.10 0.10 0.10"/> -->
@@ -27,23 +29,23 @@
         </collision>
     </link>
-    <gazebo reference="wam_link5">
+    <gazebo reference="${prefix}_link_5">
         <material>Gazebo/Grey</material>
         <selfCollide>true</selfCollide>
     </gazebo>
-    <joint name="j5_joint" type="revolute">
+    <joint name="${prefix}_joint_5" type="revolute">
         <parent link="${parent}"/>
-        <child link="wam_link5"/>
+        <child link="${prefix}_link_5"/>
         <origin xyz="-0.045 -0.3 0.0" rpy="${M_PI/2} 0 0" />
         <axis xyz="0 0 1" />
         <limit lower="-4.8" upper="1.3" effort="30" velocity="2.0"/>
-   <!--  <safety_controller k_velocity="0.5"/>-->
-   <dynamics damping="100"/>
+        <!-- <safety_controller k_velocity="0.5"/> -->
+        <dynamics damping="100"/>
     </joint>
     <transmission type="pr2_mechanism_model/SimpleTransmission" name="j5_transmission">
       <actuator name="j5" />
-      <joint name="j5_joint" />
+      <joint name="${prefix}_joint_5" />
       <mechanicalReduction>1</mechanicalReduction>
       <motorTorqueConstant>1</motorTorqueConstant>
-    <!--  <pulsesPerRevolution>90000</pulsesPerRevolution>-->
+      <!-- <pulsesPerRevolution>90000</pulsesPerRevolution> -->
     </transmission>
   </xacro:macro>
