Commit message: [iri_wam_description]   - Re-structure of the node   - New link and joint names

File: ros/iri-ros-pkg/stacks/iri_wam/branches/groovy_and_moveit/iri_wam_description/xacro/wam6.urdf.xacro (robot description, xacro)
@@ -1,15 +1,17 @@
 <?xml version="1.0"?>
 <robot xmlns:xacro="http://www.ros.org/wiki/xacro">
-<property name="M_PI" value="3.1415926535897931" />
-  <xacro:macro name="wam6" params="parent">
-    <link name="wam_link6">
+  <property name="M_PI" value="3.1415926535897931" />
+  <xacro:macro name="wam6" params="prefix parent">
+    <link name="${prefix}_link_6">
         <inertial>
+            <mass value="0.4278" />
             <origin xyz="0 0 0" rpy="0 0 0" />
-             <mass value="0.4278" />
-            <inertia  ixx="1.0" ixy="0.0"  ixz="0.0"  iyy="0.1"  iyz="0.0"  izz="0.1" />
+            <inertia ixx="1.0" ixy="0.0" ixz="0.0"
+                     iyy="1.0" iyz="0.0"
+                     izz="1.0" />
         </inertial>
         <visual>
             <origin xyz="0.0 0.0 0.0" rpy="0 0 0" />
-            <geometry name="wam_link6_visual">
+            <geometry name="${prefix}_link_6_visual">
                 <mesh filename="package://iri_wam_description/mesh/wam6.stl" scale="1.0 1.0 1.0" />
             </geometry>
@@ -20,5 +22,5 @@
         <collision>
             <origin xyz="0.0 0.0 0.0" rpy="0 0 0"/>
-            <geometry name="wam_link6_collision">
+            <geometry name="${prefix}_link_6_collision">
                 <mesh filename="package://iri_wam_description/mesh/wam6.stl" scale="1.0 1.0 1.0" />
 <!--                <box size="0.10 0.10 0.10"/> -->
@@ -27,23 +29,23 @@
         </collision>
     </link>
-    <gazebo reference="wam_link6">
+    <gazebo reference="${prefix}_link_6">
         <material>Gazebo/Grey</material>
         <selfCollide>true</selfCollide>
     </gazebo>
-    <joint name="j6_joint" type="revolute">
+    <joint name="${prefix}_joint_6" type="revolute">
         <parent link="${parent}"/>
-        <child link="wam_link6"/>
+        <child link="${prefix}_link_6"/>
         <origin xyz="0.0 0.0 0.0" rpy="-${M_PI/2} 0 0" />
         <axis xyz="0 0 1" />
         <limit lower="-1.6" upper="1.6" effort="30" velocity="2.0"/>
-        <!--  <safety_controller k_velocity="0.5"/>-->
+        <!-- <safety_controller k_velocity="0.5"/> -->
         <dynamics damping="100"/>
     </joint>
     <transmission type="pr2_mechanism_model/SimpleTransmission" name="j6_transmission">
       <actuator name="j6" />
-      <joint name="j6_joint" />
+      <joint name="${prefix}_joint_6" />
       <mechanicalReduction>1</mechanicalReduction>
       <motorTorqueConstant>1</motorTorqueConstant>
-    <!--  <pulsesPerRevolution>90000</pulsesPerRevolution>-->
+      <!-- <pulsesPerRevolution>90000</pulsesPerRevolution> -->
     </transmission>
   </xacro:macro>

File: ros/iri-ros-pkg/stacks/iri_wam/branches/groovy_and_moveit/iri_wam_description/xacro/wam7.urdf.xacro (robot description, xacro)
@@ -1,15 +1,17 @@
 <?xml version="1.0"?>
 <robot xmlns:xacro="http://www.ros.org/wiki/xacro">
-<property name="M_PI" value="3.1415926535897931" />
-  <xacro:macro name="wam7" params="parent">
-    <link name="wam_link7">
+  <property name="M_PI" value="3.1415926535897931" />
+  <xacro:macro name="wam7" params="prefix parent">
+    <link name="${prefix}_link_7">
         <inertial>
+            <mass value="0.0557" />
             <origin xyz="0 0 0" rpy="0 0 0" />
-             <mass value="0.0557" />
-            <inertia  ixx="1.0" ixy="0.0"  ixz="0.0"  iyy="0.1"  iyz="0.0"  izz="0.1" />
+            <inertia ixx="1.0" ixy="0.0" ixz="0.0"
+                     iyy="1.0" iyz="0.0"
+                     izz="1.0" />
         </inertial>
         <visual>
             <origin xyz="0.0 0.0 0.0" rpy="0 0 0" />
-            <geometry name="wam_link7_visual">
+            <geometry name="${prefix}_link_7_visual">
                 <mesh filename="package://iri_wam_description/mesh/wam7.stl" scale="1.0 1.0 1.0" />
             </geometry>
@@ -20,5 +22,5 @@
         <collision>
             <origin xyz="0.0 0.0 0.0" rpy="0 0 0"/>
-            <geometry name="wam_link7_collision">
+            <geometry name="${prefix}_link_7_collision">
                 <mesh filename="package://iri_wam_description/mesh/wam7.stl" scale="1.0 1.0 1.0" />
 <!--                <box size="0.10 0.10 0.10"/> -->
@@ -27,23 +29,23 @@
         </collision>
     </link>
-    <gazebo reference="wam_link7">
+    <gazebo reference="${prefix}_link_7">
         <material>Gazebo/Grey</material>
         <selfCollide>true</selfCollide>
     </gazebo>
-    <joint name="j7_joint" type="revolute">
+    <joint name="${prefix}_joint_7" type="revolute">
         <parent link="${parent}"/>
-        <child link="wam_link7"/>
+        <child link="${prefix}_link_7"/>
         <origin xyz="0.0 0.0 0.0" rpy="${M_PI/2} 0 0" />
         <axis xyz="0 0 1" />
         <limit lower="-2.2" upper="2.2" effort="30" velocity="2.0"/>
-      <!--  <safety_controller k_velocity="0.5"/>-->
-      <dynamics damping="100"/>
+        <!-- <safety_controller k_velocity="0.5"/> -->
+        <dynamics damping="100"/>
     </joint>
     <transmission type="pr2_mechanism_model/SimpleTransmission" name="j7_transmission">
       <actuator name="j7" />
-      <joint name="j7_joint" />
+      <joint name="${prefix}_joint_7" />
       <mechanicalReduction>1</mechanicalReduction>
       <motorTorqueConstant>1</motorTorqueConstant>
-      <!--<pulsesPerRevolution>90000</pulsesPerRevolution>-->
+      <!-- <pulsesPerRevolution>90000</pulsesPerRevolution> -->
     </transmission>
   </xacro:macro>

File: ros/iri-ros-pkg/stacks/iri_wam/branches/groovy_and_moveit/iri_wam_description/xacro/wamtcp.urdf.xacro (robot description, xacro)
@@ -1,12 +1,12 @@
 <?xml version="1.0"?>
 <robot xmlns:xacro="http://www.ros.org/wiki/xacro">
-<property name="M_PI" value="3.1415926535897931" />
-<xacro:macro name="wamtcp" params="parent">
-  <link name="wam_tcp" />
-  <joint name="wamtcp_fix" type="fixed" >
-    <parent link="${parent}" />
-    <child link="wam_tcp" />
-    <origin xyz="0.0 0.0 0.06" rpy="0 0 0" />
-  </joint>
-</xacro:macro>
+  <property name="M_PI" value="3.1415926535897931" />
+  <xacro:macro name="wamtcp" params="prefix parent">
+    <link name="${prefix}_link_tcp" />
+    <joint name="${prefix}_joint_tcp" type="fixed" >
+      <parent link="${parent}" />
+      <child link="${prefix}_link_tcp" />
+      <origin xyz="0.0 0.0 0.06" rpy="0 0 0" />
+    </joint>
+  </xacro:macro>
 </robot>

Commit message: [iri_wam_description]   - Standarizing iri_wam naming

File: ros/iri-ros-pkg/stacks/iri_wam/branches/groovy_and_moveit/iri_wam_description/urdf/wam.urdf (robot description, URDF)
Before this commit: robot iri_wam, 10 links, 9 joints
Links:
- removed link wam_link_1
- removed link wam_link_2
- removed link wam_link_3
- removed link wam_link_4
- removed link wam_link_5
- removed link wam_link_6
- removed link wam_link_7
- removed link wam_link_base
- removed link wam_link_footprint
- removed link wam_link_tcp
- added link iri_wam_link_1, mass 8.3936; collision mesh filename=package://iri_wam_description/mesh/wam1.stl scale=1.0 1.0 1.0; visual mesh filename=package://iri_wam_description/mesh/wam1.stl scale=1.0 1.0 1.0
- added link iri_wam_link_2, mass 4.8487; collision mesh filename=package://iri_wam_description/mesh/wam2.stl scale=1.0 1.0 1.0; visual mesh filename=package://iri_wam_description/mesh/wam2.stl scale=1.0 1.0 1.0
- added link iri_wam_link_3, mass 1.7251; collision mesh filename=package://iri_wam_description/mesh/wam3.stl scale=1.0 1.0 1.0; visual mesh filename=package://iri_wam_description/mesh/wam3.stl scale=1.0 1.0 1.0
- added link iri_wam_link_4, mass 2.0824; collision mesh filename=package://iri_wam_description/mesh/wam4.stl scale=1.0 1.0 1.0; visual mesh filename=package://iri_wam_description/mesh/wam4.stl scale=1.0 1.0 1.0
- added link iri_wam_link_5, mass 0.3067; collision mesh filename=package://iri_wam_description/mesh/wam5.stl scale=1.0 1.0 1.0; visual mesh filename=package://iri_wam_description/mesh/wam5.stl scale=1.0 1.0 1.0
- added link iri_wam_link_6, mass 0.4278; collision mesh filename=package://iri_wam_description/mesh/wam6.stl scale=1.0 1.0 1.0; visual mesh filename=package://iri_wam_description/mesh/wam6.stl scale=1.0 1.0 1.0
- added link iri_wam_link_7, mass 0.0557; collision mesh filename=package://iri_wam_description/mesh/wam7.stl scale=1.0 1.0 1.0; visual mesh filename=package://iri_wam_description/mesh/wam7.stl scale=1.0 1.0 1.0
- added link iri_wam_link_base, mass 20; collision mesh filename=package://iri_wam_description/mesh/wambase.stl scale=1.0 1.0 1.0; visual mesh filename=package://iri_wam_description/mesh/wambase.stl scale=1.0 1.0 1.0
- added link iri_wam_link_footprint
- added link iri_wam_link_tcp
Joints:
- removed joint wam_joint_1
- removed joint wam_joint_2
- removed joint wam_joint_3
- removed joint wam_joint_4
- removed joint wam_joint_5
- removed joint wam_joint_6
- removed joint wam_joint_7
- removed joint wam_joint_footprint
- removed joint wam_joint_tcp
- added joint iri_wam_joint_1: type revolute, parent iri_wam_link_base, child iri_wam_link_1, origin xyz=0.0 0.0 0.0 rpy=0 0 0, axis 0 0 1, limit lower=-2.6 upper=2.6 effort=30 velocity=2.0
- added joint iri_wam_joint_2: type revolute, parent iri_wam_link_1, child iri_wam_link_2, origin xyz=0.0 0.0 0.0 rpy=0 0 0, axis 0 1 0, limit lower=-2.0 upper=2.0 effort=30 velocity=2.0
- added joint iri_wam_joint_3: type revolute, parent iri_wam_link_2, child iri_wam_link_3, origin xyz=0.0 0.0 0.0 rpy=0 0 0, axis 0 0 1, limit lower=-2.8 upper=2.8 effort=30 velocity=2.0
- added joint iri_wam_joint_4: type revolute, parent iri_wam_link_3, child iri_wam_link_4, origin xyz=0.045 0.0 0.55 rpy=-1.57079632679 0 0, axis 0 0 1, limit lower=-0.9 upper=2.8 effort=35 velocity=2.0
- added joint iri_wam_joint_5: type revolute, parent iri_wam_link_4, child iri_wam_link_5, origin xyz=-0.045 -0.3 0.0 rpy=1.57079632679 0 0, axis 0 0 1, limit lower=-4.8 upper=1.3 effort=30 velocity=2.0
- added joint iri_wam_joint_6: type revolute, parent iri_wam_link_5, child iri_wam_link_6, origin xyz=0.0 0.0 0.0 rpy=-1.57079632679 0 0, axis 0 0 1, limit lower=-1.6 upper=1.6 effort=30 velocity=2.0
- added joint iri_wam_joint_7: type revolute, parent iri_wam_link_6, child iri_wam_link_7, origin xyz=0.0 0.0 0.0 rpy=1.57079632679 0 0, axis 0 0 1, limit lower=-2.2 upper=2.2 effort=30 velocity=2.0
- added joint iri_wam_joint_footprint: type fixed, parent iri_wam_link_footprint, child iri_wam_link_base, origin xyz=0.22 0.14 0.346 rpy=0 0 0
- added joint iri_wam_joint_tcp: type fixed, parent iri_wam_link_7, child iri_wam_link_tcp, origin xyz=0.0 0.0 0.06 rpy=0 0 0

File: ros/iri-ros-pkg/stacks/iri_wam/branches/groovy_and_moveit/iri_wam_description/xacro/wam.urdf.xacro (robot description, xacro)
@@ -1,5 +1,5 @@
 <?xml version="1.0"?>
 <robot name="iri_wam" xmlns:xacro="http://ros.org/wiki/xacro" >
-<!-- Set up definitions of parts of the robot body -->
+  <!-- Set up definitions of parts of the robot body -->
   <include filename="$(find iri_wam_description)/xacro/wambase.urdf.xacro" />
   <include filename="$(find iri_wam_description)/xacro/wam1.urdf.xacro" />
@@ -11,20 +11,20 @@
   <include filename="$(find iri_wam_description)/xacro/wam7.urdf.xacro" />
   <include filename="$(find iri_wam_description)/xacro/wamtcp.urdf.xacro" />
-  <!-- The first use of a macro.  This one was defined in wambase.urdf.xacro above.
+  <!-- The first use of a macro. This one was defined in wambase.urdf.xacro above.
        A macro like this will expand to a set of link and joint definitions, and to additional
        Gazebo-related extensions (sensor plugins, etc).  The macro takes an argument, name,
-       that equals "base", and uses it to generate names for its component links and joints
-       (e.g., base_link).  The included origin block is also an argument to the macro.  By convention,
+       that equals "wam", and uses it to generate names for its component links and joints
+       (e.g., wam_link_base).  The included origin block is also an argument to the macro.  By convention,
        the origin block defines where the component is w.r.t its parent (in this case the parent
        is the world frame). For more, see http://www.ros.org/wiki/xacro -->
-  <property name="robot_name" value="wam"/>
+  <property name="robot_name" value="iri_wam"/>
   <xacro:wambase prefix="${robot_name}"/>
-  <xacro:wam1 prefix="${robot_name}" parent="wam_link_base"/>
-  <xacro:wam2 prefix="${robot_name}" parent="wam_link_1"/>
-  <xacro:wam3 prefix="${robot_name}" parent="wam_link_2"/>
-  <xacro:wam4 prefix="${robot_name}" parent="wam_link_3"/>
-  <xacro:wam5 prefix="${robot_name}" parent="wam_link_4"/>
-  <xacro:wam6 prefix="${robot_name}" parent="wam_link_5"/>
-  <xacro:wam7 prefix="${robot_name}" parent="wam_link_6"/>
-  <xacro:wamtcp prefix="${robot_name}" parent="wam_link_7"/>
+  <xacro:wam1 prefix="${robot_name}" parent="${robot_name}_link_base"/>
+  <xacro:wam2 prefix="${robot_name}" parent="${robot_name}_link_1"/>
+  <xacro:wam3 prefix="${robot_name}" parent="${robot_name}_link_2"/>
+  <xacro:wam4 prefix="${robot_name}" parent="${robot_name}_link_3"/>
+  <xacro:wam5 prefix="${robot_name}" parent="${robot_name}_link_4"/>
+  <xacro:wam6 prefix="${robot_name}" parent="${robot_name}_link_5"/>
+  <xacro:wam7 prefix="${robot_name}" parent="${robot_name}_link_6"/>
+  <xacro:wamtcp prefix="${robot_name}" parent="${robot_name}_link_7"/>
 </robot>
