Commit message: [iri_wam_description]  - Xacro files update for compatibility with hydro and gazebo

File: ros/iri-ros-pkg/stacks/iri_wam/trunk/iri_wam_description/xacro/iri_wam.urdf.xacro (robot description, xacro)
@@ -1,4 +1,13 @@
 <?xml version="1.0"?>
 <robot name="iri_wam" xmlns:xacro="http://ros.org/wiki/xacro" >
+  <!-- ros_control plugin -->
+  <gazebo>
+    <plugin name="gazebo_ros_control" filename="libgazebo_ros_control.so">
+      <alwaysOn>true</alwaysOn>
+      <updateRate>1000.0</updateRate>
+      <robotParam>robot_description</robotParam>
+      <robotNamespace>/iri_wam</robotNamespace>
+    </plugin>
+  </gazebo>
   <!-- Set up definitions of parts of the robot body -->
   <xacro:include filename="$(find iri_wam_description)/xacro/iri_wam_base.urdf.xacro" />

File: ros/iri-ros-pkg/stacks/iri_wam/trunk/iri_wam_description/xacro/iri_wam_1.urdf.xacro (robot description, xacro)
@@ -42,10 +42,13 @@
         <dynamics damping="100"/>
     </joint>
-    <transmission type="pr2_mechanism_model/SimpleTransmission" name="j1_transmission">
-      <actuator name="j1" />
-      <joint name="${prefix}_joint_1" />
-      <mechanicalReduction>1</mechanicalReduction>
-      <motorTorqueConstant>1</motorTorqueConstant>
+    <transmission name="tran_1">
+      <type>transmission_interface/SimpleTransmission</type>
+      <joint name="${prefix}_joint_1"/>
+      <actuator name="motor1">
+        <hardwareInterface>EffortJointInterface</hardwareInterface>
+      	<mechanicalReduction>1</mechanicalReduction>
+        <motorTorqueConstant>1</motorTorqueConstant>
       <!-- <pulsesPerRevolution>90000</pulsesPerRevolution> -->
+      </actuator>
     </transmission>
   </xacro:macro>

File: ros/iri-ros-pkg/stacks/iri_wam/trunk/iri_wam_description/xacro/iri_wam_2.urdf.xacro (robot description, xacro)
@@ -42,10 +42,13 @@
         <dynamics damping="100"/>
     </joint>
-    <transmission type="pr2_mechanism_model/SimpleTransmission" name="j2_transmission">
-      <actuator name="j2" />
-      <joint name="${prefix}_joint_2" />
-      <mechanicalReduction>1</mechanicalReduction>
-      <motorTorqueConstant>1</motorTorqueConstant>
+    <transmission name="tran_2">
+      <type>transmission_interface/SimpleTransmission</type>
+      <joint name="${prefix}_joint_2"/>
+      <actuator name="motor1">
+        <hardwareInterface>EffortJointInterface</hardwareInterface>
+      	<mechanicalReduction>1</mechanicalReduction>
+        <motorTorqueConstant>1</motorTorqueConstant>
       <!-- <pulsesPerRevolution>90000</pulsesPerRevolution> -->
+      </actuator>
     </transmission>
   </xacro:macro>

File: ros/iri-ros-pkg/stacks/iri_wam/trunk/iri_wam_description/xacro/iri_wam_3.urdf.xacro (robot description, xacro)
@@ -42,10 +42,13 @@
         <dynamics damping="100"/>
     </joint>
-    <transmission type="pr2_mechanism_model/SimpleTransmission" name="j3_transmission">
-      <actuator name="j3" />
-      <joint name="${prefix}_joint_3" />
-      <mechanicalReduction>1</mechanicalReduction>
-      <motorTorqueConstant>1</motorTorqueConstant>
+    <transmission name="tran_3">
+      <type>transmission_interface/SimpleTransmission</type>
+      <joint name="${prefix}_joint_3"/>
+      <actuator name="motor1">
+        <hardwareInterface>EffortJointInterface</hardwareInterface>
+      	<mechanicalReduction>1</mechanicalReduction>
+        <motorTorqueConstant>1</motorTorqueConstant>
       <!-- <pulsesPerRevolution>90000</pulsesPerRevolution> -->
+      </actuator>
     </transmission>
   </xacro:macro>

File: ros/iri-ros-pkg/stacks/iri_wam/trunk/iri_wam_description/xacro/iri_wam_4.urdf.xacro (robot description, xacro)
@@ -42,10 +42,13 @@
         <dynamics damping="100"/>
     </joint>
-    <transmission type="pr2_mechanism_model/SimpleTransmission" name="j4_transmission">
-      <actuator name="j4" />
-      <joint name="${prefix}_joint_4" />
-      <mechanicalReduction>1</mechanicalReduction>
-      <motorTorqueConstant>1</motorTorqueConstant>
+    <transmission name="tran_4">
+      <type>transmission_interface/SimpleTransmission</type>
+      <joint name="${prefix}_joint_4"/>
+      <actuator name="motor1">
+        <hardwareInterface>EffortJointInterface</hardwareInterface>
+      	<mechanicalReduction>1</mechanicalReduction>
+        <motorTorqueConstant>1</motorTorqueConstant>
       <!-- <pulsesPerRevolution>90000</pulsesPerRevolution> -->
+      </actuator>
     </transmission>
   </xacro:macro>

File: ros/iri-ros-pkg/stacks/iri_wam/trunk/iri_wam_description/xacro/iri_wam_5.urdf.xacro (robot description, xacro)
@@ -42,10 +42,13 @@
         <dynamics damping="100"/>
     </joint>
-    <transmission type="pr2_mechanism_model/SimpleTransmission" name="j5_transmission">
-      <actuator name="j5" />
-      <joint name="${prefix}_joint_5" />
-      <mechanicalReduction>1</mechanicalReduction>
-      <motorTorqueConstant>1</motorTorqueConstant>
+    <transmission name="tran_5">
+      <type>transmission_interface/SimpleTransmission</type>
+      <joint name="${prefix}_joint_5"/>
+      <actuator name="motor1">
+        <hardwareInterface>EffortJointInterface</hardwareInterface>
+      	<mechanicalReduction>1</mechanicalReduction>
+        <motorTorqueConstant>1</motorTorqueConstant>
       <!-- <pulsesPerRevolution>90000</pulsesPerRevolution> -->
+      </actuator>
     </transmission>
   </xacro:macro>

File: ros/iri-ros-pkg/stacks/iri_wam/trunk/iri_wam_description/xacro/iri_wam_6.urdf.xacro (robot description, xacro)
@@ -42,10 +42,13 @@
         <dynamics damping="100"/>
     </joint>
-    <transmission type="pr2_mechanism_model/SimpleTransmission" name="j6_transmission">
-      <actuator name="j6" />
-      <joint name="${prefix}_joint_6" />
-      <mechanicalReduction>1</mechanicalReduction>
-      <motorTorqueConstant>1</motorTorqueConstant>
+    <transmission name="tran_6">
+      <type>transmission_interface/SimpleTransmission</type>
+      <joint name="${prefix}_joint_6"/>
+      <actuator name="motor1">
+        <hardwareInterface>EffortJointInterface</hardwareInterface>
+      	<mechanicalReduction>1</mechanicalReduction>
+        <motorTorqueConstant>1</motorTorqueConstant>
       <!-- <pulsesPerRevolution>90000</pulsesPerRevolution> -->
+      </actuator>
     </transmission>
   </xacro:macro>

File: ros/iri-ros-pkg/stacks/iri_wam/trunk/iri_wam_description/xacro/iri_wam_7.urdf.xacro (robot description, xacro)
@@ -42,10 +42,13 @@
         <dynamics damping="100"/>
     </joint>
-    <transmission type="pr2_mechanism_model/SimpleTransmission" name="j7_transmission">
-      <actuator name="j7" />
-      <joint name="${prefix}_joint_7" />
-      <mechanicalReduction>1</mechanicalReduction>
-      <motorTorqueConstant>1</motorTorqueConstant>
+    <transmission name="tran_7">
+      <type>transmission_interface/SimpleTransmission</type>
+      <joint name="${prefix}_joint_7"/>
+      <actuator name="motor1">
+        <hardwareInterface>EffortJointInterface</hardwareInterface>
+      	<mechanicalReduction>1</mechanicalReduction>
+        <motorTorqueConstant>1</motorTorqueConstant>
       <!-- <pulsesPerRevolution>90000</pulsesPerRevolution> -->
+      </actuator>
     </transmission>
   </xacro:macro>
