Commit message: [iri_wam_description]  - Updating miscellaneous object xacro files to spawn them into gazebo

File: ros/iri-ros-pkg/stacks/iri_wam/trunk/iri_wam_description/xacro/iri_wam_1.urdf.xacro (robot description, xacro)
@@ -45,5 +45,5 @@
       <type>transmission_interface/SimpleTransmission</type>
       <joint name="${prefix}_joint_1"/>
-      <actuator name="motor1">
+      <actuator name="motor_1">
         <hardwareInterface>EffortJointInterface</hardwareInterface>
       	<mechanicalReduction>1</mechanicalReduction>

File: ros/iri-ros-pkg/stacks/iri_wam/trunk/iri_wam_description/xacro/iri_wam_2.urdf.xacro (robot description, xacro)
@@ -45,5 +45,5 @@
       <type>transmission_interface/SimpleTransmission</type>
       <joint name="${prefix}_joint_2"/>
-      <actuator name="motor1">
+      <actuator name="motor_2">
         <hardwareInterface>EffortJointInterface</hardwareInterface>
       	<mechanicalReduction>1</mechanicalReduction>

File: ros/iri-ros-pkg/stacks/iri_wam/trunk/iri_wam_description/xacro/iri_wam_3.urdf.xacro (robot description, xacro)
@@ -45,5 +45,5 @@
       <type>transmission_interface/SimpleTransmission</type>
       <joint name="${prefix}_joint_3"/>
-      <actuator name="motor1">
+      <actuator name="motor_3">
         <hardwareInterface>EffortJointInterface</hardwareInterface>
       	<mechanicalReduction>1</mechanicalReduction>

File: ros/iri-ros-pkg/stacks/iri_wam/trunk/iri_wam_description/xacro/iri_wam_4.urdf.xacro (robot description, xacro)
@@ -45,5 +45,5 @@
       <type>transmission_interface/SimpleTransmission</type>
       <joint name="${prefix}_joint_4"/>
-      <actuator name="motor1">
+      <actuator name="motor_4">
         <hardwareInterface>EffortJointInterface</hardwareInterface>
       	<mechanicalReduction>1</mechanicalReduction>

File: ros/iri-ros-pkg/stacks/iri_wam/trunk/iri_wam_description/xacro/iri_wam_5.urdf.xacro (robot description, xacro)
@@ -45,5 +45,5 @@
       <type>transmission_interface/SimpleTransmission</type>
       <joint name="${prefix}_joint_5"/>
-      <actuator name="motor1">
+      <actuator name="motor_5">
         <hardwareInterface>EffortJointInterface</hardwareInterface>
       	<mechanicalReduction>1</mechanicalReduction>

File: ros/iri-ros-pkg/stacks/iri_wam/trunk/iri_wam_description/xacro/iri_wam_6.urdf.xacro (robot description, xacro)
@@ -45,5 +45,5 @@
       <type>transmission_interface/SimpleTransmission</type>
       <joint name="${prefix}_joint_6"/>
-      <actuator name="motor1">
+      <actuator name="motor_6">
         <hardwareInterface>EffortJointInterface</hardwareInterface>
       	<mechanicalReduction>1</mechanicalReduction>

File: ros/iri-ros-pkg/stacks/iri_wam/trunk/iri_wam_description/xacro/iri_wam_7.urdf.xacro (robot description, xacro)
@@ -45,5 +45,5 @@
       <type>transmission_interface/SimpleTransmission</type>
       <joint name="${prefix}_joint_7"/>
-      <actuator name="motor1">
+      <actuator name="motor_7">
         <hardwareInterface>EffortJointInterface</hardwareInterface>
       	<mechanicalReduction>1</mechanicalReduction>

File: ros/iri-ros-pkg/stacks/iri_wam/trunk/iri_wam_description/xacro/misc/box.urdf.xacro (robot description, xacro)
@@ -1,8 +1,4 @@
 <?xml version="1.0"?>
-<robot xmlns:sensor="http://playerstage.sourceforge.net/gazebo/xmlschema/#sensor"
-       xmlns:controller="http://playerstage.sourceforge.net/gazebo/xmlschema/#controller"
-       xmlns:interface="http://playerstage.sourceforge.net/gazebo/xmlschema/#interface"
-       xmlns:xacro="http://ros.org/wiki/xacro"
-       name="simple_box">
+<robot name="box" xmlns:xacro="http://ros.org/wiki/xacro">
   <xacro:property name="box_tx" value="0.0" />
   <xacro:property name="box_ty" value="0.0" />
@@ -39,5 +35,5 @@
   <gazebo reference="box">
     <material>Gazebo/Blue</material>
-    <turnGravityOff>true</turnGravityOff>
+    <turnGravityOff>false</turnGravityOff>
   </gazebo>
  </robot>

File: ros/iri-ros-pkg/stacks/iri_wam/trunk/iri_wam_description/xacro/misc/cylinder.urdf.xacro (robot description, xacro)
@@ -1,18 +1,4 @@
 <?xml version="1.0"?>
-<robot name="table"
-       xmlns:xi="http://www.w3.org/2001/XInclude"
-       xmlns:gazebo="http://playerstage.sourceforge.net/gazebo/xmlschema/#gz"
-       xmlns:model="http://playerstage.sourceforge.net/gazebo/xmlschema/#model"
-       xmlns:sensor="http://playerstage.sourceforge.net/gazebo/xmlschema/#sensor"
-       xmlns:body="http://playerstage.sourceforge.net/gazebo/xmlschema/#body"
-       xmlns:geom="http://playerstage.sourceforge.net/gazebo/xmlschema/#geom"
-       xmlns:joint="http://playerstage.sourceforge.net/gazebo/xmlschema/#joint"
-       xmlns:interface="http://playerstage.sourceforge.net/gazebo/xmlschema/#interface"
-       xmlns:rendering="http://playerstage.sourceforge.net/gazebo/xmlschema/#rendering"
-       xmlns:renderable="http://playerstage.sourceforge.net/gazebo/xmlschema/#renderable"
-       xmlns:controller="http://playerstage.sourceforge.net/gazebo/xmlschema/#controller"
-       xmlns:physics="http://playerstage.sourceforge.net/gazebo/xmlschema/#physics">
-  <property name="table_z" value="0.0" />
-  <property name="table_height" value="0.55" />
+<robot name="cylinder" xmlns:xacro="http://ros.org/wiki/xacro">
   <property name="object_1_x" value="0.0" />
   <property name="object_1_y" value="0.0" />
@@ -23,5 +9,5 @@
   <property name="object_1_mass"        value="0.2" />
   <property name="object_1_mu"          value="500.0" />
-  <link name="stick">
+  <link name="cylinder">
     <inertial>
       <mass value="${object_1_mass/2.0}" />
@@ -44,5 +30,5 @@
     </collision>
   </link>
-  <gazebo reference="stick">
+  <gazebo reference="cylinder">
     <material>Gazebo/BumpyMetal</material>
     <mu1>${object_1_mu}</mu1>
@@ -51,5 +37,5 @@
     <kd>1.0</kd>
     <selfCollide>true</selfCollide>
-    <turnGravityOff>true</turnGravityOff>
+    <turnGravityOff>false</turnGravityOff>
     <dampingFactor>0.001</dampingFactor>
   </gazebo>

File: ros/iri-ros-pkg/stacks/iri_wam/trunk/iri_wam_description/xacro/misc/table.urdf.xacro (robot description, xacro)
@@ -1,33 +1,12 @@
 <?xml version="1.0"?>
-<robot name="table"
-       xmlns:xi="http://www.w3.org/2001/XInclude"
-       xmlns:gazebo="http://playerstage.sourceforge.net/gazebo/xmlschema/#gz"
-       xmlns:model="http://playerstage.sourceforge.net/gazebo/xmlschema/#model"
-       xmlns:sensor="http://playerstage.sourceforge.net/gazebo/xmlschema/#sensor"
-       xmlns:body="http://playerstage.sourceforge.net/gazebo/xmlschema/#body"
-       xmlns:geom="http://playerstage.sourceforge.net/gazebo/xmlschema/#geom"
-       xmlns:joint="http://playerstage.sourceforge.net/gazebo/xmlschema/#joint"
-       xmlns:interface="http://playerstage.sourceforge.net/gazebo/xmlschema/#interface"
-       xmlns:rendering="http://playerstage.sourceforge.net/gazebo/xmlschema/#rendering"
-       xmlns:renderable="http://playerstage.sourceforge.net/gazebo/xmlschema/#renderable"
-       xmlns:controller="http://playerstage.sourceforge.net/gazebo/xmlschema/#controller"
-       xmlns:physics="http://playerstage.sourceforge.net/gazebo/xmlschema/#physics"
-       xmlns:xacro="http://www.ros.org/wiki/xacro">
-  <property name="table_height" value="0.892" />
-  <property name="table_width" value="1.14" />
+<robot name="table" xmlns:xacro="http://www.ros.org/wiki/xacro">
+  <property name="table_height" value="0.9" />
+  <property name="table_width" value="1.2" />
   <property name="table_depth" value="0.5" />
   <property name="table_x" value="0.0" />
   <property name="table_y" value="0.0" />
   <property name="table_z" value="0.0" />
-  <!-- tabletop height is .55+.01+.025=.585 -->
   <property name="table_top_thickness" value="0.05"/>
   <property name="M_PI" value="3.1415926535897931" />
-    <include filename="$(find iri_wam_description)/xacro/wam0_2.urdf.xacro" />
-    <include filename="$(find iri_wam_description)/xacro/wam1_2.urdf.xacro" />
-    <include filename="$(find iri_wam_description)/xacro/wam2_2.urdf.xacro" />
-    <include filename="$(find iri_wam_description)/xacro/wam3_2.urdf.xacro" />
-    <include filename="$(find iri_wam_description)/xacro/wam4_2.urdf.xacro" />
-    <include filename="$(find iri_wam_description)/xacro/wam5_2.urdf.xacro" />
-    <include filename="$(find iri_wam_description)/xacro/wam6_2.urdf.xacro" />
   <link name ="world" />
   <link name="leg_1">
@@ -49,12 +28,5 @@
       </geometry>
     </collision>
-   </link>
-  <gazebo reference="leg_1">
-		<material>Gazebo/LightWood</material>
-		<mu1>50.0</mu1>
-		 <mu2>50.0</mu2>
-		<kp>1000000.0</kp>
-		<kd>1.0</kd>
-	</gazebo>
+  </link>
   <joint name="table_fix1" type="fixed">
      <parent link="world"/>
@@ -62,4 +34,11 @@
      <origin xyz="0 0 ${table_depth/2}" rpy="0 0 0" />
   </joint>
+  <gazebo reference="leg_1">
+    <material>Gazebo/LightWood</material>
+    <mu1>50.0</mu1>
+    <mu2>50.0</mu2>
+    <kp>1000000.0</kp>
+    <kd>1.0</kd>
+  </gazebo>
   <link name="table_top_link">
     <inertial>
@@ -81,16 +60,16 @@
     </collision>
   </link>
+  <joint name="table_fix2" type="fixed">
+    <parent link="leg_1"/>
+    <child link="table_top_link"/>
+    <origin xyz="0 0 ${table_depth}" rpy="0 0 0" />
+  </joint>
   <gazebo reference="table_top_link">
-		<material>Gazebo/LightWood</material>
-		<mu1>50.0</mu1>
-		 <mu2>50.0</mu2>
-		<kp>1000000.0</kp>
-		<kd>1.0</kd>
-	</gazebo>
-  <joint name="table_fix2" type="fixed">
-     <parent link="leg_1"/>
-     <child link="table_top_link"/>
-     <origin xyz="0 0 ${table_depth}" rpy="0 0 0" />
-  </joint>
+    <material>Gazebo/LightWood</material>
+    <mu1>50.0</mu1>
+    <mu2>50.0</mu2>
+    <kp>1000000.0</kp>
+    <kd>1.0</kd>
+  </gazebo>
   <link name="leg_2">
     <inertial>
@@ -111,23 +90,16 @@
       </geometry>
     </collision>
-   </link>
+  </link>
+  <joint name="table_fix3" type="fixed">
+    <parent link="table_top_link"/>
+    <child link="leg_2"/>
+    <origin xyz="${table_depth-table_top_thickness} 0 0" rpy="${M_PI /2} 0 ${M_PI /2}" />
+  </joint>
   <gazebo reference="leg_2">
-		<material>Gazebo/LightWood</material>
-		<mu1>50.0</mu1>
-		 <mu2>50.0</mu2>
-		<kp>1000000.0</kp>
-		<kd>1.0</kd>
-	</gazebo>
-  <joint name="table_fix3" type="fixed">
-     <parent link="table_top_link"/>
-     <child link="leg_2"/>
-     <origin xyz="${table_depth-table_top_thickness} 0 0" rpy="${M_PI /2} 0 ${M_PI /2}" />
-  </joint>
-  <xacro:wam0 parent="table_top_link" rot="0 0 0" trasl="${table_depth/2+table_top_thickness/2} 0 -${table_depth/2- table_top_thickness}"></xacro:wam0>
- <!--  <xacro:wam1 parent="wam_link0" rot ="0 0 0" trasl="0 0 0.05"></xacro:wam1>
- <xacro:wam2 parent="wam_link1" rot ="-${M_PI /2} 0 0" trasl="0 -0.1 0"></xacro:wam2>
-  <xacro:wam3 parent="wam_link2" rot= "${M_PI /2} 0 0" trasl="-${table_depth/2-table_top_thickness+0.22+0.03} ${table_x} ${table_depth+table_top_thickness+0.1}"></xacro:wam3>
-  <xacro:wam4 parent="wam_link3" rot= "-${M_PI /2} 0 0" trasl="-${table_depth/2-table_top_thickness+0.195} -${table_depth+table_top_thickness+0.65} ${table_x}"></xacro:wam4>
-  <xacro:wam5 parent="wam_link4" rot= "${M_PI /2} 0 0" trasl="-${table_depth/2-table_top_thickness+0.24} ${table_x} ${table_depth+table_top_thickness+0.955}"></xacro:wam5>
-  <xacro:wam6 parent="wam_link5" rot= "-${M_PI /2} 0 0" trasl="-${table_depth/2-table_top_thickness+0.24} -${table_depth+table_top_thickness+0.955} ${table_x} "></xacro:wam6> -->
+    <material>Gazebo/LightWood</material>
+    <mu1>50.0</mu1>
+    <mu2>50.0</mu2>
+    <kp>1000000.0</kp>
+    <kd>1.0</kd>
+  </gazebo>
 </robot>
